File: Avionics/FlightComputer/SubArctic AM335x_2.kicad_sch (KiCad schematic)
At the start: 13 parts

Commit message: Ian Goldberg - Finished the pinout for the second sheet of the SubArctic chip and becan working on the connected circuitry
Parts:
- added R28: 33R,5%, symbol Device:R
- added R45: 22R,1%, symbol Device:R
- added R46, R47, R48: 0R,5%, symbol Device:R
Connections:
- new net: R28.1, SubArcticAM335X2.H18 (RMII1_REFCLK/XDMA_EVENT_INTR2/SPI1_CS0/UART5_TXD/MCASP1_AXR3/MMC0_POW_/MCASP1_AHCLKX/GPIO0_29)
- new net: U8. (VBUS), U9. (VB) (x3)
- new net: U6. (VBUS), U7. (VBUS) (x2)
- new net: R46.1, SubArcticAM335X2.U5 (LCD_VSYNC/GPMC_A8//PR1_EDIO_DATA_IN2/PR1_EDIO_DATA_OUT2/PR1_PRU1_PRU_R30_8/PR1_PRU1_PRU_R31_8/GPIO2_22)
- new net: R45.1, SubArcticAM335X2.V5 (LCD_PCLK/GPMC_A10//PR1_EDIO_DATA_IN4/PR1_EDIO_DATA_OUT4/PR1_PRU1_PRU_R30_10/PR1_PRU1_PRU_R31_10/GPIO2_24)
- new net: R47.1, SubArcticAM335X2.R5 (LCD_HSYNC/GPMC_A9//PR1_EDIO_DATA_IN3/PR1_EDIO_DATA_OUT3/PR1_PRU1_PRU_R30_9/PR1_PRU1_PRU_R31_9/GPIO2_23)
- new net: R48.1, SubArcticAM335X2.R6 (LCD_AC_BIAS_EN/GPMC_A11//PR1_EDIO_DATA_IN5/PR1_EDIO_DATA_OUT5/PR1_PRU1_PRU_R30_11/PR1_PRU1_PRU_R31_11/GPIO2_25)
- new net GPIO3_19: SubArcticAM335X2.C13 (MCASP0_FSR/EQEP0B_IN/MCASP0_AXR3/MCASP1_FSX/EMU2/PR1_PRU0_PRU_R30_5/PR1_PRU0_PRU_R31_5/GPIO3_19)
- new net GPIO3_20: SubArcticAM335X2.D13 (MCASP0_AXR1/EQEP0_INDEX//MCASP1_AXR0/EMU3/PR1_PRU0_PRU_R30_6/PR1_PRU0_PRU_R31_6/GPIO3_20)
- new net GPIO3_21: SubArcticAM335X2.A14 (MCASP0_AHCLKX/EQEP0_STROBE/MCASP0_AXR3/MCASP1_AXR1/EMU4/PR1_PRU0_PRU_R30_7/PR1_PRU0_PRU_R31_7/GPIO3_21)
- new net LCD_DATA0: SubArcticAM335X2.R1 (LCD_DATA0/GPMC_A0//EHRPW_M2A//PR1_PRU1_PRU_R30_0/PR1_PRU1_PRU_R31_0/GPIO2_6)
- new net LCD_DATA1: SubArcticAM335X2.R2 (LCD_DATA1/GPMC_A1//EHRPW_M2B//PR1_PRU1_PRU_R30_1/PR1_PRU1_PRU_R31_1/GPIO2_7)
- new net LCD_DATA10: SubArcticAM335X2.U3 (LCD_DATA10/GPMC_A14/EHRPW_M1A/MCASP0_AXR0//PR1_MII0_RXD1/UART3_CTSN/GPIO2_16)
- new net LCD_DATA11: SubArcticAM335X2.U4 (LCD_DATA11/GPMC_A15/EHRPW_M1B/MCASP0_AHCLKR/MCASP0_AXR2/PR1_MII0_RXD0/UART3_RTSN/GPIO2_17)
- new net LCD_DATA12: SubArcticAM335X2.V2 (LCD_DATA12/GPMC_A16/EQEP1A_IN/MCASP0_ACLKR/MCASP0_AXR2/PR1_MII0_RXLINK/UART4_CTSN/GPIO0_8)
- new net LCD_DATA13: SubArcticAM335X2.V3 (LCD_DATA13/GPMC_A17/EQEP1B_IN/MCASP0_FSR/MCASP0_AXR3/PR1_MII0_RXER/UART4_RTSN/GPIO0_9)
- new net LCD_DATA14: SubArcticAM335X2.V4 (LCD_DATA14/GPMC_A18/EQEP1_INDEX/MCASP0_AXR1/UART5_RXD/PR1_MII_MR0_CLK/UART5_CTSN/GPIO0_10)
- new net LCD_DATA15: SubArcticAM335X2.T5 (LCD_DATA15/GPMC_A19/EQEP1_STROBE/MCASP0_AHCLKX/MCASP0_AXR3/PR1_MII0_RXDV/UART5_RTSN/GPIO0_11)
- new net LCD_DATA2: SubArcticAM335X2.R3 (LCD_DATA2/GPMC_A2//EHRPW_M2_TRIPZONE_INPUT//PR1_PRU1_PRU_R30_2/PR1_PRU1_PRU_R31_2/GPIO2_8)
- new net LCD_DATA3: SubArcticAM335X2.R4 (LCD_DATA3/GPMC_A3//EHRPW_M2_SYNCI_O//PR1_PRU1_PRU_R30_3/PR1_PRU1_PRU_R31_3/GPIO2_9)
- new net LCD_DATA4: SubArcticAM335X2.T1 (LCD_DATA4/GPMC_A4//EQEP2A_IN//PR1_PRU1_PRU_R30_4/PR1_PRU1_PRU_R31_4/GPIO2_10)
- new net LCD_DATA5: SubArcticAM335X2.T2 (LCD_DATA5/GPMC_A5//EQEP2B_IN//PR1_PRU1_PRU_R30_5/PR1_PRU1_PRU_R31_5/GPIO2_11)
- new net LCD_DATA6: SubArcticAM335X2.T3 (LCD_DATA6/GPMC_A6/PR1_EDIO_DATA_IN6/EQEP2_INDEX/PR1_EDIO_DATA_OUT6/PR1_PRU1_PRU_R30_6/PR1_PRU1_PRU_R31_6/GPIO2_12)
- new net LCD_DATA7: SubArcticAM335X2.T4 (LCD_DATA7/GPMC_A7/PR1_EDIO_DATA_IN7/EQEP2_STROBE/PR1_EDIO_DATA_OUT7/PR1_PRU1_PRU_R30_7/PR1_PRU1_PRU_R31_7/GPIO2_13)
- new net LCD_DATA8: SubArcticAM335X2.U1 (LCD_DATA8/GPMC_A12/EHRPW_M1_TRIPZONE_INPUT/MCASP0_ACLKX/UART5_TXD/PR1_MII0_RXD3/UART2_CTSN/GPIO2_14)
- new net LCD_DATA9: SubArcticAM335X2.U2 (LCD_DATA9/GPMC_A13/EHRPW_M1_SYNCI_O/MCASP0_FSX/UART5_RXD/PR1_MII0_RXD2/UART2_RTSN/GPIO2_15)
- new net LCD_DE: R48.2
- new net LCD_HSYNC: R47.2
- new net LCD_PCLK: R45.2
- new net LCD_VSYNC: R46.2
- new net MDIO_CLK: SubArcticAM335X2.M18 (MDIO_CLK/TIMER5/UART5_TXD/UART3_RTSN/MMC0_SDW_P/MMC1_CLK/MMC2_CLK/GPIO0_1)
- new net MDIO_DATA: SubArcticAM335X2.M17 (MDIO_DATA/TIMER6/UART5_RXD/UART3_CTSN/MMC0_SDCD/MMC1_CMD/MMC2_CMD/GPIO0_0)
- new net MII1_COL: SubArcticAM335X2.H16 (GMII1_COL/RMII2_REFCLK/SPI1_SCLK/UART5_RXD/MCASP1_AXR2/MMC2_DAT3/MCASP0_AXR2/GPIO3_0)
- new net MII1_CRS_DV: SubArcticAM335X2.H17 (GMII1_CRS/RMII1_CRS_DV/SPI1_D0/I2C1_SDA/MCASP1_ACLKX/UART5_CTSN/UART2_RXD/GPIO3_1), SubArcticAM335X2.J16 (GMII1_TXEN/RMII1_TXEN/RGMII1_TCTL/TIMER4/MCASP1_AXR0/EQEP0_INDEX/MMC2_CMD/GPIO3_3)
- new net MII1_REFCLK: R28.2
- new net MII1_RXCLK: SubArcticAM335X2.L18 (GMII1_RXCLK/UART2_TXD/RGMII1_RCLK/MMC0_DAT6/MMC1_DAT1/UART1_DSRN/MCASP0_FSX/GPIO3_10)
- new net MII1_RXD0: SubArcticAM335X2.M16 (GMII1_RXD0/RMII1_RXD0/RGMII1_RD0/MCASP1_AHCLKX/MCASP1_AHCLKR/MCASP1_ACLKR/MCASP0_AXR3/GPIO2_21)
- new net MII1_RXD1: SubArcticAM335X2.L15 (GMII1_RXD1/RMII1_RXD1/RGMII1_RD1/MCASP1_AXR3/MCASP1_FSR/EQEP0_STROBE/MMC2_CLK/GPIO2_20)
- new net MII1_RXD2: SubArcticAM335X2.L16 (GMII1_RXD2/UART3_TXD/RGMII1_RD2/MMC0_DAT4/MMC1_DAT3/UART1_RIN/MCASP0_AXR1/GPIO2_19)
- new net MII1_RXDV: SubArcticAM335X2.J17 (GMII1_RXDV/LCD_MEMORY_CLK/RGMII1_RCTL/UART5_TXD/MCASP1_ACLKX/MMC2_DAT0/MCASP0_ACLKR/GPIO3_4)
- new net MII1_RXERR: SubArcticAM335X2.J15 (GMII1_RXERR/RMII1_RXERR/SPI1_D1/I2C1_SCL/MCASP1_FSX/UART5_RTSN/UART2_TXD/GPIO3_2)
- new net MII1_TXCL3: SubArcticAM335X2.L17 (GMII1_RXD3/UART3_RXD/RGMII1_RD3/MMC0_DAT5/MMC1_DAT2/UART1_DTRN/MCASP0_AXR0/GPIO2_18)
- new net MII1_TXCLK: SubArcticAM335X2.K18 (GMII1_TXCLK/UART2_RXD/RGMII1_TCLK/MMC0_DAT7/MMC1_DAT0/UART1_DCDN/MCASP0_ACLKX/GPIO3_9)
- new net MII1_TXD0: SubArcticAM335X2.K17 (GMII1_TXD0/RMII1_TXD0/RGMII1_TD0/MCASP1_AXR2/MCASP1_ACLKR/EQEP0B_IN/MMC1_CLK/GPIO0_28)
- new net MII1_TXD1: SubArcticAM335X2.K16 (GMII1_TXD1/RMII1_TXD1/RGMII1_TD1/MCASP1_FSR/MCASP1_AXR1/EQEP0A_IN/MMC1_CMD/GPIO0_21)
- new net MII1_TXD2: SubArcticAM335X2.K15 (GMII1_TXD2/DCAN0_RX/RGMII1_TD2/UART4_TXD/MCASP1_AXR0/MMC2_DAT2/MCASP0_AHCLKX/GPIO0_17)
- new net MII1_TXEN: SubArcticAM335X2.J18 (GMII1_TXD3/DCAN0_TX/RGMII1_TD3/UART4_RXD/MCASP1_FSX/MMC2_DAT1/MCASP0_FSR/GPIO0_16)
- new net SPI1_CS0: SubArcticAM335X2.C12 (MCASP0_AHCLKR/EHRPW_M0_SYNCI_O/MCASP0_AXR2/SPI1_CS0/ECAP2_IN_PW_M2_OUT/PR1_PRU0_PRU_R30_3/PR1_PRU0_PRU_R31_3/GPIO3_17)
- new net SPI1_D0: SubArcticAM335X2.B13 (MCASP0_FSX/EHRPW_M0B//SPI1_D0/MMC1_SDCD/PR1_PRU0_PRU_R30_1/PR1_PRU0_PRU_R31_1/GPIO3_15)
- new net SPI1_D1: SubArcticAM335X2.D12 (MCASP0_AXR0/EHRPW_M0_TRIPZONE_INPUT//SPI1_D1/MMC2_SDCD/PR1_PRU0_PRU_R30_2/PR1_PRU0_PRU_R31_2/GPIO3_16)
- new net SPI1_SCLK: SubArcticAM335X2.A13 (MCASP0_ACLKX/EHRPW_M0A//SPI1_SCLK/MMC0_SDCD/PR1_PRU0_PRU_R30_0/PR1_PRU0_PRU_R31_0/GPIO3_14)
Other:
- moved on the sheet: C34, C35, C36, FB7, R37, R52, R53, U5, U7

Commit message: Ian Goldberg - Finished the pin-out for the third schematic of the SubArctic chip. All that remains is finishing up the rest of the circuit.
Parts:
- added C155, C31, C33: 100nF,16V, symbol Device:C
- added C32: 1nF,50V, symbol Device:C
- added R10, R163, R26: 4.7K,1%, symbol Device:R
- added R11, R27, R49, R50, R51: 0R,5%, symbol Device:R
- added R165: 100K,1%, symbol Device:R
- added TP9: TestPoint, symbol Connector:TestPoint
- added U10: ~, symbol SubArctic AM335x:SN74LVC2G241DCUR
- added U11: ~, symbol SubArctic AM335x:Header_1x6Pin_2.54MM
Connections:
- net DGND: now also C155.1, R10.2, R11.1, R165.2, U10. (VCC), U11. (6)
- net USB_DC: now also R49.1
- net I2C1_SCL: now reaches SubArcticAM335X2.A16 (SPI0_CS0/MMC2_SDW_P/I2C1_SCL/EHRPW_M0_SYNCI_O/PR1_UART0_TXD/PR1_EDIO_DATA_IN1/PR1_EDIO_DATA_OUT1/GPIO0_5)
- net UART2_TXD: now reaches SubArcticAM335X2.A17 (SPI0_SCLK/UART2_RXD/I2C2_SDA/EHRPW_M0A/PR1_UART0_CTS_N/PR1_EDIO_SOF/EMU2/GPIO0_2)
- net UART2_TXD: now also SubArcticAM335X2.B17 (SPI0_D0/UART2_TXD/I2C2_SCL/EHRPW_M0B/PR1_UART0_RTS_N/PR1_EDIO_LATCH_IN/EMU3/GPIO0_3)
- net AIN3: now reaches SubArcticAM335X2.A7 (AIN3)
- net AIN6: now reaches SubArcticAM335X2.A8 (AIN6)
- net at SubArcticAM335X2.B12 (MCASP0_ACLKR/EQEP0A_IN/MCASP0_AXR2/MCASP1_ACLKX/MMC0_SDW_P/PR1_PRU0_PRU_R30_4/PR1_PRU0_PRU_R31_4/GPIO3_18): now also R51.2
- net I2C1_SDA: now reaches SubArcticAM335X2.B16 (SPI0_D1/MMC1_SDW_P/I2C1_SDA/EHRPW_M0_TRIPZONE_INPUT/PR1_UART0_RXD/PR1_EDIO_DATA_IN0/PR1_EDIO_DATA_OUT0/GPIO0_4)
- net AIN0: now reaches SubArcticAM335X2.B6 (AIN0)
- net AIN2: now reaches SubArcticAM335X2.B7 (AIN2)
- net AIN5: now reaches SubArcticAM335X2.B8 (AIN5)
- net GNDA_ADC: now reaches SubArcticAM335X2.B9 (VREFP)
- net GNDA_ADC: now also C31.1, C31.2, C32.1, C32.2, C33.1, C33.2, R27.2
- net MMC0_CD: now reaches SubArcticAM335X2.C15 (SPI0_CS1/UART3_RXD/ECAP1_IN_PW_M1_OUT/MMC0_POW_/XDMA_EVENT_INTR2/MMC0_SDCD/EMU4/GPIO0_6)
- net I2C0_SCL: now reaches SubArcticAM335X2.C16 (I2C0_SCL/TIMER7/UART2_RTSN/ECAP1_IN_PW_M1_OUT////GPIO3_6)
- net I2C0_SDA: now reaches SubArcticAM335X2.C17 (I2C0_SDA/TIMER4/UART2_CTSN/ECAP2_IN_PW_M2_OUT////GPIO3_5)
- net at SubArcticAM335X2.C18 (ECAP0_IN_PW_M0_OUT_/UART_3_T_XD/SPI1_CS1/PR1_ECAP0_ECAP_CAPIN_APW_M_O/SPI1_SCLK/MMC0_SDW_P/XDMA_EVENT__INT_R2/GPIO0_7): now also R50.2
- net WAKEUP: now reaches SubArcticAM335X2.C5 (EXT_WAKEUP)
- net WAKEUP: now also R26.2
- net PMIC_POWR_EN: now reaches SubArcticAM335X2.C6 (PMIC_POW_ER_EN)
- net AIN1: now reaches SubArcticAM335X2.C7 (AIN1)
- net AIN4: now reaches SubArcticAM335X2.C8 (AIN4)
- net at SubArcticAM335X2.C9 (AIN7): now also R10.1, R163.2
- net UART1_TXD: now reaches SubArcticAM335X2.D15 (UART1_TXD/MMC2_SDW_P/DCAN1_RX/I2C1_SCL//PR1_UART0_TXD/PR1_PRU0_PRU_R31_16/GPIO0_15)
- net UART1_RXD: now reaches SubArcticAM335X2.D16 (UART1_RXD/MMC1_SDW_P/DCAN1_TX/I2C1_SDA//PR1_UART0_RXD/PR1_PRU1_PRU_R31_16/GPIO0_14)
- net I2C2_SCL: now reaches SubArcticAM335X2.D17 (UART1_RTSN/TIMER5/DCAN0_RX/I2C2_SCL/SPI1_CS1/PR1_UART0_RTS_N/PR1_EDC_LATCH1_IN/GPIO0_13)
- net I2C2_SDA: now reaches SubArcticAM335X2.D18 (UART1_CTSN/TIMER6/DCAN0_TX/I2C2_SDA/SPI1_CS0/PR1_UART0_CTS_N/PR1_EDC_LATCH0_IN/GPIO0_12)
- net at SubArcticAM335X2.E15 (UART0_RXD/SPI1_CS0/DCAN0_TX/I2C2_SDA/ECAP2_IN_PW_M2_OUT/PR1_PRU1_PRU_R30_14/PR1_PRU1_PRU_R31_14/GPIO1_10): now also U10. (VCC)
- net at SubArcticAM335X2.E16 (UART0_TXD/SPI1_CS1/DCAN0_RX/I2C2_SCL/ECAP1_IN_PW_M1_OUT/PR1_PRU1_PRU_R30_15/PR1_PRU1_PRU_R31_15/GPIO1_11): now also U10. (VCC)
- net at SubArcticAM335X2.E17 (UART0_RTSN/UART4_TXD/DCAN1_RX/I2C1_SCL/SPI1_D1/SPI1_CS0/PR1_EDC_SYNC1_OUT/GPIO1_9): now also TP9.1
- net ETH_RST_GPIO1_8: now reaches SubArcticAM335X2.E18 (UART0_CTSN/UART4_RXD/DCAN1_TX/I2C1_SDA/SPI1_D0/TIMER7/PR1_EDC_SYNC0_OUT/GPIO1_8)
- net at SubArcticAM335X2.P15 (USB0_VBUS): now also R49.2
- net at SubArcticAM335X2.P17 (USB1_ID): now also R11.2
- net at SubArcticAM335X2.T18 (USB1_VBUS): now also R37.1
- new net: U8. (VBUS), U9. (VB) (x3)
- new net: U6. (VBUS), U7. (VBUS) (x2)
- new net: R165.1, U10. (VCC), U11. (6)
- new net: U10. (VCC), U11. (6)
- new net GPIO0_7: R50.1, R51.1
- new net VDD_3V3B: C155.2, R163.1, U10. (VCC)
- new net VDD_ADC: R27.1
- new net VRTC: R26.1
- no-connect marks 3 -> 15
Other:
- note added: "Mark pin 1 clearly"
- note added: "POWERDOWN ISOLATION"
- note added: "SubArctic AM335x Schematic #2 - Ian Goldberg"
- note added: "UART0 Serial Port USB to TTL Serial Cable 3.3V"
- note added: "USB HOST"
- title: (none) -> SubArctic AM335x Schematic #2 - Ian Goldberg
- moved on the sheet: C34, C35, C36, FB7, R37, R52, R53, U5
