File: Avionics/FlightComputer/SubArctic AM335X_3.kicad_sch (KiCad schematic)
At the start: 23 parts

Commit message: Ian Goldberg - Finished the 3rd sheet of pin-outs for the SubArctic chip. Hopefully this is the last of the manual work I do for the scematic...
Parts:
- added C100, C101, C102, C103, C105, C37, C38, C4, C5, C56, C57, C58, C59, C60, C61, C66, C68, C69, C70, C71, C72, C73, C74, C75, C76, C77, C78, C79, C80, C81, C82, C86, C87, C88, C92, C94, C97, C98, C99: 100nF,16V, symbol Device:C
- added C104, C106, C83, C84, C85, C89, C90, C91: 1uF,10V, symbol Device:C
- added C95, C96: 10uF,16V, symbol Device:C
- added FB1, FB2, FB3: 150R,800mA, symbol Device:L
- added R54: 10K,1%, symbol Device:R
- added TP2, TP3: TestPoint, symbol Connector:TestPoint
Connections:
- net DGND: now also SubArcticAM335X3.M14 (VSSA_USB2), SubArcticAM335X3.N14 (VSSA_USB1), C100.2, C101.2, C102.2, C103.2, C104.2, C105.2, C106.2, C37.2, C38.2, C4.2, C56.1, C57.1, C58.2, C59.2, C60.1, C61.1, C66.2, C68.1, C69.1, C70.1, C71.1, C72.1, C73.1, C74.2, C75.2, C76.2, C77.2, C78.2, C79.2, C80.2, C81.2, C82.2, C83.2, C84.2, C85.2, C86.2, C87.2, C88.2, C89.2, C90.2, C91.2, C92.2, C94.2, C95.2, C96.2, C97.2, C98.2, C99.2, FB3.2, R54.2
- net at SubArcticAM335X3.A2 (VDD_MPU_MON): now also TP2.1
- net at SubArcticAM335X3.A3 (TESTOUT): now also TP3.1
- net at SubArcticAM335X3.B4 (ENZ_KALDO_1P8V): now also R54.1
- net at SubArcticAM335X3.C10 (CAP_VBB_MPU): now also C91.1
- net VDD_PLL: now reaches SubArcticAM335X3.D10 (VDDS_SRAM_MPU_BB)
- net VDD_PLL: now also SubArcticAM335X3.E7 (VDDS_PLL_DDR), SubArcticAM335X3.H15 (VDDS_PLL_MPU), SubArcticAM335X3.R10 (VDDS_PLL_CORE_LCD), SubArcticAM335X3.R11 (VDDS_OSC), C106.1, C78.1, C79.1, C92.1, C94.1, FB1.1, FB1.2
- net at SubArcticAM335X3.D11 (CAP_VDD_SRAM_MPU): now also C90.1
- net at SubArcticAM335X3.D6 (CAP_VDD_RTC): now also C104.1
- net VRTC: now reaches SubArcticAM335X3.D7 (VDDS_RTC)
- net VRTC: now also C105.1
- net VDD_ADC: now reaches SubArcticAM335X3.D8 (VDDA_ADC)
- net VDD_ADC: now also C5.2, FB2.1
- net at SubArcticAM335X3.D9 (CAP_VDD_SRAM_CORE): now also C89.1
- net VDD_3V3A: now reaches SubArcticAM335X3.E10 (VDDSHV61)
- net VDD_3V3A: now also SubArcticAM335X3.E11 (VDDSHV62), SubArcticAM335X3.E12 (VDDSHV63), SubArcticAM335X3.E13 (VDDSHV64), SubArcticAM335X3.F14 (VDDSHV65), SubArcticAM335X3.G14 (VDDSHV66), SubArcticAM335X3.H14 (VDDSHV41), SubArcticAM335X3.J14 (VDDSHV42), SubArcticAM335X3.K14 (VDDSHV51), SubArcticAM335X3.L14 (VDDSHV52), SubArcticAM335X3.N15 (VDDA3P3V_USB0), SubArcticAM335X3.N5 (VDDSHV67), SubArcticAM335X3.P10 (VDDSHV21), SubArcticAM335X3.P11 (VDDSHV22), SubArcticAM335X3.P12 (VDDSHV31), SubArcticAM335X3.P13 (VDDSHV32), SubArcticAM335X3.P5 (VDDSHV68), SubArcticAM335X3.P6 (VDDSHV69), SubArcticAM335X3.P7 (VDDSHV11), SubArcticAM335X3.P8 (VDDSHV12), SubArcticAM335X3.R15 (VDDA3P3V_USB1), C37.1, C38.1, C4.1, C56.2, C57.2, C58.1, C59.1, C60.2, C61.2, C66.1, C68.2, C69.2, C70.2, C71.2, C72.2, C73.2, C74.1, C75.1, C76.1, C77.1, C87.1
- net VDDS: now reaches SubArcticAM335X3.E14 (VDDS2)
- net VDDS: now also SubArcticAM335X3.E6 (VDDS1), SubArcticAM335X3.F9 (VDDS3), SubArcticAM335X3.K13 (VDDS4), SubArcticAM335X3.N6 (VDDS5), SubArcticAM335X3.P14 (VDDS7), SubArcticAM335X3.P9 (VDDS6), C80.1, C81.1, C82.1, C83.1, C84.1, C85.1
- net VDDS_DDR: now reaches SubArcticAM335X3.E5 (VDDS_DDR1)
- net VDDS_DDR: now also SubArcticAM335X3.F5 (VDDS_DDR2), SubArcticAM335X3.G5 (VDDS_DDR3), SubArcticAM335X3.H5 (VDDS_DDR4), SubArcticAM335X3.J5 (VDDS_DDR5), SubArcticAM335X3.K5 (VDDS_DDR6), SubArcticAM335X3.L5 (VDDS_DDR7), C100.1, C101.1, C102.1, C103.1, C95.1, C96.1, C97.1, C98.1, C99.1
- net GNDA_ADC: now reaches SubArcticAM335X3.E8 (VSSA_ADC)
- net GNDA_ADC: now also C5.1, FB3.1
- net VDD_1V8: now reaches SubArcticAM335X3.E9 (VDDS_SRAM_CORE_BG)
- net VDD_1V8: now also SubArcticAM335X3.N16 (VDDA1P8V_USB0), SubArcticAM335X3.R16 (VDDA1P8V_USB1), C86.1, C88.1, FB2.2
- no-connect marks 0 -> 1
Other:
- moved on the sheet: C39, C40, C41, C42, C43, C44, C45, C46, C47, C48, C49, C50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
