File: Avionics/FlightComputer/Flightcomputersheet4.kicad_sch (KiCad schematic)
At the start: 34 parts

Commit message: Ian Goldberg - Making updates to the design for the flight computer
Parts:
- added D2, D3, D4, D5: 19-217/BHC-ZL1M2RY/3T, symbol Device:LED
- added R72, R73, R74, R75: 2.2K,5%, symbol Device:R
- added R76, R77, R78, R79: 100K,1%, symbol Device:R
- added U12, U13: DDC114YU, symbol SubArctic AM335x:DDC114YU
Connections:
- net DGND: now also R76.1, R77.1, R78.1, R79.1, U12. (6), U13. (6)
- new net: D4.2 (A), R74.2
- new net: D2.1 (K), U12. (6)
- new net: D2.2 (A), R72.2
- new net: D5.2 (A), R75.2
- new net: D4.1 (K), U13. (6)
- new net: D5.1 (K), U13. (6)
- new net: D3.1 (K), U12. (6)
- new net: D3.2 (A), R73.2
- new net USR0: R76.2, U12. (6)
- new net USR1: R77.2, U12. (6)
- new net USR2: R78.2, U13. (6)
- new net USR3: R79.2, U13. (6)
- new net VDD: R72.1, R73.1, R74.1, R75.1
Other:
- title: Flight Computer Sheet 4 - Ian Goldberg -> Flight Computer Sheet 4: LED, Configuration, and Reset - Ian Goldberg
