File: Avionics/PDU/Untitled/Untitled.kicad_sch (KiCad schematic)
At the start: 8 parts, among them J1 Conn_02x26_Odd_Even, J2 Conn_02x26_Odd_Even, J3 Screw_Terminal_01x02, J4 Screw_Terminal_01x02

Commit message: feat: pdu updates
Parts:
- added C1, C20, C25, C26, C8: 4.7uF, symbol Device:C
- added C10, C13, C15, C17, C2, C22: 0.1uF, symbol Device:C
- added C11, C23, C6: 1uF, symbol Device:C
- added C12, C3: 68uF, symbol Device:C
- added C14, C16, C18: C_Polarized, symbol Device:C_Polarized
- added C19, C4, C7: 10nF, symbol Device:C
- added C21, C9: 4.7pF, symbol Device:C
- added C24: 47uF, symbol Device:C
- added C5: 10pF, symbol Device:C
- added FB1: TDK MPZ201S221A, symbol Device:FerriteBead
- added J5, J6: Screw_Terminal_01x02, symbol Connector:Screw_Terminal_01x02
- added L1: 10uH, symbol Device:L
- added L2, L4: 8.2uH, symbol Device:L
- added L3: 4.7uH, symbol Device:L
- added R1: 100k, symbol Device:R
- added R10, R3, R8: 1M, symbol Device:R
- added R2, R5: 110k, symbol Device:R
- added R4, R9: 243k, symbol Device:R
- added R6: 412k, symbol Device:R
- added R7: 52.3k, Resistor_SMD:R_0805_2012Metric, symbol Device:R
- added U1, U2, U6: LT8610, Package_SO:MSOP-16-1EP_3x4.039mm_P0.5mm_EP1.651x2.845mm_ThermalVias, symbol Regulator_Switching:LT8610
- added U3, U4, U5: ~, symbol pdu:LTC1478
Connections:
- net 3V3_BUS: now also C12.2, C9.2, L2.2, R8.2, U2.14 (BIAS)
- net 3V3_BUS_STAT: now also U2.15 (PG)
- net 5V_BUS: now also C21.2, C24.2, L3.2, R10.2, U6.14 (BIAS)
- net 5V_BUS_STAT: now also U6.15 (PG)
- net GND: now also C1.1, C11.2, C12.1, C13.2, C14.2, C15.2, C16.2, C17.2, C18.2, C19.1, C20.1, C23.2, C24.1, C25.1, C26.1, C3.1, C4.1, C6.2, C7.1, C8.1, J6.2 (Pin_2), R2.2, R4.1, R5.2, R6.1, R7.2, R9.1, U1.17 (GND), U1.7 (GND), U1.8 (GND), U2.17 (GND), U2.7 (GND), U2.8 (GND), U3. (V_OUT2), U4. (V_OUT2), U5. (V_OUT2), U6.17 (GND), U6.7 (GND), U6.8 (GND)
- net V_BATT: now also C1.2, C26.2, C8.2, FB1.1, J5.1 (Pin_1), U1.4 (EN/UV), U1.5 (VIN), U1.6 (VIN), U2.4 (EN/UV), U2.5 (VIN), U2.6 (VIN)
- new net: C5.1, R3.1, R4.2, U1.16 (FB)
- new net: C6.1, U1.13 (INTVcc)
- new net: C7.2, U2.2 (TR/SS)
- new net: C22.2, L3.1, U6.10 (SW), U6.11 (SW), U6.9 (SW)
- new net: C22.1, U6.12 (BST)
- new net: C23.1, U6.13 (INTVcc)
- new net: C21.1, R10.1, R9.2, U6.16 (FB)
- new net: C19.2, U6.2 (TR/SS)
- new net: R7.1, U6.3 (RT)
- new net: C20.2, L4.2, U6.4 (EN/UV), U6.5 (VIN), U6.6 (VIN)
- new net: C9.1, R6.2, R8.1, U2.16 (FB)
- new net: C11.1, U2.13 (INTVcc)
- new net: C10.2, L2.1, U2.10 (SW), U2.11 (SW), U2.9 (SW)
- new net: C2.1, U1.12 (BST)
- new net: C2.2, L1.1, U1.10 (SW), U1.11 (SW), U1.9 (SW)
- new net: C10.1, U2.12 (BST)
- new net: C4.2, U1.2 (TR/SS)
- new net: R2.1, U1.3 (RT)
- new net: C25.2, FB1.2, L4.1
- new net: R5.1, U2.3 (RT)
- new net EDFA_5V: C13.1, C15.1, C17.1, C3.2, C5.2, L1.2, R1.1, R3.2, U1.14 (BIAS), U3. (V_OUT2), U4. (V_OUT2), U5. (V_OUT2)
- new net EDFA_5V_STAT: R1.2, U1.15 (PG)
- new net EDFA_5V_SWITCHED: C14.1, C16.1, C18.1, U3. (V_OUT2), U4. (V_OUT2), U5. (V_OUT2)
- new net EDFA_ENABLE: U3. (V_OUT2), U4. (V_OUT2), U5. (V_OUT2)
- new net GND_REF: J5.2 (Pin_2), J6.1 (Pin_1)
Other:
- note added: "3V3 Voltage Regulator"
- note added: "BeagleBoard Regulator (Low EMI)"
- note added: "EDFA Switch"
- note added: "EDFA Voltage Regulator"
- note added: "Mechanical Inhibits"
- moved on the sheet: H1, H2, H3, H4, J3, J4
