File: Avionics/PDU/Untitled/Untitled.kicad_sch (KiCad schematic)
At the start: 67 parts, among them J1 Conn_02x26_Odd_Even, J2 Conn_02x26_Odd_Even, J3 Screw_Terminal_01x02, J4 Screw_Terminal_01x02, J5 Screw_Terminal_01x02, J6 Screw_Terminal_01x02, J7 USB_C_Receptacle_USB2.0_14P, U1 LT8610, U2 LT8610, U6 LT8610

Commit message: PDU 1.0.0
Parts:
- removed C26: 4.7uF, Capacitor_SMD:C_0805_2012Metric, symbol Device:C
- removed FB1: TDK MPZ201S221A, symbol Device:FerriteBead
- added C17, C27, C29, C31, C32, C34, C36: 0.1uF, Capacitor_SMD:C_0805_2012Metric, symbol Device:C
- added C18, C26, C28, C30: 1uF, Capacitor_SMD:C_0805_2012Metric, symbol Device:C_Polarized
- added C33: 4.7uF, Capacitor_SMD:C_0805_2012Metric, symbol Device:C
- added C35, C39: 10uF, Capacitor_SMD:C_0805_2012Metric, symbol Device:C
- added C37, C38, C40, C41, C42, C43, C44, C51: 1uF, Capacitor_SMD:C_0805_2012Metric, symbol Device:C
- added C45, C46, C47, C48, C49, C50: 0.1UF, Capacitor_SMD:C_0805_2012Metric, symbol Device:C
- added D10, D11, D12, D8, D9: PMEG10020ELRX, Diode_SMD:Nexperia_CFP3_SOD-123W, symbol Device:D_Schottky
- added D13, D5, D6, D7: 150060RS75000, LED_SMD:LED_0603_1608Metric, symbol Device:LED
- added D14: 150060VS75000, LED_SMD:LED_0603_1608Metric, symbol Device:LED
- added D15: CMDSH-3TR, Diode_SMD:D_SOD-323F, symbol Device:D_Schottky
- added D16, D17: MBR230S1F, Diode_SMD:D_SOD-123F, symbol Device:D
- added J10, J16, J8, J9: Screw_Terminal_01x02, TerminalBlock:TerminalBlock_Xinya_XY308-2.54-2P_1x02_P2.54mm_Horizontal, symbol Connector:Screw_Terminal_01x02
- added J11, J12, J13, J14, J15: Conn_01x04, Connector_Molex:Molex_CLIK-Mate_502382-0470_1x04-1MP_P1.25mm_Vertical, symbol Connector_Generic:Conn_01x04
- added Q1: BC848ALT1G, Package_TO_SOT_SMD:SOT-23-3, symbol Transistor_BJT:2N3904
- added Q2, Q3: IRLML2803PBFCT, Package_TO_SOT_SMD:SOT-23-3, symbol Transistor_FET:NDT3055L
- added R19, R20, R22, R23: 10k, Resistor_SMD:R_0805_2012Metric, symbol Device:R
- added R21, R24: 4.7k, Resistor_SMD:R_0805_2012Metric, symbol Device:R
- added R25, R26: 100k, Resistor_SMD:R_0805_2012Metric, symbol Device:R
- added R27, R28, R29, R30: 150, Resistor_SMD:R_0805_2012Metric, symbol Device:R
- added R31: 3k, Resistor_SMD:R_0805_2012Metric, symbol Device:R
- added R32: 6.04k, Resistor_SMD:R_0805_2012Metric, symbol Device:R
- added R33: 26.7k, Resistor_SMD:R_0805_2012Metric, symbol Device:R
- added R34: 1, Resistor_SMD:R_0805_2012Metric, symbol Device:R
- added R35: 0, Resistor_SMD:R_0805_2012Metric, symbol Device:R
- added R36: 169k, Resistor_SMD:R_0805_2012Metric, symbol Device:R
- added R37: 28.4k, Resistor_SMD:R_0805_2012Metric, symbol Device:R
- added R38, R39: 3.01k, Resistor_SMD:R_0805_2012Metric, symbol Device:R
- added R40: 52.3k, Resistor_SMD:R_0805_2012Metric, symbol Device:R
- added R41: 5.1k, Resistor_SMD:R_0805_2012Metric, symbol Device:R
- added R42, R44, R46, R47, R48, R50, R51, R53, R54, R56, R57, R59: 10, Resistor_SMD:R_0805_2012Metric, symbol Device:R
- added R43, R45, R49, R52, R55, R58: 2m, Resistor_SMD:R_0805_2012Metric, symbol Device:R
- added TP1, TP2, TP3, TP4, TP5, TP6, TP7, TP8: ~, TestPoint:TestPoint_Loop_D2.50mm_Drill1.0mm_LowProfile, symbol Connector:TestPoint
- added U10, U11, U14, U9: ~, Package_SO:SOIC-8_3.9x4.9mm_P1.27mm, symbol pdu:LTC1478
- added U12: ~, Package_DFN_QFN:QFN-20-1EP_4x4mm_P0.5mm_EP2.5x2.5mm, symbol pdu:LTC4012IUFPBF
- added U13: ~, Package_SO:SOIC-8_3.9x4.9mm_P1.27mm, symbol pdu:SI4835BDY-T1-E3
- added U15: ~, Package_SO:SOIC-8-1EP_3.9x4.9mm_P1.27mm_EP2.29x3mm, symbol pdu:AO4818B
- added U16, U17, U18, U19, U20, U21: INA219AxD, Package_SO:SOIC-8_3.9x4.9mm_P1.27mm, symbol Sensor_Energy:INA219AxD
- added U5: ~, Package_SO:SOIC-8_3.9x4.9mm_P1.27mm, symbol pdu:SI4835DDY
- added U7, U8: ~, Package_SO:TSOP-6_1.65x3.05mm_P0.95mm, symbol pdu:SI4835DDV
- C14: value C_Polarized -> 1uF; footprint (none) -> Capacitor_SMD:C_0805_2012Metric
- C25: value 4.7uF -> 0.1uF
- H1, H2, H3, H4: symbol Mechanical:MountingHole -> Mechanical:MountingHole_Pad_MP
- L4: value 8.2uH -> AIML-0805-150K-T; footprint Inductor_SMD:L_Coilcraft_XxL4040 -> Inductor_SMD:L_0805_2012Metric
- U3: footprint (none) -> Package_SO:SOIC-8_3.9x4.9mm_P1.27mm
Connections:
- net 3V3_BUS: now also C29.1, J11.2 (Pin_2), J12.2 (Pin_2), J13.2 (Pin_2), J14.2 (Pin_2), J15.2 (Pin_2), TP2.1, U14.2 (V_IN1), U14.3 (V_INS), U14.6 (V_IN3), U14.7 (V_IN2)
- net 5V_BUS: now also C25.1, C17.1, C27.1, TP1.1, U10.2 (V_IN1), U10.3 (V_INS), U10.6 (V_IN3), U10.7 (V_IN2), U11.2 (V_IN1), U11.3 (V_INS), U11.6 (V_IN3), U11.7 (V_IN2), U9.2 (V_IN1), U9.3 (V_INS), U9.6 (V_IN3), U9.7 (V_IN2)
- net EDFA_5V: now also U3.2 (V_IN1), U3.3 (V_INS), U3.6 (V_IN3), U3.7 (V_IN2), TP3.1; no longer U3. (V_OUT2)
- net EDFA_5V_STAT: now also J2.19 (Pin_19)
- net EDFA_5V_SWITCHED: now also U3.1 (V_OUT1), U3.8 (V_OUT2), TP4.1; no longer U3. (V_OUT2)
- net EDFA_ENABLE: now also J1.11 (Pin_11), U3.4 (EN); no longer U3. (V_OUT2)
- net GND: now also C25.2, H1.MP, H2.MP, H3.MP, H4.MP, J2.31 (Pin_31), U3.5 (GND), C17.2, C18.2, C26.2, C27.2, C28.2, C29.2, C30.2, C31.1, C33.1, C35.1, C37.1, C38.1, C39.1, C45.1, C46.1, C47.1, C48.1, C49.1, C50.1, J10.2 (Pin_2), J11.4 (Pin_4), J12.4 (Pin_4), J13.4 (Pin_4), J14.4 (Pin_4), J15.4 (Pin_4), J8.2 (Pin_2), J9.2 (Pin_2), Q1.1 (E), Q2.3 (S), Q3.3 (S), R20.2, R22.2, R23.2, R27.1, R28.1, R29.1, R30.1, R32.1, R33.1, R37.2, U10.5 (GND), U11.5 (GND), U12.21 (GND), U14.5 (GND), U16.1 (A1), U16.6 (GND), U17.1 (A1), U17.6 (GND), U18.1 (A1), U18.6 (GND), U19.1 (A1), U19.6 (GND), U20.1 (A1), U20.6 (GND), U21.1 (A1), U21.6 (GND), U9.5 (GND); no longer C25.1, U3. (V_OUT2)
- net GND_REF: now also J16.2 (Pin_2)
- net V_BATT: now also C20.2, U6.4 (EN/UV), U6.5 (VIN), U6.6 (VIN), C35.2, D16.1 (K), R19.1, R34.2, R41.2, R57.1, R58.2, U15.5, U15.8, U5.1 (S1), U5.2 (S2), U5.3 (S3)
- net BATT_PRE_INH: now reaches J4.1 (Pin_1)
- net BATT_PRE_INH: now also J16.1 (Pin_1); no longer J3.2 (Pin_2)
- net SOLAR_TMP_3: now reaches J2.11 (Pin_11)
- net SOLAR_TMP_3: now also J13.3 (Pin_3)
- net EDFA_5V_SW: now reaches J2.21 (Pin_21)
- net EDFA_5V_SW: now also J2.22 (Pin_22)
- net SOLAR_TMP_1: now reaches J2.3 (Pin_3)
- net SOLAR_TMP_1: now also J11.3 (Pin_3)
- net SOLAR_TMP_2: now reaches J2.5 (Pin_5)
- net SOLAR_TMP_2: now also J12.3 (Pin_3)
- net SOLAR_TMP_5: now reaches J2.7 (Pin_7)
- net SOLAR_TMP_5: now also J15.3 (Pin_3)
- net SOLAR_TMP_4: now reaches J2.9 (Pin_9)
- net SOLAR_TMP_4: now also J14.3 (Pin_3)
- net SW: now reaches L4.1
- net SW: now also C36.1, D17.1 (K), U12.18 (SW), U15.3, U15.6, U15.7; no longer C25.2
- net KAPTON_ENABLE: now reaches J1.13 (Pin_13)
- net KAPTON_ENABLE: now also U9.4 (EN)
- net 5V_SW_1_EN: now reaches J1.15 (Pin_15)
- net 5V_SW_1_EN: now also U10.4 (EN)
- net 5V_SW_2_EN: now reaches J1.17 (Pin_17)
- net 5V_SW_2_EN: now also U11.4 (EN)
- net 5V_SW_1: now reaches J1.21 (Pin_21)
- net 5V_SW_1: now also C26.1, D6.2 (A), TP7.1, U10.1 (V_OUT1), U10.8 (V_OUT2)
- net ICL: now reaches J1.22 (Pin_22)
- net ICL: now also U12.8 (ICL)
- net 5V_SW_2: now reaches J1.23 (Pin_23)
- net 5V_SW_2: now also C28.1, D7.2 (A), TP8.1, U11.1 (V_OUT1), U11.8 (V_OUT2)
- net SHDN: now reaches J1.24 (Pin_24)
- net SHDN: now also U12.6 (SHDN)
- net PERIPH_EN: now reaches J1.27 (Pin_27)
- net PERIPH_EN: now also U14.4 (EN)
- net ENAB_BURN_1: now reaches J1.28 (Pin_28)
- net ENAB_BURN_1: now also R21.2, R22.1
- net BURN_FET: now reaches J1.29 (Pin_29)
- net BURN_FET: now also Q1.2 (B), R20.1
- net ENAB_BURN_2: now reaches J1.30 (Pin_30)
- net ENAB_BURN_2: now also R23.1, R24.2
- net PERIPH_PWR: now reaches J1.47 (Pin_47)
- net PERIPH_PWR: now also C30.1, C45.2, C46.2, C47.2, C48.2, C49.2, C50.2, D13.2 (A), TP5.1, U14.1 (V_OUT1), U14.8 (V_OUT2), U16.5 (VS), U17.5 (VS), U18.5 (VS), U19.5 (VS), U20.5 (VS), U21.5 (VS)
- net GNSS_UART_RX: no longer names the net of J1.35 (Pin_35)
- net GNSS_UART_TX: no longer names the net of J1.33 (Pin_33)
- net I2C_1_SCL renamed SCL
- net SCL: now also U16.4 (SCL), U17.4 (SCL), U18.4 (SCL), U19.4 (SCL), U20.4 (SCL), U21.4 (SCL)
- net I2C_1_SDA renamed SDA
- net SDA: now also U16.2 (A0), U16.3 (SDA), U17.2 (A0), U17.3 (SDA), U18.2 (A0), U18.3 (SDA), U19.2 (A0), U19.3 (SDA), U20.2 (A0), U20.3 (SDA), U21.2 (A0), U21.3 (SDA)
- net POWER_PRE_INH renamed SOLAR_PRE_INH
- net SOLAR_PRE_INH: now also D10.1 (K), D11.1 (K), D12.1 (K), D8.1 (K), D9.1 (K)
- net POWER_PRE_MPPT renamed BATT_CS
- net BATT_CS: now also R58.1, R59.1
- net V_CHARGE renamed VBATT_CHARGE
- net VBATT_CHARGE: now also C39.2, D16.2 (A), R39.2, R40.2, U12.11 (BAT)
- new net: C36.2, D15.1 (K), R35.2
- new net: C37.2, C38.2, D15.2 (A), U12.17 (INTVDD)
- new net: Q2.1 (G), R21.1
- new net: Q2.2 (D), R25.1, U7.3 (G)
- new net: D12.2 (A), R45.1, R46.1
- new net: D8.2 (A), R52.1, R53.1
- new net: D9.2 (A), R55.1, R56.1
- new net: L4.2, R38.2, R40.1
- new net: R25.2, R26.2, U5.5 (D1), U5.6 (D2), U5.7 (D3), U5.8 (D4), U7.4 (S1), U8.4 (S1)
- new net: D10.2 (A), R43.1, R48.1
- new net: C34.1, R34.1, U12.2 (CLP), U13.1 (S1), U13.2 (S2), U13.3 (S3)
- new net: U12.3 (INFET), U13.4 (G)
- new net: C34.2, R41.1, U12.1 (CLN)
- new net: J8.1 (Pin_1), U7.1 (D2), U7.2 (D3), U7.5 (D4), U7.6 (D1)
- new net: Q3.1 (G), R24.1
- new net: Q3.2 (D), R26.1, U8.3 (G)
- new net: C51.2, R57.2, U21.7 (IN-)
- new net: C33.2, R33.2, U12.13 (PROG)
- new net: R39.1, U12.14 (CSN)
- new net: Q1.3 (C), R19.2, U5.4 (G)
- new net: R36.2, R37.1, U12.9 (VFB)
- new net: D11.2 (A), R49.1, R50.1
- new net: R36.1, U12.10 (FBDIV)
- new net: R38.1, U12.15 (CSP)
- new net: C51.1, R59.2, U21.8 (IN+)
- new net: R35.1, U12.20 (BOOST)
- new net: D7.1 (K), R29.2
- new net: C32.1, R32.2
- new net: C32.2, U12.12 (ITH)
- new net: D14.2 (A), R31.2
- new net: D5.1 (K), R27.2
- new net: D13.1 (K), R30.2
- new net: D6.1 (K), R28.2
- new net: J9.1 (Pin_1), U8.1 (D2), U8.2 (D3), U8.5 (D4), U8.6 (D1)
- new net BGATE: U12.16 (BGATE), U15.4
- new net CHRG: D14.1 (K), U12.7 (CHRG)
- new net CS_SOL1_VIN+: C44.2, R54.2, U17.8 (IN+)
- new net CS_SOL1_VIN-: C44.1, R56.2, U17.7 (IN-)
- new net CS_SOL2_VIN+: C43.2, R51.2, U16.8 (IN+)
- new net CS_SOL2_VIN-: C43.1, R53.2, U16.7 (IN-)
- new net CS_SOL3_VIN+: C40.2, R47.2, U18.8 (IN+)
- new net CS_SOL3_VIN-: C40.1, R48.2, U18.7 (IN-)
- new net CS_SOL4_VIN+: C41.2, R44.2, U19.8 (IN+)
- new net CS_SOL4_VIN-: C41.1, R50.2, U19.7 (IN-)
- new net CS_SOL5_VIN+: C42.2, R42.2, U20.8 (IN+)
- new net CS_SOL5_VIN-: C42.1, R46.2, U20.7 (IN-)
- new net KAPTON_PWR: C18.1, D5.2 (A), J10.1 (Pin_1), TP6.1, U9.1 (V_OUT1), U9.8 (V_OUT2)
- new net S2: D17.2 (A), U15.2
- new net SOLAR_IN_1: J11.1 (Pin_1), R54.1, R55.2
- new net SOLAR_IN_2: J12.1 (Pin_1), R51.1, R52.2
- new net SOLAR_IN_3: J13.1 (Pin_1), R43.2, R47.1
- new net SOLAR_IN_4: J14.1 (Pin_1), R44.1, R49.2
- new net SOLAR_IN_5: J15.1 (Pin_1), R42.1, R45.2
- new net SOLAR_PRE_MPPT: C31.2, J3.2 (Pin_2), R31.1, U12.4 (DCIN), U13.5 (D1), U13.6 (D2), U13.7 (D3), U13.8 (D4)
- new net TGATE: U12.19 (TGATE), U15.1
- no-connect marks 4 -> 42
Other:
- note added: "5V Regulator"
- note added: "Antenna Deployment"
- note added: "Beagleboard Peripherals Switch"
- note added: "Connectors"
- note added: "Kapton Switch"
- note added: "Misc Switch 1"
- note added: "Misc Switch 2"
- note added: "Mounting Holes"
- note added: "Temp Sensor"
- note added: "USB Connector"
- note removed: "5V Regulator (Low EMI)"
- moved on the sheet: C1, C10, C11, C12, C13, C14, C15, C16, C19, C2, C20, C21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

Commit message: feat: PDU 2.0.0
Parts:
- removed C27: 0.1uF, Capacitor_SMD:C_0805_2012Metric, symbol Device:C
- removed C28: 1uF, Capacitor_SMD:C_0805_2012Metric, symbol Device:C_Polarized
- removed D7: 150060RS75000, LED_SMD:LED_0603_1608Metric, symbol Device:LED
- removed R16: 10k, Resistor_SMD:R_0805_2012Metric, symbol Device:R
- removed R29: 150, Resistor_SMD:R_0805_2012Metric, symbol Device:R
- removed TP6, TP8: ~, TestPoint:TestPoint_Loop_D2.50mm_Drill1.0mm_LowProfile, symbol Connector:TestPoint
- removed U11: ~, Package_SO:SOIC-8_3.9x4.9mm_P1.27mm, symbol pdu:LTC1478
- C1, C11, C13, C14, C15, C17, C18, C19, C20, C23, C25, C26, C29, C30, C4, C45, C46, C47, C48, C49, C50, C6, C7, C8: footprint Capacitor_SMD:C_0805_2012Metric -> Capacitor_SMD:C_0402_1005Metric
- C21: value 4.7pF -> 10pF
- R11, R12, R13, R14, R27, R28, R30: footprint Resistor_SMD:R_0805_2012Metric -> Resistor_SMD:R_0603_1608Metric
- R15: value 45.3k -> 0
- R2: value 110k -> 18.2k; footprint Resistor_SMD:R_0805_2012Metric -> Capacitor_SMD:C_0402_1005Metric
- R40: value 52.3k -> 1
- R43, R45, R49, R52, R55, R58: footprint Resistor_SMD:R_0805_2012Metric -> Resistor_SMD:R_2512_6332Metric
- R5: footprint Resistor_SMD:R_0805_2012Metric -> Capacitor_SMD:C_0402_1005Metric
- R7: value 52.3k -> 18.2k; footprint Resistor_SMD:R_0805_2012Metric -> Capacitor_SMD:C_0402_1005Metric
- TP1, TP2, TP3, TP4, TP5, TP7: footprint TestPoint:TestPoint_Loop_D2.50mm_Drill1.0mm_LowProfile -> TestPoint:TestPoint_Pad_2.0x2.0mm
- U15: footprint Package_SO:SOIC-8-1EP_3.9x4.9mm_P1.27mm_EP2.29x3mm -> Package_SO:SOIC-8_3.9x4.9mm_P1.27mm
Connections:
- net 3V3_BUS: no longer C15.2, U4.5 (SHUTDOWN), U4.8 (V_IN)
- net 5V_SW_1_EN: now also J1.31 (Pin_31); no longer J1.15 (Pin_15)
- net CHRG: now also J1.24 (Pin_24)
- net EDFA_ENABLE: now also J1.13 (Pin_13); no longer J1.11 (Pin_11)
- net KAPTON_ENABLE: now also J1.11 (Pin_11); no longer J1.13 (Pin_13)
- net PDU_TEMP: now also U4.1 (V_OUT); no longer J2.1 (Pin_1), R15.2
- net PERIPH_PWR: now also C15.2, U4.5 (SHUTDOWN), U4.8 (V_IN)
- net SHDN: now also J1.26 (Pin_26); no longer J1.24 (Pin_24)
- net SOLAR_TMP_1: now also J1.50 (Pin_50); no longer J2.3 (Pin_3)
- net SOLAR_TMP_2: now also J1.49 (Pin_49); no longer J2.5 (Pin_5)
- net SOLAR_TMP_3: now also J1.48 (Pin_48); no longer J2.11 (Pin_11)
- net SOLAR_TMP_4: now also J2.1 (Pin_1); no longer J2.9 (Pin_9)
- net SOLAR_TMP_5: now also J2.2 (Pin_2); no longer J2.7 (Pin_7)
- net FB_1: now reaches C5.1, R3.1, R4.2, U1.16 (FB)
- net at R15.1: now also R38.2, R40.1; no longer U4.1 (V_OUT)
- net SW_3: now reaches C22.2, L3.1, U6.10 (SW), U6.11 (SW), U6.9 (SW)
- net FB_3: now reaches C21.1, R10.1, R9.2, U6.16 (FB)
- net FB_2: now reaches C9.1, R6.2, R8.1, U2.16 (FB)
- net SW_2: now reaches C10.2, L2.1, U2.10 (SW), U2.11 (SW), U2.9 (SW)
- net SW_1: now reaches C2.2, L1.1, U1.10 (SW), U1.11 (SW), U1.9 (SW)
- net 5V_SW_2: no longer names the net of J1.23 (Pin_23)
- net 5V_SW_2_EN: no longer names the net of J1.17 (Pin_17)
- new net: L4.2, R15.2
- no-connect marks 42 -> 37
Other:
- note removed: "Misc Switch 2"
