File: Avionics/PDU/Untitled/Untitled.kicad_pcb (KiCad board)
At the start: 4 copper layers, 90.2 x 95.9 mm, 4 parts

Commit message: feat: pdu updates
Parts:
- added R7: 52.3k, Resistor_SMD:R_0805_2012Metric, F.Cu at (112.1, 69.0)
- added U1: LT8610, Package_SO:MSOP-16-1EP_3x4.039mm_P0.5mm_EP1.651x2.845mm_ThermalVias, F.Cu at (132.1, 70.7)
- added U2: LT8610, Package_SO:MSOP-16-1EP_3x4.039mm_P0.5mm_EP1.651x2.845mm_ThermalVias, F.Cu at (132.9, 84.0)
- added U6: LT8610, Package_SO:MSOP-16-1EP_3x4.039mm_P0.5mm_EP1.651x2.845mm_ThermalVias, F.Cu at (132.6, 96.5)

Commit message: feat: pdu updates (inc. pci104)
Parts:
- added C1: 4.7uF, Capacitor_SMD:C_0805_2012Metric, F.Cu at (90.0, 80.6)
- added C10: 0.1uF, Capacitor_SMD:C_0805_2012Metric, F.Cu at (150.7, 93.4)
- added C11: 1uF, Capacitor_SMD:C_0805_2012Metric, F.Cu at (150.7, 96.4)
- added C12: 68uF, Capacitor_SMD:C_0805_2012Metric, F.Cu at (150.7, 99.5)
- added C13: 0.1uF, Capacitor_SMD:C_0805_2012Metric, F.Cu at (94.0, 128.5)
- added C15: 0.1uF, Capacitor_SMD:C_0805_2012Metric, F.Cu at (95.7, 140.3)
- added C16: 4.7uF, Capacitor_SMD:C_0805_2012Metric, F.Cu at (84.0, 115.5)
- added C19: 10nF, Capacitor_SMD:C_0805_2012Metric, F.Cu at (116.4, 117.3)
- added C2: 0.1uF, Capacitor_SMD:C_0805_2012Metric, F.Cu at (101.4, 78.7)
- added C20: 4.7uF, Capacitor_SMD:C_0805_2012Metric, F.Cu at (120.9, 99.2)
- added C21: 4.7pF, Capacitor_SMD:C_0805_2012Metric, F.Cu at (120.9, 102.2)
- added C22: 0.1uF, Capacitor_SMD:C_0805_2012Metric, F.Cu at (120.9, 105.2)
- added C23: 1uF, Capacitor_SMD:C_0805_2012Metric, F.Cu at (120.9, 108.3)
- added C24: 47uF, Capacitor_SMD:C_0805_2012Metric, F.Cu at (120.9, 111.3)
- added C25: 4.7uF, Capacitor_SMD:C_0805_2012Metric, F.Cu at (120.9, 114.3)
- added C26: 4.7uF, Capacitor_SMD:C_0805_2012Metric, F.Cu at (120.9, 117.3)
- added C3: 68uF, Capacitor_SMD:C_0805_2012Metric, F.Cu at (96.5, 82.5)
- added C4: 10nF, Capacitor_SMD:C_0805_2012Metric, F.Cu at (89.0, 73.9)
- added C5: 10pF, Capacitor_SMD:C_0805_2012Metric, F.Cu at (104.9, 78.7)
- added C6: 1uF, Capacitor_SMD:C_0805_2012Metric, F.Cu at (101.4, 75.3)
- added C7: 10nF, Capacitor_SMD:C_0805_2012Metric, F.Cu at (146.3, 105.5)
- added C8: 4.7uF, Capacitor_SMD:C_0805_2012Metric, F.Cu at (150.7, 87.4)
- added C9: 4.7pF, Capacitor_SMD:C_0805_2012Metric, F.Cu at (150.7, 90.4)
- added D1: 150060VS75000, LED_SMD:LED_0603_1608Metric, F.Cu at (126.9, 124.0)
- added D2: 150060VS75000, LED_SMD:LED_0603_1608Metric, F.Cu at (96.7, 85.7)
- added D3: 150060VS75000, LED_SMD:LED_0603_1608Metric, F.Cu at (150.7, 103.6)
- added D4: 150060RS75000, LED_SMD:LED_0603_1608Metric, F.Cu at (99.3, 128.0)
- added G***: LOGO, LOGO, F.Cu at (141.5, 138.5)
- added J1: Conn_02x26_Odd_Even, Connector_PinHeader_2.54mm:PinHeader_2x26_P2.54mm_Vertical, F.Cu at (84.0, 62.9)
- added J2: Conn_02x26_Odd_Even, Connector_PinHeader_2.54mm:PinHeader_2x26_P2.54mm_Vertical, F.Cu at (84.0, 57.6)
- added J3: Screw_Terminal_01x02, TerminalBlock:TerminalBlock_Xinya_XY308-2.54-2P_1x02_P2.54mm_Horizontal, F.Cu at (74.5, 68.0)
- added J4: Screw_Terminal_01x02, TerminalBlock:TerminalBlock_Xinya_XY308-2.54-2P_1x02_P2.54mm_Horizontal, F.Cu at (74.5, 75.0)
- added J5: Screw_Terminal_01x02, TerminalBlock:TerminalBlock_Xinya_XY308-2.54-2P_1x02_P2.54mm_Horizontal, F.Cu at (74.5, 91.7)
- added J6: Screw_Terminal_01x02, TerminalBlock:TerminalBlock_Xinya_XY308-2.54-2P_1x02_P2.54mm_Horizontal, F.Cu at (74.5, 82.0)
- added J7: USB_C_Receptacle_USB2.0_14P, Connector_USB:USB_C_Receptacle_GCT_USB4105-xx-A_16P_TopMnt_Horizontal, F.Cu at (73.6, 111.7)
- added L1: 10uH, Inductor_SMD:L_Coilcraft_XxL4040, F.Cu at (100.8, 82.6)
- added L2: 8.2uH, Inductor_SMD:L_Coilcraft_XxL4040, F.Cu at (153.8, 98.6)
- added L3: 4.7uH, Inductor_SMD:L_Coilcraft_XxL4040, F.Cu at (127.0, 117.0)
- added L4: 8.2uH, Inductor_SMD:L_Coilcraft_XxL4040, F.Cu at (134.0, 117.0)
- added R1: 100k, Resistor_SMD:R_0805_2012Metric, F.Cu at (101.3, 71.9)
- added R10: 1M, Resistor_SMD:R_0805_2012Metric, F.Cu at (132.8, 108.5)
- added R11: 150, Resistor_SMD:R_0805_2012Metric, F.Cu at (132.8, 111.5)
- added R12: 150, Resistor_SMD:R_0805_2012Metric, F.Cu at (93.3, 85.6)
- added R13: 65, Resistor_SMD:R_0805_2012Metric, F.Cu at (143.6, 90.6)
- added R14: 150, Resistor_SMD:R_0805_2012Metric, F.Cu at (99.4, 124.0)
- added R15: 45.3k, Resistor_SMD:R_0805_2012Metric, F.Cu at (83.4, 138.6)
- added R16: 10k, Resistor_SMD:R_0805_2012Metric, F.Cu at (83.4, 141.9)
- added R17: 5.1k, Resistor_SMD:R_0805_2012Metric, F.Cu at (84.0, 112.0)
- added R18: 5.1k, Resistor_SMD:R_0805_2012Metric, F.Cu at (84.0, 108.5)
- added R2: 110k, Resistor_SMD:R_0805_2012Metric, F.Cu at (89.0, 77.3)
- added R3: 1M, Resistor_SMD:R_0805_2012Metric, F.Cu at (104.9, 71.9)
- added R4: 243k, Resistor_SMD:R_0805_2012Metric, F.Cu at (97.0, 72.1)
- added R5: 110k, Resistor_SMD:R_0805_2012Metric, F.Cu at (140.5, 100.4)
- added R6: 412k, Resistor_SMD:R_0805_2012Metric, F.Cu at (140.4, 95.1)
- added R8: 1M, Resistor_SMD:R_0805_2012Metric, F.Cu at (145.9, 103.6)
- added R9: 243k, Resistor_SMD:R_0805_2012Metric, F.Cu at (121.7, 107.0)
- added U4: ~, Package_SO:SOIC-8-1EP_3.9x4.9mm_P1.27mm_EP2.41x3.3mm, F.Cu at (89.9, 140.2)
- moved R7 44.0 mm to (121.6, 112.0)
- moved U1 37.6 mm to (95.1, 77.8)
- moved U2 18.2 mm to (146.3, 96.4)
- moved U6 14.2 mm to (127.3, 109.8)
Routing:
- net GND: track 0.00 -> 35.0 mm, vias 0 -> 3
- net GND_REF: track 0.00 -> 26.4 mm
- net /EDFA_5V: track 0.00 -> 21.5 mm
- net Net-(U1-FB): track 0.00 -> 20.5 mm
- net Net-(C2-Pad2): track 0.00 -> 8.63 mm
- net /3V3_BUS: track 0.00 -> 8.17 mm
- net Net-(J7-CC1): track 0.00 -> 6.66 mm
- net Net-(J7-CC2): track 0.00 -> 6.45 mm
- net /EDFA_5V_STAT: track 0.00 -> 6.42 mm
- net /V_USB: track 0.00 -> 6.37 mm
- net V_BATT: track 0.00 -> 6.22 mm, vias 0 -> 1
- net Net-(U1-TR/SS): track 0.00 -> 4.52 mm
- net Net-(U1-INTVcc): track 0.00 -> 4.08 mm
- net Net-(U1-BST): track 0.00 -> 3.50 mm
- net Net-(U4-V_OUT): track 0.00 -> 3.25 mm
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- added copper zone on F.Cu, net GND
- added copper zone on In1.Cu, net GND
- added copper zone on In2.Cu, net V_BATT
Other:
- board text added: "PULSE-A"
- board text added: "batt power"
- board text added: "edfa regulator"
- board text added: "inhibits"
- board text added: "pdu temp"
- board text added: "power distribution unit"
- board text added: "rev. 1, mm.dd.yy"
- board text added: "usb charge"

Commit message: PDU 1.0.0
Parts:
- added C14: 1uF, Capacitor_SMD:C_0805_2012Metric, F.Cu at (124.3, 103.5)
- added C17: 0.1uF, Capacitor_SMD:C_0805_2012Metric, F.Cu at (138.6, 127.8)
- added C18: 1uF, Capacitor_SMD:C_0805_2012Metric, F.Cu at (147.4, 124.0)
- added C27: 0.1uF, Capacitor_SMD:C_0805_2012Metric, F.Cu at (90.0, 103.5)
- added C28: 1uF, Capacitor_SMD:C_0805_2012Metric, F.Cu at (103.7, 103.8)
- added C29: 0.1uF, Capacitor_SMD:C_0805_2012Metric, F.Cu at (90.0, 119.0)
- added C30: 1uF, Capacitor_SMD:C_0805_2012Metric, F.Cu at (104.0, 119.0)
- added C31: 0.1uF, Capacitor_SMD:C_0805_2012Metric, B.Cu at (110.5, 111.0)
- added C32: 0.1uF, Capacitor_SMD:C_0805_2012Metric, B.Cu at (98.0, 108.5)
- added C33: 4.7uF, Capacitor_SMD:C_0805_2012Metric, B.Cu at (92.0, 109.3)
- added C34: 0.1uF, Capacitor_SMD:C_0805_2012Metric, B.Cu at (107.4, 97.6)
- added C35: 10uF, Capacitor_SMD:C_0805_2012Metric, B.Cu at (117.7, 94.0)
- added C36: 0.1uF, Capacitor_SMD:C_0805_2012Metric, B.Cu at (96.6, 96.7)
- added C37: 1uF, Capacitor_SMD:C_0805_2012Metric, B.Cu at (91.0, 86.5)
- added C38: 1uF, Capacitor_SMD:C_0805_2012Metric, B.Cu at (87.5, 86.5)
- added C39: 10uF, Capacitor_SMD:C_0805_2012Metric, B.Cu at (99.1, 114.5)
- added C40: 1uF, Capacitor_SMD:C_0805_2012Metric, F.Cu at (140.5, 97.5)
- added C41: 1uF, Capacitor_SMD:C_0805_2012Metric, F.Cu at (120.3, 109.7)
- added C42: 1uF, Capacitor_SMD:C_0805_2012Metric, F.Cu at (132.0, 89.3)
- added C43: 1uF, Capacitor_SMD:C_0805_2012Metric, F.Cu at (100.0, 129.1)
- added C44: 1uF, Capacitor_SMD:C_0805_2012Metric, F.Cu at (80.9, 124.4)
- added C45: 0.1UF, Capacitor_SMD:C_0805_2012Metric, F.Cu at (100.1, 134.0)
- added C46: 0.1UF, Capacitor_SMD:C_0805_2012Metric, F.Cu at (80.9, 129.4)
- added C47: 0.1UF, Capacitor_SMD:C_0805_2012Metric, F.Cu at (140.5, 102.4)
- added C48: 0.1UF, Capacitor_SMD:C_0805_2012Metric, F.Cu at (120.3, 115.1)
- added C49: 0.1UF, Capacitor_SMD:C_0805_2012Metric, F.Cu at (132.0, 94.5)
- added C50: 0.1UF, Capacitor_SMD:C_0805_2012Metric, F.Cu at (89.9, 92.5)
- added C51: 1uF, Capacitor_SMD:C_0805_2012Metric, F.Cu at (89.9, 97.5)
- added D10: PMEG10020ELRX, Diode_SMD:Nexperia_CFP3_SOD-123W, F.Cu at (130.5, 120.5)
- added D11: PMEG10020ELRX, Diode_SMD:Nexperia_CFP3_SOD-123W, F.Cu at (125.5, 120.5)
- added D12: PMEG10020ELRX, Diode_SMD:Nexperia_CFP3_SOD-123W, F.Cu at (128.0, 120.5)
- added D13: 150060RS75000, LED_SMD:LED_0603_1608Metric, F.Cu at (101.0, 117.0)
- added D14: 150060VS75000, LED_SMD:LED_0603_1608Metric, B.Cu at (106.3, 107.1)
- added D15: CMDSH-3TR, Diode_SMD:D_SOD-323F, B.Cu at (96.2, 86.4)
- added D16: MBR230S1F, Diode_SMD:D_SOD-123F, B.Cu at (86.5, 109.0)
- added D17: MBR230S1F, Diode_SMD:D_SOD-123F, B.Cu at (109.0, 87.4)
- added D5: 150060RS75000, LED_SMD:LED_0603_1608Metric, F.Cu at (153.7, 131.5)
- added D6: 150060RS75000, LED_SMD:LED_0603_1608Metric, F.Cu at (100.5, 109.3)
- added D7: 150060RS75000, LED_SMD:LED_0603_1608Metric, F.Cu at (100.4, 101.4)
- added D8: PMEG10020ELRX, Diode_SMD:Nexperia_CFP3_SOD-123W, F.Cu at (123.0, 120.5)
- added D9: PMEG10020ELRX, Diode_SMD:Nexperia_CFP3_SOD-123W, F.Cu at (120.5, 120.5)
- added J10: Screw_Terminal_01x02, TerminalBlock:TerminalBlock_Xinya_XY308-2.54-2P_1x02_P2.54mm_Horizontal, F.Cu at (156.0, 127.0)
- added J11: Conn_01x04, Connector_Molex:Molex_CLIK-Mate_502382-0470_1x04-1MP_P1.25mm_Vertical, B.Cu at (76.0, 126.0)
- added J12: Conn_01x04, Connector_Molex:Molex_CLIK-Mate_502382-0470_1x04-1MP_P1.25mm_Vertical, B.Cu at (109.0, 140.0)
- added J13: Conn_01x04, Connector_Molex:Molex_CLIK-Mate_502382-0470_1x04-1MP_P1.25mm_Vertical, B.Cu at (154.0, 76.5)
- added J14: Conn_01x04, Connector_Molex:Molex_CLIK-Mate_502382-0470_1x04-1MP_P1.25mm_Vertical, B.Cu at (154.0, 86.5)
- added J15: Conn_01x04, Connector_Molex:Molex_CLIK-Mate_502382-0470_1x04-1MP_P1.25mm_Vertical, B.Cu at (154.0, 96.5)
- added J16: Screw_Terminal_01x02, TerminalBlock:TerminalBlock_Xinya_XY308-2.54-2P_1x02_P2.54mm_Horizontal, F.Cu at (74.5, 91.5)
- added J8: Screw_Terminal_01x02, TerminalBlock:TerminalBlock_Xinya_XY308-2.54-2P_1x02_P2.54mm_Horizontal, F.Cu at (155.8, 115.3)
- added J9: Screw_Terminal_01x02, TerminalBlock:TerminalBlock_Xinya_XY308-2.54-2P_1x02_P2.54mm_Horizontal, F.Cu at (155.8, 108.5)
- added Q1: BC848ALT1G, Package_TO_SOT_SMD:SOT-23-3, B.Cu at (122.8, 109.0)
- added Q2: IRLML2803PBFCT, Package_TO_SOT_SMD:SOT-23-3, B.Cu at (143.0, 113.5)
- added Q3: IRLML2803PBFCT, Package_TO_SOT_SMD:SOT-23-3, B.Cu at (143.0, 105.0)
- added R19: 10k, Resistor_SMD:R_0805_2012Metric, B.Cu at (122.8, 113.2)
- added R20: 10k, Resistor_SMD:R_0805_2012Metric, B.Cu at (126.0, 109.0)
- added R21: 4.7k, Resistor_SMD:R_0805_2012Metric, B.Cu at (142.9, 109.3)
- added R22: 10k, Resistor_SMD:R_0805_2012Metric, B.Cu at (139.5, 111.9)
- added R23: 10k, Resistor_SMD:R_0805_2012Metric, B.Cu at (139.5, 103.5)
- added R24: 4.7k, Resistor_SMD:R_0805_2012Metric, B.Cu at (143.0, 100.7)
- added R25: 100k, Resistor_SMD:R_0805_2012Metric, B.Cu at (148.4, 117.7)
- added R26: 100k, Resistor_SMD:R_0805_2012Metric, B.Cu at (148.4, 109.3)
- added R27: 150, Resistor_SMD:R_0805_2012Metric, F.Cu at (157.2, 131.7)
- added R28: 150, Resistor_SMD:R_0805_2012Metric, F.Cu at (100.6, 112.7)
- added R29: 150, Resistor_SMD:R_0805_2012Metric, F.Cu at (100.7, 104.7)
- added R30: 150, Resistor_SMD:R_0805_2012Metric, F.Cu at (101.0, 120.5)
- added R31: 3k, Resistor_SMD:R_0805_2012Metric, B.Cu at (110.5, 107.1)
- added R32: 6.04k, Resistor_SMD:R_0805_2012Metric, B.Cu at (92.1, 112.7)
- added R33: 26.7k, Resistor_SMD:R_0805_2012Metric, B.Cu at (92.0, 116.0)
- added R34: 1, Resistor_SMD:R_0805_2012Metric, B.Cu at (107.4, 94.0)
- added R35: 0, Resistor_SMD:R_0805_2012Metric, B.Cu at (95.3, 92.0)
- added R36: 169k, Resistor_SMD:R_0805_2012Metric, B.Cu at (102.9, 114.5)
- added R37: 28.4k, Resistor_SMD:R_0805_2012Metric, B.Cu at (106.6, 114.5)
- added R38: 3.01k, Resistor_SMD:R_0805_2012Metric, B.Cu at (93.3, 104.5)
- added R39: 3.01k, Resistor_SMD:R_0805_2012Metric, B.Cu at (85.5, 104.5)
- added R40: 52.3k, Resistor_SMD:R_0805_2012Metric, B.Cu at (89.4, 104.5)
- added R41: 5.1k, Resistor_SMD:R_0805_2012Metric, B.Cu at (113.1, 94.0)
- added R42: 10, Resistor_SMD:R_0805_2012Metric, F.Cu at (136.4, 89.0)
- added R43: 2m, Resistor_SMD:R_0805_2012Metric, F.Cu at (149.0, 98.7)
- added R44: 10, Resistor_SMD:R_0805_2012Metric, F.Cu at (124.4, 109.3)
- added R45: 2m, Resistor_SMD:R_0805_2012Metric, F.Cu at (140.5, 90.9)
- added R46: 10, Resistor_SMD:R_0805_2012Metric, F.Cu at (136.4, 92.3)
- added R47: 10, Resistor_SMD:R_0805_2012Metric, F.Cu at (144.5, 97.1)
- added R48: 10, Resistor_SMD:R_0805_2012Metric, F.Cu at (144.5, 100.2)
- added R49: 2m, Resistor_SMD:R_0805_2012Metric, F.Cu at (128.8, 111.0)
- added R50: 10, Resistor_SMD:R_0805_2012Metric, F.Cu at (124.5, 112.7)
- added R51: 10, Resistor_SMD:R_0805_2012Metric, F.Cu at (104.7, 128.5)
- added R52: 2m, Resistor_SMD:R_0805_2012Metric, F.Cu at (109.9, 132.5)
- added R53: 10, Resistor_SMD:R_0805_2012Metric, F.Cu at (104.7, 131.7)
- added R54: 10, Resistor_SMD:R_0805_2012Metric, F.Cu at (85.5, 123.7)
- added R55: 2m, Resistor_SMD:R_0805_2012Metric, F.Cu at (89.5, 125.5)
- added R56: 10, Resistor_SMD:R_0805_2012Metric, F.Cu at (85.5, 127.0)
- added R57: 10, Resistor_SMD:R_0805_2012Metric, F.Cu at (85.7, 95.9)
- added R58: 2m, Resistor_SMD:R_0805_2012Metric, F.Cu at (83.0, 87.5)
- added R59: 10, Resistor_SMD:R_0805_2012Metric, F.Cu at (85.7, 99.0)
- added TP1: ~, TestPoint:TestPoint_Loop_D2.50mm_Drill1.0mm_LowProfile, F.Cu at (107.0, 66.6)
- added TP2: ~, TestPoint:TestPoint_Loop_D2.50mm_Drill1.0mm_LowProfile, F.Cu at (95.5, 124.5)
- added TP3: ~, TestPoint:TestPoint_Loop_D2.50mm_Drill1.0mm_LowProfile, F.Cu at (111.5, 66.6)
- added TP4: ~, TestPoint:TestPoint_Loop_D2.50mm_Drill1.0mm_LowProfile, F.Cu at (127.0, 98.0)
- added TP5: ~, TestPoint:TestPoint_Loop_D2.50mm_Drill1.0mm_LowProfile, F.Cu at (142.5, 66.6)
- added TP6: ~, TestPoint:TestPoint_Loop_D2.50mm_Drill1.0mm_LowProfile, F.Cu at (138.0, 123.5)
- added TP7: ~, TestPoint:TestPoint_Loop_D2.50mm_Drill1.0mm_LowProfile, F.Cu at (94.0, 66.6)
- added TP8: ~, TestPoint:TestPoint_Loop_D2.50mm_Drill1.0mm_LowProfile, F.Cu at (102.0, 66.6)
- added U10: ~, Package_SO:SOIC-8_3.9x4.9mm_P1.27mm, F.Cu at (95.0, 111.1)
- added U11: ~, Package_SO:SOIC-8_3.9x4.9mm_P1.27mm, F.Cu at (94.9, 103.2)
- added U12: ~, Package_DFN_QFN:QFN-20-1EP_4x4mm_P0.5mm_EP2.5x2.5mm, B.Cu at (102.1, 101.5)
- added U13: ~, Package_SO:SOIC-8_3.9x4.9mm_P1.27mm, B.Cu at (115.5, 101.0)
- added U14: ~, Package_SO:SOIC-8_3.9x4.9mm_P1.27mm, F.Cu at (95.0, 119.0)
- added U15: ~, Package_SO:SOIC-8-1EP_3.9x4.9mm_P1.27mm_EP2.29x3mm, B.Cu at (103.6, 86.5)
- added U16: INA219AxD, Package_SO:SOIC-8_3.9x4.9mm_P1.27mm, F.Cu at (95.0, 132.5)
- added U17: INA219AxD, Package_SO:SOIC-8_3.9x4.9mm_P1.27mm, F.Cu at (76.0, 128.0)
- added U18: INA219AxD, Package_SO:SOIC-8_3.9x4.9mm_P1.27mm, F.Cu at (135.5, 101.0)
- added U19: INA219AxD, Package_SO:SOIC-8_3.9x4.9mm_P1.27mm, F.Cu at (115.3, 113.7)
- added U20: INA219AxD, Package_SO:SOIC-8_3.9x4.9mm_P1.27mm, F.Cu at (127.0, 93.3)
- added U21: INA219AxD, Package_SO:SOIC-8_3.9x4.9mm_P1.27mm, F.Cu at (94.9, 95.0)
- added U3: ~, Package_SO:SOIC-8_3.9x4.9mm_P1.27mm, F.Cu at (115.3, 103.4)
- added U5: ~, Package_SO:SOIC-8_3.9x4.9mm_P1.27mm, B.Cu at (132.5, 110.1)
- added U7: ~, Package_SO:TSOP-6_1.65x3.05mm_P0.95mm, B.Cu at (148.4, 113.5)
- added U8: ~, Package_SO:TSOP-6_1.65x3.05mm_P0.95mm, B.Cu at (148.4, 105.0)
- added U9: ~, Package_SO:SOIC-8_3.9x4.9mm_P1.27mm, F.Cu at (144.5, 128.4)
- C25: value 4.7uF -> 0.1uF
- C26: value 4.7uF -> 1uF
- L4: value 8.2uH -> AIML-0805-150K-T; footprint Inductor_SMD:L_Coilcraft_XxL4040 -> Inductor_SMD:L_0805_2012Metric; moved to B.Cu
- moved C19 49.2 mm to (138.9, 73.5)
- moved C7 45.0 mm to (114.5, 73.6)
- moved C23 44.7 mm to (150.4, 74.7)
- moved R9 42.8 mm to (146.6, 72.3), turned to -90 degrees
- moved R10 42.7 mm to (154.0, 71.5)
- moved D1 42.6 mm to (146.6, 86.2)
- moved L4 41.9 mm to (95.5, 100.5), turned to 180 degrees
- moved L3 41.6 mm to (150.8, 82.8), turned to -90 degrees
- moved C21 41.0 mm to (154.1, 78.2)
- moved C22 40.0 mm to (150.4, 78.2)
- moved R7 38.1 mm to (138.9, 78.0), turned to 180 degrees
- moved C24 38.1 mm to (146.4, 83.0)
- moved U6 36.2 mm to (144.4, 77.9)
- moved C8 35.8 mm to (115.5, 81.1), turned to 90 degrees
- moved R8 35.7 mm to (130.1, 71.6)
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Connections:
- C20 pad 2: Net-(U6-EN/UV) -> V_BATT
- C25 pad 1: GND -> /5V_BUS
- C25 pad 2: Net-(C25-Pad2) -> GND
- C26 pad 1: GND -> /5V_SW_1
- C26 pad 2: V_BATT -> GND
- J1 pad 11: unconnected-(J1-Pin_11-Pad11) -> /EDFA_ENABLE
- J1 pad 13: unconnected-(J1-Pin_13-Pad13) -> /KAPTON_ENABLE
- J1 pad 15: unconnected-(J1-Pin_15-Pad15) -> /5V_SW_1_EN
- J1 pad 17: unconnected-(J1-Pin_17-Pad17) -> /5V_SW_2_EN
- J1 pad 21: unconnected-(J1-Pin_21-Pad21) -> /5V_SW_1
- J1 pad 22: unconnected-(J1-Pin_22-Pad22) -> /ICL
- J1 pad 23: unconnected-(J1-Pin_23-Pad23) -> /5V_SW_2
- J1 pad 24: unconnected-(J1-Pin_24-Pad24) -> /SHDN
- J1 pad 27: unconnected-(J1-Pin_27-Pad27) -> /PERIPH_EN
- J1 pad 28: unconnected-(J1-Pin_28-Pad28) -> /ENAB_BURN_1
- J1 pad 29: unconnected-(J1-Pin_29-Pad29) -> /BURN_FET
- J1 pad 30: unconnected-(J1-Pin_30-Pad30) -> /ENAB_BURN_2
- J1 pad 33: /GNSS_UART_TX -> unconnected-(J1-Pin_33-Pad33)
- J1 pad 35: /GNSS_UART_RX -> unconnected-(J1-Pin_35-Pad35)
- J1 pad 41: /I2C_1_SDA -> /SDA
- J1 pad 43: /I2C_1_SCL -> /SCL
- J1 pad 47: unconnected-(J1-Pin_47-Pad47) -> /PERIPH_PWR
- J2 pad 11: unconnected-(J2-Pin_11-Pad11) -> /SOLAR_TMP_3
- J2 pad 19: unconnected-(J2-Pin_19-Pad19) -> /EDFA_5V_STAT
- J2 pad 21: unconnected-(J2-Pin_21-Pad21) -> /EDFA_5V_SW
- J2 pad 22: unconnected-(J2-Pin_22-Pad22) -> /EDFA_5V_SW
- J2 pad 3: unconnected-(J2-Pin_3-Pad3) -> /SOLAR_TMP_1
- J2 pad 31: unconnected-(J2-Pin_31-Pad31) -> GND
- J2 pad 5: unconnected-(J2-Pin_5-Pad5) -> /SOLAR_TMP_2
- J2 pad 7: unconnected-(J2-Pin_7-Pad7) -> /SOLAR_TMP_5
- J2 pad 9: unconnected-(J2-Pin_9-Pad9) -> /SOLAR_TMP_4
- J3 pad 1: /POWER_PRE_INH -> /SOLAR_PRE_INH
- J3 pad 2: Net-(J3-Pin_2) -> /SOLAR_PRE_MPPT
- J4 pad 1: Net-(J3-Pin_2) -> /BATT_PRE_INH
- J4 pad 2: /POWER_PRE_MPPT -> /BATT_CS
- J5 pad 1: /V_CHARGE -> /VBATT_CHARGE
- L4 pad 1: Net-(C25-Pad2) -> /SW
- L4 pad 2: Net-(U6-EN/UV) -> Net-(L4-Pad2)
- U6 pad 4: Net-(U6-EN/UV) -> V_BATT
- U6 pad 5: Net-(U6-EN/UV) -> V_BATT
- U6 pad 6: Net-(U6-EN/UV) -> V_BATT
Routing:
- net /3V3_BUS: track 8.17 -> 295.7 mm, vias 0 -> 4
- net /5V_BUS: track 0.00 -> 257.7 mm, vias 0 -> 5
- net /PERIPH_PWR: track 0.00 -> 182.5 mm, vias 0 -> 9
- net GND: track 35.0 -> 213.1 mm, vias 3 -> 42
- net /SDA: track 0.00 -> 162.3 mm, vias 0 -> 9
- net /SCL: track 0.00 -> 159.6 mm, vias 0 -> 6
- net /SOLAR_PRE_INH: track 0.00 -> 109.6 mm, vias 0 -> 1
- net /SOLAR_TMP_2: track 0.00 -> 100.5 mm
- net /PDU_TEMP: track 0.00 -> 98.4 mm
- net /KAPTON_ENABLE: track 0.00 -> 89.4 mm, vias 0 -> 1
- net /SOLAR_PRE_MPPT: track 0.00 -> 87.7 mm, vias 0 -> 1
- net /SOLAR_TMP_5: track 0.00 -> 79.0 mm
- net /5V_SW_1: track 0.00 -> 74.6 mm, vias 0 -> 2
- net /SOLAR_TMP_1: track 0.00 -> 73.7 mm
- net /SOLAR_TMP_4: track 0.00 -> 72.2 mm
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Other:
- board text added: "3v3 reg stat"
- board text added: "5v reg stat"
- board text added: "antenna deployment"
- board text added: "batt connectors"
- board text added: "batt heat"
- board text added: "batt heat stat"
- board text added: "edfa reg stat"
- board text added: "edfa switch stat"
- board text added: "periph switch stat"
- board text added: "rev. 1.0.0, 09.23.24"
- board text added: "switch 1 stat"
- board text added: "switch 2 stat"
- board text added: "usb continuity"
- board text removed: "batt power"
- board text removed: "edfa regulator"
- board text removed: "pdu temp"
- board text removed: "rev. 1, mm.dd.yy"
- board text removed: "usb charge"

Commit message: feat: PDU 2.0.0
Parts:
- removed C27: 0.1uF, Capacitor_SMD:C_0805_2012Metric
- removed C28: 1uF, Capacitor_SMD:C_0805_2012Metric
- removed D7: 150060RS75000, LED_SMD:LED_0603_1608Metric
- removed R16: 10k, Resistor_SMD:R_0805_2012Metric
- removed R29: 150, Resistor_SMD:R_0805_2012Metric
- removed TP6, TP8: ~, TestPoint:TestPoint_Loop_D2.50mm_Drill1.0mm_LowProfile
- removed U11: ~, Package_SO:SOIC-8_3.9x4.9mm_P1.27mm
- C1, C11, C19, C20, C23, C4, C6, C7, C8: footprint Capacitor_SMD:C_0805_2012Metric -> Capacitor_SMD:C_0402_1005Metric; moved to B.Cu
- C10, C12, C2, C21, C22, C24, C3, C5, C9, L1, L2, L3, R1, R10, R3, R4, R6, R8, R9, U1, U2, U6: moved to B.Cu
- C13, C14, C15, C17, C18, C25, C26, C29, C30, C45, C46, C47, C48, C49, C50: footprint Capacitor_SMD:C_0805_2012Metric -> Capacitor_SMD:C_0402_1005Metric
- C31, C32, C33, C34, C35, C36, C37, C38, C39, D14, D15, D16, D17, J11, J12, J13, J14, J15, L4, R31, R32, R33, R34, R35, R36, R37, R38, R39, R41, U12, U13: moved to F.Cu
- R11, R12, R13, R14, R27, R28, R30: footprint Resistor_SMD:R_0805_2012Metric -> Resistor_SMD:R_0603_1608Metric
- R15: value 45.3k -> 0
- R2, R5, R7: footprint Resistor_SMD:R_0805_2012Metric -> Capacitor_SMD:C_0402_1005Metric; moved to B.Cu
- R40: value 52.3k -> 1; moved to F.Cu
- R43, R45, R49, R52, R55, R58: footprint Resistor_SMD:R_0805_2012Metric -> Resistor_SMD:R_2512_6332Metric
- TP1, TP2, TP3, TP4, TP5, TP7: footprint TestPoint:TestPoint_Loop_D2.50mm_Drill1.0mm_LowProfile -> TestPoint:TestPoint_Pad_2.0x2.0mm
- U15: footprint Package_SO:SOIC-8-1EP_3.9x4.9mm_P1.27mm_EP2.29x3mm -> Package_SO:SOIC-8_3.9x4.9mm_P1.27mm; moved to F.Cu
- moved J11 85.4 mm to (154.5, 92.3)
- moved J12 81.7 mm to (154.5, 72.1), turned to -90 degrees
- moved J14 79.6 mm to (75.3, 74.9)
- moved J15 79.6 mm to (75.3, 84.9)
- moved C45 73.0 mm to (138.3, 71.8), turned to 0 degrees
- moved R52 71.3 mm to (147.4, 71.9), turned to 90 degrees
- moved C43 70.4 mm to (141.0, 71.8)
- moved U16 70.3 mm to (137.1, 76.1), turned to 90 degrees
- moved R51 70.3 mm to (143.8, 70.1)
- moved R53 70.2 mm to (143.7, 73.4)
- moved R10 69.5 mm to (120.5, 132.4), turned to 180 degrees
- moved U17 68.7 mm to (137.0, 96.4), turned to 90 degrees
- moved C46 68.5 mm to (138.3, 92.1), turned to 0 degrees
- moved R8 68.2 mm to (99.9, 132.8), turned to 180 degrees
- moved C44 68.0 mm to (140.8, 92.3)
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Connections:
- net Net-(C10-Pad2) renamed /SW_2
- net Net-(C2-Pad2) renamed /SW_1
- net Net-(C22-Pad2) renamed /SW_3
- net Net-(U1-FB) renamed /FB_1
- net Net-(U2-FB) renamed /FB_2
- net Net-(U6-FB) renamed /FB_3
- C15 pad 2: /3V3_BUS -> /PERIPH_PWR
- J1 pad 11: /EDFA_ENABLE -> /KAPTON_ENABLE
- J1 pad 13: /KAPTON_ENABLE -> /EDFA_ENABLE
- J1 pad 15: /5V_SW_1_EN -> unconnected-(J1-Pin_15-Pad15)
- J1 pad 17: /5V_SW_2_EN -> unconnected-(J1-Pin_17-Pad17)
- J1 pad 23: /5V_SW_2 -> unconnected-(J1-Pin_23-Pad23)
- J1 pad 24: /SHDN -> /CHRG
- J1 pad 26: unconnected-(J1-Pin_26-Pad26) -> /SHDN
- J1 pad 31: unconnected-(J1-Pin_31-Pad31) -> /5V_SW_1_EN
- J1 pad 48: unconnected-(J1-Pin_48-Pad48) -> /SOLAR_TMP_3
- J1 pad 49: unconnected-(J1-Pin_49-Pad49) -> /SOLAR_TMP_2
- J1 pad 50: unconnected-(J1-Pin_50-Pad50) -> /SOLAR_TMP_1
- J2 pad 1: /PDU_TEMP -> /SOLAR_TMP_4
- J2 pad 11: /SOLAR_TMP_3 -> unconnected-(J2-Pin_11-Pad11)
- J2 pad 2: unconnected-(J2-Pin_2-Pad2) -> /SOLAR_TMP_5
- J2 pad 3: /SOLAR_TMP_1 -> unconnected-(J2-Pin_3-Pad3)
- J2 pad 5: /SOLAR_TMP_2 -> unconnected-(J2-Pin_5-Pad5)
- J2 pad 7: /SOLAR_TMP_5 -> unconnected-(J2-Pin_7-Pad7)
- J2 pad 9: /SOLAR_TMP_4 -> unconnected-(J2-Pin_9-Pad9)
- R15 pad 1: Net-(U4-V_OUT) -> Net-(R15-Pad1)
- R15 pad 2: /PDU_TEMP -> Net-(L4-Pad2)
- R38 pad 2: Net-(L4-Pad2) -> Net-(R15-Pad1)
- R40 pad 1: Net-(L4-Pad2) -> Net-(R15-Pad1)
- U4 pad 1: Net-(U4-V_OUT) -> /PDU_TEMP
- U4 pad 5: /3V3_BUS -> /PERIPH_PWR
- U4 pad 8: /3V3_BUS -> /PERIPH_PWR
Routing:
- net GND: track 213.1 -> 34.5 mm, vias 42 -> 26
- net /PDU_TEMP: track 98.4 -> 0.00 mm
- net /SOLAR_TMP_2: track 100.5 -> 17.6 mm
- net /5V_SW_2: track 63.7 -> 0.00 mm, vias 1 -> 0
- net /3V3_BUS_STAT: track 26.3 -> 88.4 mm
- net /5V_SW_2_EN: track 53.0 -> 0.00 mm, vias 2 -> 0
- net /SOLAR_TMP_4: track 72.2 -> 21.8 mm
- net /SOLAR_TMP_5: track 79.0 -> 37.7 mm
- net /ICL: track 60.2 -> 21.2 mm, vias 2 -> 0
- net Net-(D9-A): track 39.7 -> 6.22 mm
- net /KAPTON_PWR: track 27.0 -> 60.3 mm, vias 0 -> 2
- net /SOLAR_IN_4: track 41.5 -> 8.61 mm, vias 1 -> 0
- net /SOLAR_TMP_3: track 66.5 -> 35.9 mm
- net Net-(D12-A): track 36.2 -> 6.04 mm, vias 2 -> 0
- net /SHDN: track 51.7 -> 21.6 mm, vias 2 -> 0
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- added copper zone on F.Cu, net /BATT_CS
- added copper zone on B.Cu, net /FB_1
- added copper zone on B.Cu, net /FB_2
- added copper zone on B.Cu, net /FB_3
- added copper zone on B.Cu, net /SW_1
- added copper zone on B.Cu, net /SW_2
- added copper zone on B.Cu, net /SW_3
- added copper zone on B.Cu, net GND
- added copper zone on F.Cu, net V_BATT
Other:
- outline, holes or cut-outs redrawn
- board text added: "3V3"
- board text added: "5V"
- board text added: "AVIONICS"
- board text added: "Antenna"
- board text added: "Batt Connectors"
- board text added: "Charge"
- board text added: "EDFA"
- board text added: "EDFA Switch"
- board text added: "I Chrg"
- board text added: "Inhibit Switches"
- board text added: "Kapton"
- board text added: "Kapton Switch"
- board text added: "Misc Switch"
- board text added: "Periph Switch"
- board text added: "Status LEDs"
- board text added: "VBATT"
- board text added: "made by graydon sk"
- board text added: "rev. 2.0.0, 10.22.24"
- board text removed: "5v reg stat"
- board text removed: "antenna deployment"
- board text removed: "batt connectors"
- board text removed: "batt heat"
- board text removed: "batt heat stat"
- board text removed: "edfa reg stat"
- board text removed: "inhibits"
- board text removed: "periph switch stat"
- board text removed: "rev. 1.0.0, 09.23.24"
- board text removed: "switch 1 stat"
- board text removed: "switch 2 stat"
- board text removed: "usb continuity"
