File: Avionics/BurnCircuit/_autosave-Burn Circuit.kicad_sch (KiCad schematic)
At the start: 16 parts, among them J1 5037630291, J2 5037630291, Q1 NPN, Q2 FDS6375, Q3 FDS6375, U1 PE014006

Commit message: all but Q1
Parts:
- removed D1: 1N4148WT, Diode_SMD:D_SOD-523, symbol Diode:1N4148WT
- removed R8: 4.7K, symbol Device:R
- removed R9: 100K, symbol Device:R
- added 4.7K1: R6, Resistor_THT:R_Axial_DIN0204_L3.6mm_D1.6mm_P7.62mm_Horizontal, symbol Device:R
- added D1: 1N4001, Diode_THT:D_DO-41_SOD81_P10.16mm_Horizontal, symbol Diode:1N4001
- added R2: 4.7K, Resistor_THT:R_Axial_DIN0204_L3.6mm_D1.6mm_P7.62mm_Horizontal, symbol Device:R
- R1: footprint (none) -> Resistor_THT:R_Axial_DIN0207_L6.3mm_D2.5mm_P10.16mm_Horizontal
- R3: footprint (none) -> 100K resistor:YAG_RSF100_YAG
- R4: footprint (none) -> Resistor_THT:R_Axial_DIN0204_L3.6mm_D1.6mm_P7.62mm_Horizontal
- R5: value 4.7K -> 10K; footprint (none) -> Resistor_THT:R_Axial_DIN0204_L3.6mm_D1.6mm_P7.62mm_Horizontal
- R7: value 10K -> 100K; footprint (none) -> 100K resistor:YAG_RSF100_YAG
- U1: footprint RELAY5-PE_CO -> PE014006:RELAY5-PE_CO
Connections:
- net EN_BURN1: now also R2.1; no longer R5.1
- net EN_BURN2: now also R5.1, 4.7K1.1; no longer R7.1
- net GND: now also R5.2; no longer R7.2
- net VBATT: now also D1.1 (K)
- net at MOSFET2.1 (G): now also 4.7K1.2
- net at MOSFET2.3 (D), Q3.4: now also R7.2
- net at MOSFET1.1 (G): now also R2.2; no longer R5.2
- net at Q2.1, Q3.1, R3.1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: now also R7.1
- net at Q1.1 (C), U1.A2: now also D1.2 (A)
Other:
- moved on the sheet: MOSFET1, R3, R4
