File: Avionics/BeagleBonePC104/BeagleBonePC104.kicad_sch (KiCad schematic)
At the start: 14 parts, among them U4 TJA1051T-3, U5 TMP36xS

Commit message: Ian Golberg - Tentatively Finalized v3 of the flight computer board.
Parts:
- added C2: 0.1µF, Capacitor_SMD:C_0805_2012Metric, symbol Device:C
- added D4: CAN_PWR, LED_SMD:LED_0805_2012Metric, symbol Device:LED
- added D5: TEMP_PWR, LED_SMD:LED_0805_2012Metric, symbol Device:LED
- added D6: CLK_PWR, LED_SMD:LED_0805_2012Metric, symbol Device:LED
- added R6, R7, R8: 15, Resistor_SMD:R_0805_2012Metric, symbol Device:R
- added TP1: TestPoint, TestPoint:TestPoint_Keystone_5000-5004_Miniature, symbol Connector:TestPoint
- added TP2, TP3, TP4: TestPoint, FlightCompuer:TestPointPad, symbol Connector:TestPoint
- added U3: ~, FlightCompuer:831054046, symbol FlightComputer:831054046_10MHz_Oscillator
- added U6, U7, U8, U9: ~, FlightCompuer:SPDT Through Hole Switch, symbol FlightComputer:2.54mm_Switch
- R4: value 150 -> 100; footprint Resistor_SMD:R_0603_1608Metric -> Resistor_SMD:R_0805_2012Metric
- U2: footprint PCI104Connector:PCI104ConnectorComplete -> PCI104Connector:PC104ConnectorFootprint
- renumbered R6 to R9
Connections:
- net 3V3: now also U2.80 (3V3_MAIN), TP3.1, U6.2, U8.2, U9.2; no longer C1.1, U4.3 (VCC), U4.5 (VIO), U5.5 (~{SHUTDOWN}), U5.8 (+Vs)
- net 5V: now also U7.2; no longer R1.1, R2.1, U1.5 (VDD_5V), U1.6 (VDD_5V)
- net GND: now also C2.2, R6.2, R7.2, R8.2, TP2.1, U3.2 (GND)
- net GPIO2_6: now also U2.70 (ADCS_BOOT); no longer U2.36
- net 10MHz_CLK: now reaches U2.103
- net 10MHz_CLK: now also TP1.1, U3.3 (OUTPUT)
- new net: R1.1, R2.1, U1.5 (VDD_5V), U1.6 (VDD_5V), U7.1
- new net: D6.1 (K), R8.1
- new net: C2.1, D6.2 (A), TP4.1, U3.4 (+Vs), U6.1
- new net: C1.1, D5.2 (A), U5.5 (~{SHUTDOWN}), U5.8 (+Vs), U9.1
- new net: D4.1 (K), R6.1
- new net: D4.2 (A), U4.3 (VCC), U4.5 (VIO), U8.1
- new net: D5.1 (K), R7.1
- new net 10MHz_CLK_STANDBY: U3.1 (STANDBY)
- no-connect marks 104 -> 107
Other:
- note added: "(Oscilloscope)"
- note added: "10MHz Clock"
- note added: "10MHz Clock Signal"
- note added: "A"
- note added: "BeagleBone PWR"
- note added: "CAN_PWR"
- note added: "CLK_PWR"
- note added: "TEMP_PWR"
- note added: "V"
- moved on the sheet: C1, D1, D2, D3, R1, R2, R3, R4, R5, R9, U4, U5

Commit message: Ian Goldberg - Finished Rev. 3 of the Flight Computer PCB.
Parts:
- added TP5: TestPoint, TestPoint:TestPoint_Keystone_5000-5004_Miniature, symbol Connector:TestPoint
Connections:
- net GND: now also TP5.1
Other:
- note added: "Ground Connection Testpoint"
Changed lines of the file:
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@@
 	(wire
 		(pts
+			(xy 123.19 204.47) (xy 123.19 209.55)
+		)
+		(stroke
+			(width 0)
+			(type default)
+		)
+	)
+	(wire
+		(pts
 			(xy 170.18 172.72) (xy 176.53 172.72)
 		)
@@
 	)
 	(rectangle
+		(start 111.76 194.31)
+		(end 139.7 218.44)
+		(stroke
+			(width 0)
+			(type default)
+		)
+		(fill
+			(type none)
+		)
+	)
+	(rectangle
 		(start 273.05 121.92)
 		(end 321.31 168.91)
@@
 		)
 	)
+	(text "Ground Connection Testpoint\n"
+		(exclude_from_sim no)
+		(at 125.476 193.04 0)
+		(effects
+			(font
+				(size 1.27 1.27)
+			)
+		)
+	)
 	(text "From VDD_5V\nBeaglebone supplies \nits own 3.3V\n"
 		(exclude_from_sim no)
@@
 	)
 	(symbol
+		(lib_id "power:GND")
+		(at 123.19 209.55 0)
+		(unit 1)
+		(exclude_from_sim no)
+		(in_bom yes)
+		(on_board yes)
+		(dnp no)
+		(fields_autoplaced yes)
+		(property "Reference" "#PWR09"
+			(at 123.19 215.9 0)
+			(effects
+				(font
+					(size 1.27 1.27)
+				)
+				(hide yes)
+			)
+		)
+		(property "Value" "GND"
+			(at 123.19 214.63 0)
+			(effects
+				(font
+					(size 1.27 1.27)
+				)
+			)
+		)
+		(property "Footprint" ""
+			(at 123.19 209.55 0)
+			(effects
+				(font
+					(size 1.27 1.27)
+				)
+				(hide yes)
+			)
+		)
+		(property "Datasheet" ""
+			(at 123.19 209.55 0)
+			(effects
+				(font
+					(size 1.27 1.27)
+				)
+				(hide yes)
+			)
+		)
+		(property "Description" "Power symbol creates a global label with name \"GND\" , ground"
+			(at 123.19 209.55 0)
+			(effects
+				(font
+					(size 1.27 1.27)
+				)
+				(hide yes)
+			)
+		)
+		(pin "1"
+		)
+		(instances
+			(project "BeagleBonePC104"
+				(path "/c19e4e36-81b6-4ac2-a6e5-e9e0c2677815"
+					(reference "#PWR09")
+					(unit 1)
+				)
+			)
+		)
+	)
+	(symbol
 		(lib_id "Device:R")
 		(at 90.17 92.71 0)
@@
 					(unit 1)
 				)
+			)
+		)
+	)
+	(symbol
+		(lib_id "Connector:TestPoint")
+		(at 123.19 204.47 0)
+		(unit 1)
+		(exclude_from_sim no)
+		(in_bom yes)
+		(on_board yes)
+		(dnp no)
+		(property "Reference" "TP5"
+			(at 125.73 199.8979 0)
+			(effects
+				(font
+					(size 1.27 1.27)
+				)
+				(justify left)
+			)
+		)
+		(property "Value" "TestPoint"
+			(at 125.73 202.4379 0)
+			(effects
+				(font
+					(size 1.27 1.27)
+				)
+				(justify left)
+			)
+		)
+		(property "Footprint" "TestPoint:TestPoint_Keystone_5000-5004_Miniature"
+			(at 128.27 204.47 0)
+			(effects
+				(font
+					(size 1.27 1.27)
+				)
+				(hide yes)
+			)
+		)
+		(property "Datasheet" "~"
+			(at 128.27 204.47 0)
+			(effects
+				(font
+					(size 1.27 1.27)
+				)
+				(hide yes)
+			)
+		)
+		(property "Description" "test point"
+			(at 123.19 204.47 0)
+			(effects
+				(font
+					(size 1.27 1.27)
+				)
+				(hide yes)
+			)
+		)
+		(pin "1"
+		)
+		(instances
+			(project "BeagleBonePC104"
+				(path "/c19e4e36-81b6-4ac2-a6e5-e9e0c2677815"
+					(reference "TP5")
+					(unit 1)
+				)

Commit message: Ian Goldberg - Pushing preliminary versions of version 4
Parts:
- removed C2: 0.1µF, Capacitor_SMD:C_0805_2012Metric, symbol Device:C
- removed D6: CLK_PWR, LED_SMD:LED_0805_2012Metric, symbol Device:LED
- removed R8: 15, Resistor_SMD:R_0805_2012Metric, symbol Device:R
- removed TP1: TestPoint, TestPoint:TestPoint_Keystone_5000-5004_Miniature, symbol Connector:TestPoint
- removed TP2, TP3, TP4: TestPoint, FlightCompuer:TestPointPad, symbol Connector:TestPoint
- removed U3: ~, FlightCompuer:831054046, symbol FlightComputer:831054046_10MHz_Oscillator
- removed U6, U7, U8, U9: ~, FlightCompuer:SPDT Through Hole Switch, symbol FlightComputer:2.54mm_Switch
- added BT1: Battery_Cell, Battery:BatteryHolder_Keystone_106_1x20mm, symbol Device:Battery_Cell
- added Q1: 2N7002, Package_TO_SOT_SMD:SOT-23, symbol Transistor_FET:2N7002
- added R12, R13: 10k, Resistor_SMD:R_0805_2012Metric, symbol Device:R
- added RTC_MFP1, TP6-32.768_kHz1: TestPoint, TestPoint:TestPoint_Keystone_5000-5004_Miniature, symbol Connector:TestPoint
- added SW1, SW2: SW_Push, symbol Switch:SW_Push
- added U10: MCP7940N-xSN, Package_SO:SOIC-8_3.9x4.9mm_P1.27mm, symbol Timer_RTC:MCP7940N-xSN
- added U12, U14: ~, FlightCompuer:XTAL4_SiT1533_SIT, symbol FlightComputer:SIT1533AC-H5-DCC-32.768E
- added U13: ~, FlightCompuer:QFN50P400X400X100-25N, symbol FlightComputer:MSP430FR2433_
- added U3: W25N01GVZEIG_TR, FlightCompuer:SON127P800X600X80-9N, symbol FlightComputer:W25N01GVZEIG_TR
- added U7: MAX14662, Package_DFN_QFN:QFN-28-1EP_4x4mm_P0.4mm_EP2.6x2.6mm, symbol Analog_Switch:MAX14662
- R1, R2: value 5.6k -> 2.2k; footprint Resistor_THT:R_Axial_DIN0207_L6.3mm_D2.5mm_P10.16mm_Horizontal -> Resistor_SMD:R_0805_2012Metric
Connections:
- net 10MHz_CLK_STANDBY: now also U1.46 (GPIO2_7)
- net 3V3: now also U3.8 (VCC), U7.2 (A1), U7.26 (V_{CC}), U7.3 (A2), U7.4 (A3), U7.5 (A4), U7.6 (A5), U7.7 (A6), U7.8 (A7), U7.9 (A8)
- net 5V: now also U1.5 (VDD_5V), U1.6 (VDD_5V)
- net FC_TEMP: now also U1.40 (GPIO2_13); no longer U1.23 (GPIO1_17), U2.96
- net GND: now also BT1.2 (-), Q1.2 (S), SW1.2, SW2.2, U10.4 (VSS), U12.2 (GND), U13.18 (DVSS), U13.21 (P2.0/XOUT), U14.2 (GND), U3.4 (GND), U3.9 (GND), U7.11 (GND), U7.25 (GND), U7.29 (GND); no longer U1.47 (GND), U1.48 (GND)
- net GPI02_22: now also U1.27 (GPIO3_19); no longer U1.73 (GPIO2_22)
- net GPIO0_7: now also U13.9 (P1.2/UCB0SIMO/UCB0SDA/TA0.2/A2/Veref-); no longer U2.71
- net GPIO1_12: now also U1.12 (GPIO1_28); no longer U1.58 (GPIO1_12)
- net GPIO1_13: now also U1.11 (UART4_RXD); no longer U1.57 (GPIO1_13)
- net GPIO1_14: now also U1.16 (GPIO1_14); no longer U1.62 (GPIO1_14)
- net GPIO1_15: now also U1.15 (GPIO1_16); no longer U1.61 (GPIO1_15)
- net GPIO1_16: now also U13.12 (P3.0); no longer U2.92
- net GPIO1_26: now also U1.14 (GPIO0_26); no longer U1.60 (GPIO0_26)
- net GPIO1_27: now also U1.17 (I2C1_SCL); no longer U1.63 (GPIO0_27)
- net GPIO1_28: now also U13.10 (P1.3/UCB0SOMI/UCB0SCL/MCLK/A3); no longer U2.95
- net GPIO1_29: now also U1.26 (GPIO1_29); no longer U1.72 (GPIO1_29)
- net GPIO2_1: now also U1.18 (I2C1_SDA); no longer U1.64 (GPIO2_1)
- net GPIO2_10: now also U1.41 (GPIO3_20); no longer U1.87 (GPIO2_10)
- net GPIO2_11: now also U1.42 (GPIO2_11); no longer U1.88 (GPIO2_11)
- net GPIO2_12: now also U1.39 (GPIO2_12), U2.46; no longer U1.85 (GPIO2_12), U2.44
- net GPIO2_13: now also U1.40 (GPIO2_13); no longer U1.86 (GPIO2_13)
- net GPIO2_24: now also U1.28 (SPI1_CS0); no longer U1.74 (GPIO2_24)
- net GPIO2_8: now also U1.43 (GPIO2_8); no longer U1.89 (GPIO2_8)
- net GPIO2_9: now also U1.44 (GPIO2_9); no longer U1.90 (GPIO2_9)
- net GPIO3_20: now also U13.8 (P1.1/UCB0CLK/TA0.1/A1); no longer U2.73
- net I2C_SCL: now also U10.6 (SCL), U7.24 (SCLK/SCL)
- net I2C_SDA: now also R2.1, U10.5 (SDA), U7.27 (DIN/SDA); no longer R2.2
- net SYS_RESETn: now also U13.7 (P1.0/UCB0STE/TA0CLK/A0/Veref+); no longer D3.2 (A)
- net UART_RX: now also U13.3 (P1.4/UCA0TXD/UCA0SIMO/TA1.2/TCK/A4/VREF+), U13.4 (P1.5/UCA0RXD/UCA0SOMI/TA1.1/TMS/A5); no longer U1.84 (UART5_RXD)
- net UART_TX: no longer U1.83 (UART5_TXD)
- net TEMP_PWR: now reaches C1.1, D5.2 (A), U5.5 (~{SHUTDOWN}), U5.8 (+Vs)
- net TEMP_PWR: now also U7.19 (B3)
- net SPI_CS: now reaches U1.28 (SPI1_CS0)
- net SPI_CS: now also U3.1 (/CS)
- net SPI_MOSI: now reaches U1.29 (SPI1_D0)
- net SPI_MOSI: now also U3.5 (DI(IO0))
- net SPI_MISO: now reaches U1.30 (SPI1_D1)
- net SPI_MISO: now also U3.2 (DO(IO1))
- net SPI_SCLK: now reaches U1.31 (UART5_CTSN)
- net SPI_SCLK: now also U3.6 (CLK)
- net CAN_PWR: now reaches D4.2 (A), U4.3 (VCC), U4.5 (VIO)
- net CAN_PWR: now also U7.18 (B4)
- net SPWTDIO: now reaches U2.51
- net SPWTDIO: now also Q1.3 (D), R13.2, SW2.1, U13.1 (RST/NMI/SBWTDIO)
- net SPWTCK: now reaches U2.52
- net SPWTCK: now also U13.2 (TEST/SBWTCK)
- net 10MHz_CLK: no longer names the net of U2.103
- removed net GPIO2_23: U1.75 (GPIO2_23), U2.46
- net GPIO2_25: no longer names the net of U2.42
- net GPIO2_25: no longer U1.76 (GPIO2_25)
- net GPIO2_6: no longer names the net of U2.70 (ADCS_BOOT)
- net GPIO2_6: no longer U1.91 (GPIO2_6)
- net GPIO2_7: no longer names the net of U2.68 (ADCS_ENABLE)
- net GPIO2_7: no longer U1.92 (GPIO2_7)
- net GPIO3_19: no longer names the net of U2.74
- net GPIO3_19: no longer U1.27 (GPIO3_19)
- new net: TP6-32.768_kHz1.1, U10.1 (X1), U12.3 (CLK_OUT)
- new net: R1.1, R2.2, U1.4 (GPIO1_7)
- new net: BT1.1 (+), U10.3 (VBAT)
- new net: U13.22 (P2.1/XIN), U14.3 (CLK_OUT)
- new net MSP430_PWR: R13.1, U13.24 (DVCC), U14.4 (Vdd), U7.21 (B1)
- new net MSP430_RST: Q1.1 (G), U1.45 (GPIO2_6)
- new net NAND_~{HOLD}(I/O3): U1.30 (SPI1_D1), U3.7 (/HOLD(IO3))
- new net NAND_~{WP}(I/O2): U1.29 (SPI1_D0), U3.3 (/WP(IO2))
- new net RTC_MFP: R12.2, RTC_MFP1.1, U1.27 (GPIO3_19), U10.7 (MFP)
- new net RTC_PWR: R12.1, U10.8 (VCC), U12.4 (Vdd), U7.20 (B2)
- new net SWITCH_MODE_SEL: U7.1 (SPI/~{I²C})
- new net SWITCH_SHUTDOWN: U7.22 (~{SD})
- new net ~{SYS_RESETn}: D3.2 (A), SW1.1
- no-connect marks 107 -> 122
Other:
- note added: "32.768 kHz Silicon MEMS Oscillator"
- note added: "BeagleBone Black"
- note added: "BeagleBone Manual Reset"
- note added: "CR2032 (20mm, single)"
- note added: "Check that these I2C resistors are the right resistance and can connect to the beaglebone-supplied 3V3 line"
- note added: "Check to see whether the exposed pad is connected to ground it appears in the layout editor"
- note added: "Double check this"
- note added: "MSP430 Manual Reset"
- note added: "Make sure cap. is proximate to temp IC"
- note added: "Make sure to power the MSP430FR2433 LaunchPad from the same power supply and use the same ground"
- note added: "N-channel mosfet pulls reset line low to reset MSP430"
- note added: "NAND Flash Memory IC"
- note added: "PC/104 Header"
- note added: "RTC is always on. When RTC_PWR isn't high it is operating on battery power"
- note added: "Real-Time clock with Battery Backup"
- note added: "TI MSP430FR2433 Watchdog Processor"
- note added: "This line needs a pullup resistor"
- note added: "Watchdog Processor"
- note removed: "(Oscilloscope)"
- note removed: "10MHz Clock"
- note removed: "10MHz Clock Signal"
- note removed: "A"
- note removed: "BeagleBone PWR"
- note removed: "CLK_PWR"
- note removed: "From VDD_5V Beaglebone supplies its own 3.3V"
- note removed: "Ground Connection Testpoint"
- note removed: "PCI104 Header"
- note removed: "TEMP_PWR"
- note removed: "V"
- title: BeagleBone Black PC104 Motherboard - Ian Goldberg -> Flight Computer Motherboard - Ian Goldberg
- moved on the sheet: C1, D1, D2, D3, D4, D5, R1, R2, R3, R4, R5, R6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
