File: Avionics/Batt_Boardv1/_autosave-Batt_Boardv1.kicad_pcb (KiCad board)
At the start: 2 copper layers, 17 parts, among them U3 TMP36xS

Commit message: need to fic tracks
Connections:
- BT13 pad P2: /V_BATT -> (no net)
- BT14 pad P2: /V_BATT -> (no net)
- BT15 pad P2: /V_BATT -> (no net)
- BT16 pad P2: /V_BATT -> (no net)
- BT17 pad P2: /V_BATT -> (no net)
- BT18 pad P2: /V_BATT -> (no net)
- C2 pad 1: Net-(D1-A) -> /V_BATT
- D1 pad 1: Net-(D1-K) -> /V_BATT
- R2 pad 1: Net-(D1-K) -> /V_BATT
- U1 pad 41: unconnected-(U1-I2C1_SDA-Pad41) -> /V_BATT
- U1 pad 43: unconnected-(U1-I2C1_SCL-Pad43) -> /V_BATT
- U1 pad 44: unconnected-(U1-Pad44) -> /V_BATT
- U1 pad 45: unconnected-(U1-Pad45) -> /V_BATT
- U1 pad 46: unconnected-(U1-Pad46) -> /V_BATT
- U1 pad 47: unconnected-(U1-Pad47) -> /V_BATT
- U1 pad 53: /batt_board_temp -> /V_BATT
- U3 pad 1: /batt_board_temp -> /V_BATT
- U3 pad 2: (no net) -> /V_BATT
- U3 pad 3: (no net) -> /V_BATT
- U3 pad 4: Net-(U3-GND) -> /V_BATT
Routing:
- net /batt_board_temp: track 21.2 -> 0.00 mm
- net /V_BATT: track 330.4 -> 351.7 mm
