File: Avionics/Batt_Boardv1/Batt_Boardv1.kicad_pcb (KiCad board)
At the start: 2 copper layers, 17 parts, among them U3 TMP36xS

Commit message: back to the schematic drawing board
Parts:
- moved BT17 7.00 mm to (178.3, 122.5)
- moved BT18 7.00 mm to (239.0, 122.5)
- moved BT11 7.00 mm to (178.3, 122.5)
- moved BT12 7.00 mm to (239.1, 122.5)
- moved BT7 6.00 mm to (178.4, 87.5)
- moved BT8 6.00 mm to (239.3, 87.5)
- moved BT13 6.00 mm to (178.4, 87.5)
- moved BT14 6.00 mm to (239.1, 87.5)
- moved D1 2.43 mm to (179.2, 70.5)
- moved C2 2.43 mm to (179.2, 70.5)
- moved R2 2.43 mm to (182.2, 70.5)
- moved U3 2.43 mm to (174.5, 70.5)
Connections:
- BT10 pad P2: /V_BATT -> (no net)
- BT11 pad P2: /V_BATT -> (no net)
- BT13 pad P2: /V_BATT -> (no net)
- BT14 pad P2: /V_BATT -> (no net)
- BT15 pad P2: /V_BATT -> (no net)
- BT16 pad P2: /V_BATT -> (no net)
- BT17 pad P2: /V_BATT -> (no net)
- BT18 pad P2: /V_BATT -> (no net)
- BT7 pad P2: /V_BATT -> (no net)
- BT8 pad P2: /V_BATT -> (no net)
- BT9 pad P2: /V_BATT -> (no net)
- U1 pad 100: /V_BATT -> unconnected-(U1-V_BAT-Pad100)
- U1 pad 97: /V_BATT -> unconnected-(U1-V_BAT-Pad97)
- U1 pad 98: /V_BATT -> unconnected-(U1-V_BAT-Pad98)
Routing:
- net /V_BATT: track 330.4 -> 0.00 mm
- net (no net): track 10.8 -> 5.28 mm
- net /batt_board_temp: track 21.2 -> 23.8 mm
