File: Avionics/Batt_Boardv1/Batt_Boardv1.kicad_sch (KiCad schematic)
At the start: 13 parts

Commit message: yippie
Parts:
- removed BT1, BT10, BT11, BT12, BT2, BT3, BT4, BT5, BT6, BT7, BT8, BT9: 54, 54:BAT_54, symbol Battery Holder:54
- added BT10, BT11, BT12, BT13, BT14, BT15, BT16, BT17, BT18, BT7, BT8, BT9: 54, Battery 54:BAT_254TR, symbol 54 -- Battery clips:54
- U1: footprint GPIO2_7 -> PC104:PC104ConnectorFootprint (1)
Connections:
- net V_BATT: now reaches U1.100 (V_BAT)
- net V_BATT: now also U1.97 (V_BAT), U1.98 (V_BAT), BT16.1_1, BT17.1_1, BT18.1_1
- new net: BT13.1_1, BT8.1_1
- new net: BT10.1_1, BT14.1_1
- new net: BT12.1_1, BT15.1_1
- new net GND: BT11.1_1, BT7.1_1, BT9.1_1

Commit message: need to fic tracks
Parts:
- added C2: 0.1µF, Capacitor_SMD:C_0805_2012Metric, symbol Device:C
- added D1: TEMP_PWR, LED_SMD:LED_0805_2012Metric, symbol Device:LED
- added R2: 15, Resistor_SMD:R_0805_2012Metric, symbol Device:R
- added U3: TMP36xS, Package_SO:SOIC-8_3.9x4.9mm_P1.27mm, symbol Sensor_Temperature:TMP36xS
Connections:
- net batt_board_temp: now reaches U1.53 (TEMP_1)
- net batt_board_temp: now also U3.1 (V_{OUT})
- new net: D1.1 (K), R2.1
- new net: C2.2, R2.2, U3.4 (GND)
- new net: C2.1, D1.2 (A), U3.5 (~{SHUTDOWN}), U3.8 (+Vs)

Commit message: back to the schematic drawing board
Parts:
- added J1, J2: Screw_Terminal_01x02, symbol Connector:Screw_Terminal_01x02
Connections:
- net GND: now also J1.2 (Pin_2)
- net at BT14.1_1: now also BT10.1; no longer BT10.1_1
- net V_BATT renamed BATT_CS
- net BATT_CS: now also J1.1 (Pin_1); no longer U1.100 (V_BAT), U1.97 (V_BAT), U1.98 (V_BAT)
Other:
- note added: "batt charge"
- note added: "batt discharge"
Changed lines of the file:
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@@
-	(wire
-		(pts
-			(xy 158.75 73.66) (xy 148.59 73.66)
-		)
-		(stroke
-			(width 0)
-			(type default)
-		)
-	)
 	(wire
 		(pts
@@
 	(wire
 		(pts
+			(xy 207.01 99.06) (xy 213.36 99.06)
+		)
+		(stroke
+			(width 0)
+			(type default)
+		)
+	)
+	(wire
+		(pts
 			(xy 228.6 36.83) (xy 224.79 36.83)
 		)
@@
 	(wire
 		(pts
-			(xy 148.59 96.52) (xy 165.1 96.52)
+			(xy 148.59 96.52) (xy 162.56 96.52)
 		)
 		(stroke
@@
 	(wire
 		(pts
-			(xy 116.84 73.66) (xy 113.03 73.66)
-		)
-		(stroke
-			(width 0)
-			(type default)
-		)
-	)
-	(wire
-		(pts
 			(xy 113.03 17.78) (xy 118.11 17.78)
 		)
@@
 	(wire
 		(pts
-			(xy 158.75 76.2) (xy 148.59 76.2)
-		)
-		(stroke
-			(width 0)
-			(type default)
-		)
-	)
-	(wire
-		(pts
 			(xy 30.48 119.38) (xy 30.48 132.08)
 		)
@@
 	(wire
 		(pts
+			(xy 207.01 100.33) (xy 207.01 99.06)
+		)
+		(stroke
+			(width 0)
+			(type default)
+		)
+	)
+	(wire
+		(pts
 			(xy 148.59 132.08) (xy 143.51 132.08)
 		)
@@
 	(wire
 		(pts
+			(xy 203.2 96.52) (xy 213.36 96.52)
+		)
+		(stroke
+			(width 0)
+			(type default)
+		)
+	)
+	(wire
+		(pts
 			(xy 203.2 40.64) (xy 203.2 43.18)
 		)
@@
 		)
 	)
-	(label "V_BATT"
-		(at 158.75 76.2 0)
-		(fields_autoplaced yes)
+	(text "batt charge"
+		(exclude_from_sim no)
+		(at 192.786 115.062 0)
 		(effects
 			(font
 				(size 1.27 1.27)
 			)
-			(justify left bottom)
-		)
-	)
-	(label "V_BATT"
-		(at 158.75 73.66 0)
+		)
+	)
+	(text "batt discharge"
+		(exclude_from_sim no)
+		(at 192.786 97.79 0)
+		(effects
+			(font
+				(size 1.27 1.27)
+			)
+		)
+	)
+	(label "BATT_CS"
+		(at 162.56 96.52 0)
 		(fields_autoplaced yes)
 		(effects
@@
 		)
 	)
-	(label "V_BATT"
-		(at 165.1 96.52 0)
-		(fields_autoplaced yes)
-		(effects
-			(font
-				(size 1.27 1.27)
-			)
-			(justify left bottom)
-		)
-	)
-	(label "V_BATT"
-		(at 116.84 73.66 0)
+	(label "BATT_CS"
+		(at 203.2 96.52 0)
 		(fields_autoplaced yes)
 		(effects
@@
 	)
 	(symbol
+		(lib_name "54_1")
 		(lib_id "54 -- Battery clips:54")
 		(at 72.39 119.38 180)
@@
 			)
 		)
-		(pin "1_1"
+		(pin "1"
 		)
 		(instances
@@
 				(path "/a5e22de5-0e9e-4e3b-9cf5-d999de47cef4"
 					(reference "BT10")
+					(unit 1)
+				)
+			)
+		)
+	)
+	(symbol
+		(lib_id "power:GND")
+		(at 207.01 100.33 0)
+		(unit 1)
+		(exclude_from_sim no)
+		(in_bom yes)
+		(on_board yes)
+		(dnp no)
+		(fields_autoplaced yes)
+		(property "Reference" "#PWR02"
+			(at 207.01 106.68 0)
+			(effects
+				(font
+					(size 1.27 1.27)
+				)
+				(hide yes)
+			)
+		)
+		(property "Value" "GND"
+			(at 207.01 105.41 0)
+			(effects
+				(font
+					(size 1.27 1.27)
+				)
+			)
+		)
+		(property "Footprint" ""
+			(at 207.01 100.33 0)
+			(effects
+				(font
+					(size 1.27 1.27)
+				)
+				(hide yes)
+			)
+		)
+		(property "Datasheet" ""
+			(at 207.01 100.33 0)
+			(effects
+				(font
+					(size 1.27 1.27)
+				)
+				(hide yes)
+			)
+		)
+		(property "Description" "Power symbol creates a global label with name \"GND\" , ground"
+			(at 207.01 100.33 0)
+			(effects
+				(font
+					(size 1.27 1.27)
+				)
+				(hide yes)
+			)
+		)
+		(pin "1"
+		)
+		(instances
+			(project "Batt_Boardv1"
+				(path "/a5e22de5-0e9e-4e3b-9cf5-d999de47cef4"
+					(reference "#PWR02")
 					(unit 1)
 				)
@@
 	)
 	(symbol
+		(lib_id "Connector:Screw_Terminal_01x02")
+		(at 218.44 113.03 0)
+		(unit 1)
+		(exclude_from_sim no)
+		(in_bom yes)
+		(on_board yes)
+		(dnp no)
+		(fields_autoplaced yes)
+		(property "Reference" "J2"
+			(at 220.98 113.0299 0)
+			(effects
+				(font
+					(size 1.27 1.27)
+				)
+				(justify left)
+			)
+		)
+		(property "Value" "Screw_Terminal_01x02"
+			(at 220.98 115.5699 0)
+			(effects
+				(font
+					(size 1.27 1.27)
+				)
+				(justify left)
+			)
+		)
+		(property "Footprint" ""
+			(at 218.44 113.03 0)
+			(effects
+				(font
+					(size 1.27 1.27)
+				)
+				(hide yes)
+			)
+		)
+		(property "Datasheet" "~"
+			(at 218.44 113.03 0)
+			(effects
+				(font
+					(size 1.27 1.27)
+				)
+				(hide yes)
+			)
+		)
+		(property "Description" "Generic screw terminal, single row, 01x02, script generated (kicad-library-utils/schlib/autogen/connector/)"
+			(at 218.44 113.03 0)
+			(effects
+				(font
+					(size 1.27 1.27)
+				)
+				(hide yes)
+			)
+		)
+		(pin "1"
+		)
+		(pin "2"
+		)
+		(instances
+			(project "Batt_Boardv1"
+				(path "/a5e22de5-0e9e-4e3b-9cf5-d999de47cef4"
+					(reference "J2")
+					(unit 1)
+				)
+			)
+		)
+	)
+	(symbol
 		(lib_id "54 -- Battery clips:54")
 		(at 133.35 106.68 180)
@@
 					(unit 1)
 				)
+			)
+		)
+	)
+	(symbol
+		(lib_id "Connector:Screw_Terminal_01x02")
+		(at 218.44 96.52 0)
+		(unit 1)
+		(exclude_from_sim no)
+		(in_bom yes)
+		(on_board yes)
+		(dnp no)
+		(fields_autoplaced yes)
+		(property "Reference" "J1"
+			(at 220.98 96.5199 0)
+			(effects
+				(font
+					(size 1.27 1.27)
+				)
+				(justify left)
+			)
+		)
+		(property "Value" "Screw_Terminal_01x02"
+			(at 220.98 99.0599 0)
+			(effects
+				(font
+					(size 1.27 1.27)
+				)
+				(justify left)
+			)
+		)
+		(property "Footprint" ""
+			(at 218.44 96.52 0)
+			(effects
+				(font
+					(size 1.27 1.27)
+				)
+				(hide yes)
+			)
+		)
+		(property "Datasheet" "~"
+			(at 218.44 96.52 0)
+			(effects
+				(font
+					(size 1.27 1.27)
+				)
+				(hide yes)
+			)
+		)
+		(property "Description" "Generic screw terminal, single row, 01x02, script generated (kicad-library-utils/schlib/autogen/connector/)"
+			(at 218.44 96.52 0)
+			(effects
+				(font
+					(size 1.27 1.27)
+				)
+				(hide yes)
+			)
+		)
+		(pin "1"
+		)
+		(pin "2"
+		)
+		(instances
+			(project ""
+				(path "/a5e22de5-0e9e-4e3b-9cf5-d999de47cef4"
+					(reference "J1")
+					(unit 1)
+				)
