File: Avionics/Batt_Boardv2/_autosave-Batt_Boardv1.kicad_pcb (KiCad board)
At the start: 2 copper layers, 43 parts, among them J3 Screw_Terminal_01x01, J4 JST_PH_S2B-PH-SM4, J5 Screw_Terminal_01x02, J6 Screw_Terminal_01x02, J7 Screw_Terminal_01x02, J8 Screw_Terminal_01x02, Q1 IRF7458, Q2 IRF7458, U3 TMP36xS

Commit message: just need traces
Parts:
- moved H3 134.5 mm to (249.1, 55.0)
- moved H4 101.2 mm to (176.5, 55.0)
- moved H2 99.5 mm to (249.0, 140.5)
- moved H1 21.7 mm to (169.0, 140.5)
- moved U1 0.32 mm to (164.0, 145.6)
Connections:
- H1 pad 1: Net-(H1-Pad1) -> /Pack -
- H2 pad 1: Net-(H1-Pad1) -> /Pack -
- H3 pad 1: Net-(H1-Pad1) -> /Pack -
- H4 pad 1: Net-(H1-Pad1) -> /Pack -
Routing:
- net /Pack -: track 0.00 -> 0.93 mm
- net (no net): track 1.56 -> 0.63 mm
Changed lines of the file:
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@@
 	(net 120 "/Pack +")
 	(net 121 "/BM")
-	(net 122 "Net-(H1-Pad1)")
 	(footprint "Battery 54:BAT_254TR"
 		(layer "F.Cu")
@@
 	(footprint "MountingHole:MountingHole_3.2mm_M3_DIN965_Pad"
 		(layer "F.Cu")
-		(at 149.5 152.5)
+		(at 176.5 55)
 		(descr "Mounting Hole 3.2mm, M3, DIN965")
 		(tags "mounting hole 3.2mm m3 din965")
@@
 		)
 		(pad "1" thru_hole circle
-			(at 0 0)
-			(size 5.6 5.6)
+			(at 0 0 90)
+			(size 6.4 6.4)
 			(drill 3.2)
 			(layers "*.Cu" "*.Mask")
 			(remove_unused_layers no)
-			(net 122 "Net-(H1-Pad1)")
+			(net 86 "/Pack -")
 			(pinfunction "1")
 			(pintype "input")
@@
 			(layer "F.Fab")
 		)
-		(pad "1" smd rect
-			(at 8.005 0)
-			(size 4.24 3.3)
-			(layers "F.Cu" "F.Paste" "F.Mask")
-			(solder_mask_margin 0.102)
-		)
 		(pad "P1" smd rect
 			(at -8.005 0)
@@
 			(solder_mask_margin 0.102)
 		)
+		(pad "P2" smd rect
+			(at 8.005 0)
+			(size 4.24 3.3)
+			(layers "F.Cu" "F.Paste" "F.Mask")
+			(solder_mask_margin 0.102)
+		)
 	)
 	(footprint "PC104:PC104ConnectorFootprint (1)"
 		(layer "F.Cu")
-		(at 163.96175 145.269563)
+		(at 164.03 145.58)
 		(property "Reference" "U1"
 			(at 0 -0.5 0)
@@
 		(fp_arc
 			(start 35.147914 0)
-			(mid 35.848689 -1.754737)
+			(mid 35.848689 -1.75474)
 			(end 37.585 -2.5)
 			(stroke
@@
 		(fp_arc
 			(start 90.17 -38.358018)
-			(mid 88.379938 -39.143672)
+			(mid 88.380013 -39.143777)
 			(end 87.67 -40.965104)
 			(stroke
@@
 			(layer "F.SilkS")
 		)
-		(fp_text user "2"
-			(at 5.1 -90.22 90)
+		(fp_text user "H2"
+			(at 0.65 -88.768 0)
 			(unlocked yes)
 			(layer "F.SilkS")
 			(effects
 				(font
-					(size 1 1)
-					(thickness 0.1)
+					(size 1.2 1.2)
+					(thickness 0.2)
+					(bold yes)
 				)
 				(justify left bottom)
 			)
 		)
-		(fp_text user "2"
-			(at 5.1 -85.14 90)
+		(fp_text user "1"
+			(at 5.1 -87.7 90)
 			(unlocked yes)
 			(layer "F.SilkS")
@@
 			)
 		)
-		(fp_text user "H1"
-			(at 0.65 -83.688 0)
+		(fp_text user "2"
+			(at 5.1 -90.22 90)
 			(unlocked yes)
 			(layer "F.SilkS")
 			(effects
 				(font
-					(size 1.2 1.2)
-					(thickness 0.2)
-					(bold yes)
+					(size 1 1)
+					(thickness 0.1)
 				)
 				(justify left bottom)
 			)
 		)
-		(fp_text user "1"
-			(at 5.1 -82.62 90)
+		(fp_text user "2"
+			(at 5.1 -85.14 90)
 			(unlocked yes)
 			(layer "F.SilkS")
@@
 		)
 		(fp_text user "1"
-			(at 5.1 -87.7 90)
+			(at 5.1 -82.62 90)
 			(unlocked yes)
 			(layer "F.SilkS")
@@
 			)
 		)
-		(fp_text user "H2"
-			(at 0.65 -88.768 0)
+		(fp_text user "H1"
+			(at 0.65 -83.688 0)
 			(unlocked yes)
 			(layer "F.SilkS")
@@
 		)
 		(group ""
-			(members "036b6d63-091a-419e-a862-c77e6786d5ea" "03cd645c-b3ad-4845-b72c-31f0cf236868"
-				"11398654-1f42-4cb3-8018-85149fc15028" "1c1c4805-9afe-40d6-895e-ed3d4d596081"
-				"1e663f32-e6ba-4f4c-9ef0-587d0e8a0370" "1ff6fa6d-0a36-4c65-85b0-b129fd1bc1b7"
-				"21eb91d6-48d7-4c8c-addd-5c7839fdb4ae" "227df9ef-8829-4802-b95a-f62b39a7db58"
-				"282c1a42-680e-4f74-bf3d-4b9432f4464c" "34666ffe-b873-4b68-b536-dfe37a07a068"
-				"3595fbf6-2a4e-4aa8-8c31-aa028fd77079" "385824c8-28f3-4cc0-a262-3c9f885cba25"
-				"39d94564-79d3-4261-9d80-7453b027e713" "3f4091e7-290e-4f66-9313-26340642c460"
-				"3ffc80ae-7ea6-4c71-af83-7fdbd9165b9c" "433c1e3d-3987-4d38-bb67-754123406231"
-				"53a9d06c-bf0d-42ff-a3b2-28eb2eb3db03" "53ce5a00-6274-4d47-8319-7425afc17611"
-				"5a4c060a-db49-44ac-b982-5fa3a960ceb4" "61f955d6-2ed2-4836-8415-dfb0fb11cd2c"
-				"64e2fa01-78e9-40e8-904b-a6ce6111ed8c" "661dd79d-2f6e-4d58-b5b5-45f7e71e7caf"
-				"69435117-0abe-47c2-a505-a2cceff54362" "6a70b96a-d06b-494b-a8b9-76dceb6a8164"
-				"6d609488-c940-472e-8e31-a11dbc52c003" "6ec135a4-ab3e-4dc6-aaff-b0eba9286596"
-				"71eed347-3190-46ab-8dd3-b52f035bd6a3" "72cb09f3-6136-4ebf-b82d-25fbc8d34a31"
-				"7320310d-085d-4df4-b97f-efb6a0be10a1" "7df5456a-d702-4a3e-9c95-28233afd572a"
-				"8004d504-f2d8-462a-9acf-e58a14a9045e" "8c57ee4a-6b0c-4c0a-bb43-3c5bf036dffc"
-				"8cc9a322-584f-4aa5-b8ef-d7a36fb3a2ca" "99846578-0ee9-42ec-acc0-bde774dd4ac9"
-				"9e2cd252-f267-46f6-a225-56424b8ac752" "a52d0e3b-cec8-4853-80f5-b1b6306a5497"
-				"b11a6ed7-cf76-48ef-a3b6-ab88175f130a" "b137293e-4bdc-4cd6-8dc6-d9c2cdcc4502"
-				"bbf4c3db-9043-48e1-bfce-cc362ca5e167" "bd21f47c-b4b5-4c78-87a8-fbc3c714c4d1"
-				"c36420a4-dfec-422d-8089-2051e362f7ff" "c8a660f8-37d1-463a-b1ae-f8d1b1af4164"
-				"cb6cc8af-e187-450c-afbd-4834ea33a896" "cbd458d6-b0d4-4faf-9012-0f0b4a82cd7e"
-				"cf3aa338-b465-458d-9a1f-78a0bb35e475" "d75a3eb5-a45e-4b42-99a1-48dcbd1c4b41"
-				"db268b79-d174-4f5f-a175-9cb3eee8121d" "e3e99399-b9e7-4586-b2c6-db200aa0120b"
-				"ee6aafaa-110b-4506-af12-fc5760a886ef" "ee93e5d3-e32b-4bc6-b519-fe7e623388e1"
-				"f7213b7e-0199-443b-b06b-0f20d426a270" "fa22a542-fead-4d3e-b245-ad9ed83e36cb"
+			(members "01604dd4-c9bb-48ee-8ec8-a5b7de931a7b" "01f8a85c-1ea7-471a-9a9a-b3471f81a3db"
+				"0936e409-7120-4e1f-b66f-4aa1e5cc9e27" "133c8c0a-6f75-42e1-9125-5736bca81f10"
+				"1891f26e-dc64-41b6-b3c5-1fe7e92421ed" "23efa8d0-5344-4228-a894-3f1e46d1f985"
+				"29f8295f-0f8f-451e-b76d-40320ab36ab6" "2bdbe886-a1c3-498f-be47-b321381202ce"
+				"2d376743-a7ab-4988-b400-60562e0396fe" "2f4eaa3f-7d2a-4610-8b55-8a6ba2d83991"
+				"2fec14fe-f3fe-467c-b70a-04fc267291b4" "4444398e-39cb-4a3d-9324-6528c4b03ac3"
+				"48915209-7950-49b9-8d65-eb6bfe0de954" "4bb79391-1dc4-469f-aef1-4c164bef2bda"
+				"4dd482a0-2de1-4f0c-b64f-393e1bd6066c" "507bd215-10e8-4f31-9fba-e9692aa33fde"
+				"543b164a-7e73-4689-ae61-bfd29646fd17" "5b3f4ac2-0cd8-4d36-85a4-cf57668d8ed3"
+				"673f25b1-70a5-47bb-a864-6012ae4dea09" "692a7eda-c097-4617-b653-56f9b9d3fe02"
+				"6b2b0fc3-76e5-4428-9096-445ee8a45073" "7c8a8676-943d-4e82-80a3-dfc88c8dd920"
+				"8bd9f10b-5449-4919-aa76-55f526ec3046" "9352d76e-49fa-4ada-b3ab-6c999e7b1254"
+				"9463de17-d63b-487f-a50a-ee845a54798f" "9bd59068-25a4-42e2-9ef5-ff918237c25e"
+				"9ce90f6f-1da8-4c58-8ad6-b2dbfadad12b" "9f91476b-bb0e-4093-9a29-51ccf96da7f0"
+				"a0c34055-14a1-4262-bc05-f2829766f8b1" "a332d8ff-10d3-4ada-9c70-29edc3817ff9"
+				"ad511e5a-93c9-4f2c-8665-1aae5cddcef1" "b00b856d-88c7-47ba-86a8-08632e6fd087"
+				"b52399f4-4ef9-4ae0-9666-a3eabbcd20a3" "b58f3eb1-f08b-4fbe-a6d4-d08619fa9751"
+				"b784df8d-0088-460a-8a97-94933ce2626e" "becf178e-1017-47aa-ad92-28662231b1c8"
+				"c540caf7-e499-4372-8355-1515093025c1" "c669d3fa-821a-4aa0-b8d2-3937ddadfbb9"
+				"cadd3765-6d6d-4d3c-8bc2-e2d0723c7a12" "cb549325-2be1-412f-beeb-0b2b985832df"
+				"d94bef7f-1e29-43db-bce7-66f91db0105a" "da513111-89dd-46d6-ae73-4fd92d3d1b30"
+				"e02fa95e-0748-48d0-a4f7-78831bd91bcc" "e115fa85-998f-457c-9972-08b2b6776a45"
+				"e15b20ac-4f4b-4143-83bf-ccd1979a7da8" "e7217de1-b52a-4e5a-a886-331bf392f06c"
+				"f041d212-2653-4800-a7f3-e6c5d20921a3" "f5ff5c97-3ffe-494f-8a44-ad55a300d962"
+				"f70190f0-992d-465e-a84c-fcb4e5796165" "f93c9c8e-b989-4e34-b6e3-ee3c0f3a92e8"
+				"f99bfcd9-ea83-470f-86f5-54d7061dc025" "fc6fba1e-d8a8-49e3-857e-6c031d062efb"
 			)
 		)
@@
 	(footprint "MountingHole:MountingHole_3.2mm_M3_DIN965_Pad"
 		(layer "F.Cu")
-		(at 149.5 138.2)
+		(at 249 140.5)
 		(descr "Mounting Hole 3.2mm, M3, DIN965")
 		(tags "mounting hole 3.2mm m3 din965")
@@
 		(sheetname "Root")
 		(sheetfile "Batt_Boardv1.kicad_sch")
-		(attr exclude_from_pos_files)
+		(attr exclude_from_pos_files exclude_from_bom)
 		(fp_circle
 			(center 0 0)
@@
 		)
 		(pad "1" thru_hole circle
-			(at 0 0)
-			(size 5.6 5.6)
+			(at 0 0 90)
+			(size 6.4 6.4)
 			(drill 3.2)
 			(layers "*.Cu" "*.Mask")
 			(remove_unused_layers no)
-			(net 122 "Net-(H1-Pad1)")
+			(net 86 "/Pack -")
 			(pinfunction "1")
 			(pintype "input")
@@
 	(footprint "MountingHole:MountingHole_3.2mm_M3_DIN965_Pad"
 		(layer "F.Cu")
-		(at 149.5 145.35)
+		(at 249.11 55)
 		(descr "Mounting Hole 3.2mm, M3, DIN965")
 		(tags "mounting hole 3.2mm m3 din965")
@@
 			(layers "*.Cu" "*.Mask")
 			(remove_unused_layers no)
-			(net 122 "Net-(H1-Pad1)")
+			(net 86 "/Pack -")
 			(pinfunction "1")
 			(pintype "input")
@@
 	(footprint "MountingHole:MountingHole_3.2mm_M3_DIN965_Pad"
 		(layer "F.Cu")
-		(at 149.5 131.05)
+		(at 169 140.5)
 		(descr "Mounting Hole 3.2mm, M3, DIN965")
 		(tags "mounting hole 3.2mm m3 din965")
@@
 			(layers "*.Cu" "*.Mask")
 			(remove_unused_layers no)
-			(net 122 "Net-(H1-Pad1)")
+			(net 86 "/Pack -")
 			(pinfunction "1")
 			(pintype "input")
@@
 		(width 0.2)
 		(layer "F.Cu")
-		(net 0)
+		(net 86)
 	)
 	(group ""
