File: Avionics/Batt_Boardv2/Batt_Boardv1.kicad_sch (KiCad schematic)
At the start: 39 parts, among them J3 Screw_Terminal_01x01, J4 JST_PH_S2B-PH-SM4, J5 Screw_Terminal_01x02, J6 Screw_Terminal_01x02, J7 Screw_Terminal_01x02, J8 Screw_Terminal_01x02, Q1 IRF7458, Q2 IRF7458, U3 TMP36xS

Commit message: just need traces
Parts:
- added TP1, TP2, TP3, TP4: TestPoint, TestPoint:TestPoint_Loop_D1.80mm_Drill1.0mm_Beaded, symbol Connector:TestPoint
Connections:
- net PACK+ is gone; now on net Pack +: J4.1 (Pin_1), J5.1 (Pin_1), J6.1 (Pin_1), J7.1 (Pin_1), J8.1 (Pin_1)
- net B-: now also TP1.1
- net BM: now also TP2.1
- net PACK-: no longer J4.2 (Pin_2), J5.2 (Pin_2), J6.2 (Pin_2), J7.2 (Pin_2), J8.2 (Pin_2)
- net GND: now reaches C2.2, R2.2, U3.4 (GND)
- net + renamed Pack +
- net Pack +: now also TP4.1
- net - renamed Pack -
- net Pack -: now also J4.2 (Pin_2), J5.2 (Pin_2), J6.2 (Pin_2), J7.2 (Pin_2), J8.2 (Pin_2), TP3.1
- no-connect marks 0 -> 100
Other:
- note added: "Test Points"
- moved on the sheet: J4, J5, J6, J7, J8

Commit message: meeting
Parts:
- removed D1: TEMP_PWR, LED_SMD:LED_0805_2012Metric, symbol Device:LED
- removed H1, H2, H3, H4: MountingHole_Pad, MountingHole:MountingHole_3.2mm_M3_DIN965_Pad, symbol Mechanical:MountingHole_Pad
- removed J3: Screw_Terminal_01x01, Connector_PinHeader_1.00mm:PinHeader_1x01_P1.00mm_Vertical, symbol Connector:Screw_Terminal_01x01
- removed J4: JST_PH_S2B-PH-SM4, Connector_JST:JST_PH_S2B-PH-SM4-TB_1x02-1MP_P2.00mm_Horizontal, symbol Connector:Screw_Terminal_01x02
- removed J5, J6, J7, J8: Screw_Terminal_01x02, TerminalBlock:TerminalBlock_Altech_AK300-2_P5.00mm, symbol Connector:Screw_Terminal_01x02
- removed R2: 15, Resistor_SMD:R_0805_2012Metric, symbol Device:R
- removed TH1: Thermistor, Resistor_THT:R_Axial_DIN0204_L3.6mm_D1.6mm_P5.08mm_Vertical, symbol Device:Thermistor
- C1, C3, C4, C5: footprint Capacitor_SMD:C_0603_1608Metric -> Capacitor_SMD:C_0805_2012Metric
- R1: footprint Resistor_SMD:R_2512_6332Metric -> Package_TO_SOT_SMD:TO-263-2
- R4, R5: footprint Resistor_SMD:R_0603_1608Metric -> Resistor_SMD:R_0805_2012Metric
- S-8252: renamed from R5460N233AF1; footprint Connector_PinHeader_2.54mm:PinHeader_2x03_P2.54mm_Vertical_SMD -> Package_TO_SOT_SMD:SOT-23-5
Connections:
- net Pack + is gone; now on net BATT_CS: BT16.1_1, BT17.1_1, BT18.1_1, TP4.1
- net Pack - is gone; now on net GND: C1.2, Q2.1 (S), Q2.2 (S), Q2.3 (S), R3.2, TP3.1
- net BATT_CS: now also U1.10, U1.11, U1.12 (BGLBON_RST), U1.9
- net BM: now also BT12.1_1, BT13.1_1, BT15.1_1, BT8.1_1
- net GND: now also U1.81 (GND), U1.82 (GND), U1.83 (GND), U1.84 (GND)
- net batt_board_temp: now also U1.57 (TEMP_7); no longer U1.53 (TEMP_1)
- net 3V3: now reaches U1.79 (3V3_MAIN)
- net 3V3: now also C2.1, U1.80 (3V3_MAIN), U3.5 (~{SHUTDOWN}), U3.8 (+Vs)
- no-connect marks 100 -> 93
Other:
- note removed: "OPTIONAL"
- note removed: "Vertical or horizontal JST_PH"

Commit message: feat: batt & PDU progress
Parts:
- removed BT10, BT11, BT12, BT13, BT14, BT15, BT17, BT18, BT7, BT8, BT9: 54, Battery 54:BAT_254TR, symbol 54 -- Battery clips:54
- removed U1: ~, PC104:PC104ConnectorFootprint (1), symbol PC104:PCI104
- added BT1, BT2, BT3, BT4, BT5: 54, 254:BAT_254_1, symbol 54 -- Battery clips:54
- added H1, H2, H3, H4: MountingHole, MountingHole:MountingHole_3.2mm_M3_Pad_TopBottom, symbol Mechanical:MountingHole_Pad_MP
- added J1, J2: Conn_02x26_Odd_Even, Connector_PinHeader_2.54mm:PinHeader_2x26_P2.54mm_Vertical, symbol Connector_Generic:Conn_02x26_Odd_Even
- BT16: footprint Battery 54:BAT_254TR -> 254:BAT_254_1
Connections:
- net B-: now also BT3.2 (BATT-), BT4.2 (BATT-), BT5.2 (BATT-)
- net BM: now also BT16.2 (BATT-), BT2.2 (BATT-), BT3.1 (BATT+), BT5.1 (BATT+)
- net GND: now also H1.MP, H2.MP, H3.MP, H4.MP; no longer C1.2, C2.2, Q2.1 (S), Q2.2 (S), Q2.3 (S), R3.2, TP3.1, U3.4 (GND)
- net BATT_CS renamed BATT_PRE_INH
- net BATT_PRE_INH: now also BT16.1 (BATT+), BT1.1 (BATT+), BT2.1 (BATT+), J1.11 (Pin_11), J1.12 (Pin_12), J1.13 (Pin_13), J1.14 (Pin_14), J1.5 (Pin_5), J1.6 (Pin_6), J1.7 (Pin_7), J1.8 (Pin_8); no longer BT16.1_1
- new net: BT1.2 (BATT-), BT4.1 (BATT+)
- new net 3V3_BUS: J2.27 (Pin_27), J2.28 (Pin_28)
- new net 3V3_BUS_STAT: J2.24 (Pin_24)
- new net 5V_BUS: J2.25 (Pin_25), J2.26 (Pin_26)
- new net 5V_BUS_STAT: J2.23 (Pin_23)
- new net 5V_SW_1: J1.21 (Pin_21)
- new net 5V_SW_1_EN: J1.31 (Pin_31)
- new net BURN_FET: J1.29 (Pin_29)
- new net CHRG: J1.24 (Pin_24)
- new net EDFA_5V_STAT: J2.19 (Pin_19)
- new net EDFA_5V_SW: J2.21 (Pin_21), J2.22 (Pin_22)
- new net ENAB_BURN_1: J1.28 (Pin_28)
- new net ENAB_BURN_2: J1.30 (Pin_30)
- new net GNDREF: C1.2, C2.2, J1.33 (Pin_33), J1.34 (Pin_34), J1.35 (Pin_35), J1.36 (Pin_36), Q2.1 (S), Q2.2 (S), Q2.3 (S), R3.2, TP3.1, U3.4 (GND)
- new net ICL: J1.22 (Pin_22)
- new net PERIPH_EN: J1.27 (Pin_27)
- new net PERIPH_PWR: J1.47 (Pin_47)
- new net SCL: J1.43 (Pin_43)
- new net SDA: J1.41 (Pin_41)
- new net SHDN: J1.26 (Pin_26)
- new net SOLAR_TMP_+Y: J1.48 (Pin_48)
- new net SOLAR_TMP_-Y: J1.50 (Pin_50)
- new net SOLAR_TMP_-Z: J1.49 (Pin_49)
- new net SOLAR_TMP_4: J2.1 (Pin_1)
- new net SOLAR_TMP_5: J2.2 (Pin_2)
- new net V_BATT: J2.46 (Pin_46), J2.48 (Pin_48)
- no-connect marks 93 -> 22
Other:
- note added: "Inner Bank"
- note added: "Outer Bank"

Commit message: PDU 3.0.0
Connections:
- net BM: now also BT1.2 (BATT-), BT4.1 (BATT+)
Changed lines of the file:
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@@
+	)
+	(junction
+		(at 88.9 119.38)
+		(diameter 0)
+		(color 0 0 0 0)
 	)
 	(junction
@@
 	(wire
 		(pts
+			(xy 73.66 119.38) (xy 88.9 119.38)
+		)
+		(stroke
+			(width 0)
+			(type default)
+		)
+	)
+	(wire
+		(pts
 			(xy 217.17 69.85) (xy 217.17 59.69)
 		)
@@
 	(wire
 		(pts
-			(xy 73.66 119.38) (xy 104.14 119.38)
-		)
-		(stroke
-			(width 0)
-			(type default)
-		)
-	)
-	(wire
-		(pts
 			(xy 147.32 44.45) (xy 149.86 44.45)
 		)
@@
 	(wire
 		(pts
+			(xy 88.9 119.38) (xy 104.14 119.38)
+		)
+		(stroke
+			(width 0)
+			(type default)
+		)
+	)
+	(wire
+		(pts
 			(xy 105.41 85.09) (xy 115.57 85.09)
 		)
@@
 	(wire
 		(pts
-			(xy 88.9 106.68) (xy 88.9 132.08)
+			(xy 88.9 106.68) (xy 88.9 119.38)
 		)
 		(stroke
@@
 		)
 		(stroke
+			(width 0)
+			(type default)
+		)
+	)
+	(wire
+		(pts
+			(xy 88.9 119.38) (xy 88.9 132.08)
+		)
+		(stroke
