File: Avionics/PowerDistribution/PowerDistribution.kicad_sch (KiCad schematic)
At the start: 175 parts, among them J1 Conn_02x26_Odd_Even, J10 Screw_Terminal_01x02, J11 Conn_01x04, J12 Conn_01x04, J13 Conn_01x04, J14 Conn_01x04, J15 Conn_01x04, J16 Screw_Terminal_01x02, J2 Conn_02x26_Odd_Even, J3 Screw_Terminal_01x02, J4 Screw_Terminal_01x02, J5 Screw_Terminal_01x02, J6 Screw_Terminal_01x02, J7 USB_C_Receptacle_USB2.0_14P, J8 Screw_Terminal_01x02, J9 Screw_Terminal_01x02, Q1 BC848ALT1G, Q2 IRLML2803PBFCT, Q3 IRLML2803PBFCT, U1 LT8610, U16 INA219AxD, U17 INA219AxD, U18 INA219AxD, U19 INA219AxD, U2 LT8610, U20 INA219AxD, U21 INA219AxD, U6 LT8610

Commit message: feat: batt & PDU progress
Parts:
- removed C31, C32, C34, C36: 0.1uF, Capacitor_SMD:C_0805_2012Metric, symbol Device:C
- removed C33: 4.7uF, Capacitor_SMD:C_0805_2012Metric, symbol Device:C
- removed C35, C39: 10uF, Capacitor_SMD:C_0805_2012Metric, symbol Device:C
- removed C37, C38: 1uF, Capacitor_SMD:C_0805_2012Metric, symbol Device:C
- removed D14: 150060VS75000, LED_SMD:LED_0603_1608Metric, symbol Device:LED
- removed D15: CMDSH-3TR, Diode_SMD:D_SOD-323F, symbol Device:D_Schottky
- removed D16, D17: MBR230S1F, Diode_SMD:D_SOD-123F, symbol Device:D
- removed J10, J16, J3, J4, J5, J6, J8, J9: Screw_Terminal_01x02, TerminalBlock:TerminalBlock_Xinya_XY308-2.54-2P_1x02_P2.54mm_Horizontal, symbol Connector:Screw_Terminal_01x02
- removed J14, J15: Conn_01x04, Connector_Molex:Molex_CLIK-Mate_502382-0470_1x04-1MP_P1.25mm_Vertical, symbol Connector_Generic:Conn_01x04
- removed L4: AIML-0805-150K-T, Inductor_SMD:L_0805_2012Metric, symbol Device:L
- removed R32: 6.04k, Resistor_SMD:R_0805_2012Metric, symbol Device:R
- removed R35: 0, Resistor_SMD:R_0805_2012Metric, symbol Device:R
- removed R36: 169k, Resistor_SMD:R_0805_2012Metric, symbol Device:R
- removed R37: 28.4k, Resistor_SMD:R_0805_2012Metric, symbol Device:R
- removed R38, R39: 3.01k, Resistor_SMD:R_0805_2012Metric, symbol Device:R
- removed R40: 1, Resistor_SMD:R_0805_2012Metric, symbol Device:R
- removed R41: 5.1k, Resistor_SMD:R_0805_2012Metric, symbol Device:R
- removed U12: ~, Package_DFN_QFN:QFN-20-1EP_4x4mm_P0.5mm_EP2.5x2.5mm, symbol pdu:LTC4012IUFPBF
- removed U13: ~, Package_SO:SOIC-8_3.9x4.9mm_P1.27mm, symbol pdu:SI4835BDY-T1-E3
- removed U15: ~, Package_SO:SOIC-8_3.9x4.9mm_P1.27mm, symbol pdu:AO4818B
- removed U19, U20: INA219AxD, Package_SO:SOIC-8_3.9x4.9mm_P1.27mm, symbol Sensor_Energy:INA219AxD
- added C27: 0.1uF, Capacitor_SMD:C_0805_2012Metric, symbol Device:C
- added C28: 20uF, Capacitor_SMD:C_0805_2012Metric, symbol Device:C
- added C52, C53, C55, C56: 10uF, Capacitor_SMD:C_0805_2012Metric, symbol Device:C
- added C54: 47nF, Capacitor_SMD:C_0805_2012Metric, symbol Device:C
- added C57: 1uF, Capacitor_SMD:C_0805_2012Metric, symbol Device:C
- added D18: 1N4148, Diode_SMD:D_SOD-123, symbol Device:D
- added D19, D20: 150060RS75000, LED_SMD:LED_0603_1608Metric, symbol Device:LED
- added D7: 150060VS75000, LED_SMD:LED_0603_1608Metric, symbol Device:LED
- added J10, J14, J9: Conn_01x02, Connector_PinHeader_1.00mm:PinHeader_1x02_P1.00mm_Horizontal, symbol Connector_Generic:Conn_01x02
- added J15, J3, J4, J5, J6, J8: Conn_01x02, Connector_Molex:Molex_CLIK-Mate_502382-0270_1x02-1MP_P1.25mm_Vertical, symbol Connector_Generic:Conn_01x02
- added L5: AIML-0805-1RO, Inductor_SMD:L_0805_2012Metric, symbol Device:L
- added L6: TBD, Inductor_SMD:L_Vishay_IHLP-2525, symbol Device:L
- added R16: 10k, Resistor_SMD:R_0603_1608Metric, symbol Device:R
- added R29: 3.16k, Resistor_SMD:R_0805_2012Metric, symbol Device:R
- added R60, R65: TBD, Resistor_SMD:R_0603_1608Metric, symbol Device:R
- added R61, R62, R64: TBD, Resistor_SMD:R_0805_2012Metric, symbol Device:R
- added U11: ~, Package_DFN_QFN:VQFN-24-1EP_4x4mm_P0.5mm_EP2.5x2.5mm, symbol pdu:BQ25883RGER
- added U19: LT3652EDD, Package_DFN_QFN:DFN-12-1EP_3x3mm_P0.45mm_EP1.65x2.38mm, symbol Battery_Management:LT3652EDD
- C41: value 1uF -> 20uF
- C42: value 1uF -> 22uF
- C48: value 0.1UF -> 1uF; footprint Capacitor_SMD:C_0402_1005Metric -> Capacitor_SMD:C_0805_2012Metric
- C49: value 0.1UF -> 4.7uF; footprint Capacitor_SMD:C_0402_1005Metric -> Capacitor_SMD:C_0805_2012Metric
- D11, D12: value PMEG10020ELRX -> CMSH3-40MA; footprint Diode_SMD:Nexperia_CFP3_SOD-123W -> Diode_SMD:D_SMA
- H1, H2, H3, H4: footprint MountingHole:MountingHole_3.2mm_M3_Pad -> MountingHole:MountingHole_3.2mm_M3_Pad_TopBottom
- R31: value 3k -> 0
- R33: value 26.7k -> 0
- R34: value 1 -> 0
- R42: value 10 -> 5.23k
- R44: value 10 -> 30.1k
- R45: value 2m -> 10k; footprint Resistor_SMD:R_2512_6332Metric -> Resistor_SMD:R_0805_2012Metric
- R46: value 10 -> 165m; footprint Resistor_SMD:R_0805_2012Metric -> Resistor_SMD:R_2816_7142Metric
- R49: value 2m -> TBD; footprint Resistor_SMD:R_2512_6332Metric -> Resistor_SMD:R_0805_2012Metric
- R50: value 10 -> TBD
- R58: footprint Resistor_SMD:R_2512_6332Metric -> Package_TO_SOT_SMD:TO-263-2
Connections:
- net EDFA_5V_SWITCHED is gone; now on net EDFA_5V_SW: C14.1, D4.2 (A), TP4.1, U3.1 (V_OUT1), U3.8 (V_OUT2)
- net SOLAR_IN_5 is gone; now on net THM: R42.1, R45.2
- net V_USB is gone; now on net V_BUS: C16.2, J7.A4 (VBUS), J7.A9 (VBUS), J7.B4 (VBUS), J7.B9 (VBUS)
- net BATT_CS: now also J4.1 (Pin_1)
- net BATT_PRE_INH: now also C42.2, J1.5 (Pin_5), J1.6 (Pin_6), J1.7 (Pin_7), J1.8 (Pin_8), C27.2, J4.2 (Pin_2), J9.1 (Pin_1)
- net CHRG: now also R60.2, U19.4 (~{CHRG})
- net D+: now also U11.24 (D+)
- net D-: now also U11.1 (D-)
- net GND: now also R15.2, R31.2, R33.2, R34.2, J10.2 (Pin_2), J15.2 (Pin_2), J5.2 (Pin_2), J6.2 (Pin_2), J8.2 (Pin_2); no longer C1.1, C11.2, C12.1, C19.1, C20.1, C23.2, C24.1, C3.1, C4.1, C48.1, C49.1, C6.2, C7.1, C8.1, R2.2, R33.1, R4.1, R5.2, R6.1, R7.2, R9.1, U1.17 (GND), U1.7 (GND), U1.8 (GND), U2.17 (GND), U2.7 (GND), U2.8 (GND), U6.17 (GND), U6.7 (GND), U6.8 (GND)
- net GND_REF: now also C41.2, C42.1, C48.2, C49.1, R44.1, R45.1, C27.1, C28.2, C52.2, C53.2, J10.1 (Pin_1), J6.1 (Pin_1), R29.2, U11.19 (GND), U11.20 (GND), U11.25 (GND)
- net KAPTON_PWR: now also J15.1 (Pin_1)
- net PERIPH_PWR: no longer C48.2, C49.2
- net SCL: now also U11.5 (SCL)
- net SDA: now also U11.4 (SDA)
- net SOLAR_PRE_INH: now also J3.1 (Pin_1); no longer D11.1 (K), D12.1 (K)
- net SOLAR_PRE_MPPT: now also R49.1, C55.2, D19.2 (A), D20.2 (A), J3.2 (Pin_2), U19.1 (V_{IN}); no longer R31.1
- net SW: now also C54.2, L5.1, U11.16 (SYS), U11.17 (SW), U11.18 (SW)
- net V_BATT: now also D11.1 (K), J14.1 (Pin_1); no longer R34.2
- net sol_2_diode: now reaches D8.2 (A), R52.1, R53.1
- net GNDA: now reaches R15.1
- net GNDA: now also C1.1, C11.2, C12.1, C19.1, C20.1, C23.2, C24.1, C3.1, C4.1, C6.2, C7.1, C8.1, D12.2 (A), R2.2, R31.1, R33.1, R34.1, R4.1, R5.2, R50.2, R6.1, R7.2, R9.1, U1.17 (GND), U1.7 (GND), U1.8 (GND), U2.17 (GND), U2.7 (GND), U2.8 (GND), U6.17 (GND), U6.7 (GND), U6.8 (GND), C55.1, C56.2, R61.2, U19.13 (GND), U19.6 (TIMER)
- net sol_1_diode: now reaches D9.2 (A), R55.1, R56.1
- net sol_3_diode: now reaches D10.2 (A), R43.1, R48.1
- net b1: now reaches U7.1 (D2), U7.2 (D3), U7.5 (D4), U7.6 (D1)
- net b1: now also J5.1 (Pin_1)
- net b2: now reaches U8.1 (D2), U8.2 (D3), U8.5 (D4), U8.6 (D1)
- net b2: now also J8.1 (Pin_1)
- net CS_SOL4_VIN+ renamed THM
- net THM: now also U11.7 (TS); no longer C41.2
- net CS_SOL4_VIN- renamed USB_RBF
- net USB_RBF: now also C28.1, J14.2 (Pin_2), U11.15 (SYS), U11.16 (SYS); no longer R50.2
- net CS_SOL5_VIN+ renamed V_BUS
- net V_BUS: now also C48.1, U11.23 (VBUS); no longer C42.2
- net CS_SOL5_VIN- renamed OUT
- net OUT: now also D11.2 (A), C56.1, D18.2 (A), R62.1, U19.9 (BAT); no longer C42.1
- net SOLAR_IN_1 renamed SOLAR_IN_-Z
- net SOLAR_IN_2 renamed SOLAR_IN_+Y
- net SOLAR_IN_3 renamed SOLAR_IN_-Y
- net SOLAR_IN_4: no longer names the net of R49.2
- net SOLAR_IN_4: now also R50.1, U19.2 (V_{IN_REG}); no longer R44.1
- net SOLAR_TMP_1 renamed SOLAR_TMP_-Y
- net SOLAR_TMP_-Y: now also J13.3 (Pin_3); no longer J11.3 (Pin_3)
- net SOLAR_TMP_2 renamed SOLAR_TMP_+Y
- net SOLAR_TMP_+Y: now also J1.48 (Pin_48); no longer J1.49 (Pin_49)
- removed net SOLAR_TMP_3: J1.48 (Pin_48), J13.3 (Pin_3)
- new net: C54.1, U11.12 (BTST)
- new net: C57.1, D18.1 (K), U19.11 (BOOST)
- new net: R64.1, U19.7 (V_{FB})
- new net: D19.1 (K), R60.1
- new net: D7.1 (K), U11.2 (STAT)
- new net: R29.1, U11.8 (ILIM)
- new net: R61.1, R62.2, R64.2
- new net: D20.1 (K), R65.1
- new net: D7.2 (A), R16.1
- new net CHRG_RBF: C52.1, J9.2 (Pin_2), U11.13 (BAT), U11.14 (BAT)
- new net FAULT: R65.2, U19.5 (~{FAULT})
- new net PMID: C53.1, L5.2, U11.21 (PMID), U11.22 (PMID)
- new net REGN: C49.2, R16.2, U11.11 (REGN)
- new net SENSE: L6.1, R46.1, U19.10 (SENSE)
- new net SOLAR_TMP_-Z: J1.49 (Pin_49), J11.3 (Pin_3)
- new net SW_CHRG: C57.2, D12.1 (K), L6.2, U19.12 (SW)
- no-connect marks 37 -> 35
Other:
- note added: "Battery Float Voltage Divider"
- note added: "I_chrg = 0.6 A"
- note added: "MPPT Divider"
- note added: "R = 100mV / I_chrg"
- note added: "Sense Resistor"
- moved on the sheet: C16, R17, R18

Commit message: PDU 3.0.0
Parts:
- added TP6: ~, TestPoint:TestPoint_Pad_2.0x2.0mm, symbol Connector:TestPoint
- J10, J14, J9: footprint Connector_PinHeader_1.00mm:PinHeader_1x02_P1.00mm_Horizontal -> Connector_PinHeader_2.54mm:PinHeader_1x02_P2.54mm_Horizontal
Connections:
- net SOLAR_TMP_5 is gone; now on net PDU_TEMP: J2.2 (Pin_2)
- net 3V3_BUS: no longer C12.2, C29.1, C9.2, D3.2 (A), L2.2, R8.2, TP2.1, U14.2 (V_IN1), U14.3 (V_INS), U14.6 (V_IN3), U14.7 (V_IN2), U2.14 (BIAS)
- net 3V3_BUS_STAT: no longer U2.15 (PG)
- net 5V_BUS: no longer C17.1, C21.2, C24.2, C25.1, D1.2 (A), L3.2, R10.2, TP1.1, U10.2 (V_IN1), U10.3 (V_INS), U10.6 (V_IN3), U10.7 (V_IN2), U6.14 (BIAS), U9.2 (V_IN1), U9.3 (V_INS), U9.6 (V_IN3), U9.7 (V_IN2)
- net 5V_BUS_STAT: no longer U6.15 (PG)
- net 5V_SW_1: no longer C26.1, D6.2 (A), TP7.1, U10.1 (V_OUT1), U10.8 (V_OUT2)
- net 5V_SW_1_EN: no longer U10.4 (EN)
- net BATT_CS: now also R57.1, R58.2; no longer R58.1, R59.1
- net CHRG: no longer U19.4 (~{CHRG})
- net EDFA_5V_SW: no longer C14.1, D4.2 (A), TP4.1, U3.1 (V_OUT1), U3.8 (V_OUT2)
- net EDFA_ENABLE: now also J1.15 (Pin_15); no longer J1.13 (Pin_13), U3.4 (EN)
- net FAULT: no longer U19.5 (~{FAULT})
- net GNDA: now also C20.2; no longer C20.1
- net GND_REF: now also J1.10 (Pin_10), J1.11 (Pin_11), J1.12 (Pin_12), J1.9 (Pin_9)
- net KAPTON_ENABLE: now also J1.13 (Pin_13); no longer J1.11 (Pin_11), U9.4 (EN)
- net KAPTON_PWR: now also TP6.1
- net PERIPH_EN: no longer U14.4 (EN)
- net PERIPH_PWR: no longer C30.1, C45.2, C46.2, C47.2, C50.2, D13.2 (A), TP5.1, U14.1 (V_OUT1), U14.8 (V_OUT2), U16.5 (VS), U17.5 (VS), U18.5 (VS), U21.5 (VS)
- net V_BATT: now also C20.1, J2.45 (Pin_45), R58.1, R59.1; no longer C20.2, R57.1, R58.2
- net SOLAR_TMP_4: no longer names the net of J2.1 (Pin_1)
- new net 3V3: C12.2, C29.1, C9.2, D3.2 (A), L2.2, R8.2, TP2.1, U14.2 (V_IN1), U14.3 (V_INS), U14.6 (V_IN3), U14.7 (V_IN2), U2.14 (BIAS)
- new net 3V3_S: C30.1, C45.2, C46.2, C47.2, C50.2, D13.2 (A), TP5.1, U14.1 (V_OUT1), U14.8 (V_OUT2), U16.5 (VS), U17.5 (VS), U18.5 (VS), U21.5 (VS)
- new net 3V3_STAT: U2.15 (PG)
- new net 3V3_S_EN: U14.4 (EN)
- new net 5V: C17.1, C21.2, C24.2, C25.1, D1.2 (A), L3.2, R10.2, TP1.1, U10.2 (V_IN1), U10.3 (V_INS), U10.6 (V_IN3), U10.7 (V_IN2), U6.14 (BIAS), U9.2 (V_IN1), U9.3 (V_INS), U9.6 (V_IN3), U9.7 (V_IN2)
- new net 5V_S: C26.1, D6.2 (A), TP7.1, U10.1 (V_OUT1), U10.8 (V_OUT2)
- new net 5V_STAT: U6.15 (PG)
- new net 5V_S_EN: U10.4 (EN)
- new net EDFA_5V_EN: U3.4 (EN)
- new net EDFA_5V_S: C14.1, D4.2 (A), TP4.1, U3.1 (V_OUT1), U3.8 (V_OUT2)
- new net KAPTON_EN: U9.4 (EN)
- new net ~{CHRG}: U19.4 (~{CHRG})
- new net ~{FAULT}: U19.5 (~{FAULT})
- no-connect marks 35 -> 70
Other:
- note added: "+Y Panel"
- note added: "-Y Panel"
- note added: "-Z Panel"
- note added: "2512 (5W)"
- note added: "2A max current per switch"
- note added: "3V3 Regulator"
- note added: "ALL COMPONENTS ARE 0805 UNLESS OTHERWISE SPECIFIED"
- note added: "Analog Ground Jumpers"
- note added: "Batt Heat"
- note added: "Battery Charging"
- note added: "CHRG"
- note added: "Current/Voltage Sensors"
- note added: "EDFA Regulator"
- note added: "GND"
- note added: "High-Side"
- note added: "Inhibits"
- note added: "Input Voltage Filtering"
- note added: "Low-Side"
- note added: "Power Switches"
- note added: "RBF Pins"
- note added: "Solar Panel Inputs"
- note added: "TO-263 (35W)"
- note added: "Temperature Sensor"
- note added: "USB"
- note added: "Voltage Regulators"
- note added: "output in celsius"
- note added: "reference: Artemis Kit PDU v02"
- note added: "reference: PyCubed Mainboard v05"
- note removed: "3V3 Voltage Regulator"
- note removed: "Connectors"
- note removed: "EDFA Voltage Regulator"
- note removed: "Mechanical Inhibits"
- note removed: "Temp Sensor"
- company: (none) -> UChicago Space Program
- title: (none) -> PULSE-A Power Distribution Unit (PDU)
- moved on the sheet: C1, C10, C11, C12, C13, C14, C15, C16, C17, C18, C19, C2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

Commit message: feat: Batt Board v2, PDU v3 in progress; refactor: various cleanups
Parts:
- removed C40, C43, C44: 1uF, Capacitor_SMD:C_0805_2012Metric, symbol Device:C
- removed R34: 0, Resistor_SMD:R_0805_2012Metric, symbol Device:R
- removed R47, R48, R51, R53, R54, R56: 10, Resistor_SMD:R_0805_2012Metric, symbol Device:R
- removed R58: 2m, Package_TO_SOT_SMD:TO-263-2, symbol Device:R
- added C31, C32, C33: 1uF, Capacitor_SMD:C_0603_1608Metric, symbol Device:C
- added R32, R35, R36, R37, R38, R39: 10, Resistor_SMD:R_0603_1608Metric, symbol Device:R
- C1, C11, C13, C14, C15, C17, C18, C19, C20, C23, C25, C26, C29, C30, C4, C45, C46, C47, C50, C6, C7, C8: footprint Capacitor_SMD:C_0402_1005Metric -> Capacitor_SMD:C_0603_1608Metric
- C49, C51: footprint Capacitor_SMD:C_0805_2012Metric -> Capacitor_SMD:C_0603_1608Metric
- D13, D4, D5, D6: value 150060RS75000 -> 150060AS75000
- J11, J12, J13: footprint Connector_Molex:Molex_CLIK-Mate_502382-0470_1x04-1MP_P1.25mm_Vertical -> Connector_Molex:Molex_Pico-Lock_205338-0004_1x04-1MP_P2.00mm_Horizontal
- J15, J3, J4, J5, J6, J8: footprint Connector_Molex:Molex_CLIK-Mate_502382-0270_1x02-1MP_P1.25mm_Vertical -> Connector_Molex:Molex_Pico-Lock_205338-0002_1x02-1MP_P2.00mm_Horizontal
- L6: footprint Inductor_SMD:L_Vishay_IHLP-2525 -> Inductor_SMD:L_0805_2012Metric
- R1, R29, R42, R44, R45, R57, R59: footprint Resistor_SMD:R_0805_2012Metric -> Resistor_SMD:R_0603_1608Metric
- R2, R5, R7: footprint Capacitor_SMD:C_0402_1005Metric -> Resistor_SMD:R_0603_1608Metric
- R30: value 150 -> 65
- R33: value 0 -> 2m; footprint Resistor_SMD:R_0805_2012Metric -> Resistor_SMD:R_2512_6332Metric
- R46: footprint Resistor_SMD:R_2816_7142Metric -> Resistor_SMD:R_0805_2012Metric
- TP1, TP2, TP3: footprint TestPoint:TestPoint_Pad_2.0x2.0mm -> TestPoint:TestPoint_Keystone_5000-5004_Miniature
- U7, U8: symbol pdu:SI4835DDV -> pdu:SI3407DV-T1-GE3
Connections:
- net 5V_BUS is gone; now on net 5V: J2.25 (Pin_25), J2.26 (Pin_26)
- net 5V_SW_1 is gone; now on net 5V_S: J1.21 (Pin_21)
- net 5V_SW_1_EN is gone; now on net 5V_S_EN: J1.31 (Pin_31)
- net EDFA_5V_SW is gone; now on net EDFA_5V_S: J2.21 (Pin_21), J2.22 (Pin_22)
- net ICL is gone; now on net FAULT: J1.22 (Pin_22)
- net KAPTON_ENABLE is gone; now on net KAPTON_EN: J1.13 (Pin_13)
- net 3V3: now also C15.2, J2.27 (Pin_27), J2.28 (Pin_28), U4.5 (SHUTDOWN), U4.8 (V_IN)
- net 3V3_BUS: no longer J2.27 (Pin_27), J2.28 (Pin_28)
- net BATT_CS: now also J4.2 (Pin_2), R33.1; no longer J4.1 (Pin_1)
- net CS_SOL1_VIN+: now also C33.2, R32.1
- net CS_SOL1_VIN-: now also C33.1, R35.1
- net CS_SOL2_VIN+: now also C32.2, R36.1
- net CS_SOL2_VIN-: now also C32.1, R37.1
- net CS_SOL3_VIN+: now also C31.2, R38.1
- net CS_SOL3_VIN-: now also C31.1, R39.1
- net GND: now also C1.1, C11.2, C12.1, C19.1, C20.2, C23.2, C24.1, C3.1, C4.1, C6.2, C7.1, C8.1, R2.2, R4.1, R5.2, R6.1, R7.2, R9.1, U1.17 (GND), U1.7 (GND), U1.8 (GND), U2.17 (GND), U2.7 (GND), U2.8 (GND), U6.17 (GND), U6.7 (GND), U6.8 (GND); no longer R33.2
- net GNDA: no longer C1.1, C11.2, C12.1, C19.1, C20.2, C23.2, C24.1, C3.1, C4.1, C6.2, C7.1, C8.1, R2.2, R33.1, R4.1, R5.2, R6.1, R7.2, R9.1, U1.17 (GND), U1.7 (GND), U1.8 (GND), U2.17 (GND), U2.7 (GND), U2.8 (GND), U6.17 (GND), U6.7 (GND), U6.8 (GND)
- net PERIPH_PWR: no longer C15.2, U4.5 (SHUTDOWN), U4.8 (V_IN)
- net SHDN: now also U19.3 (~{SHDN})
- net SOLAR_IN_+Y: now also R36.2
- net SOLAR_IN_-Y: now also R38.2
- net SOLAR_IN_-Z: now also R32.2
- net V_BATT: now also R33.2
- net sol_1_diode: now also R35.2
- net sol_2_diode: now also R37.2
- net sol_3_diode: now also R39.2
- net BATT_PRE_INH renamed RAW_BATT
- net RAW_BATT: no longer C27.2, C42.2, J4.2 (Pin_2), J9.1 (Pin_1)
- net EDFA_ENABLE renamed EDFA_EN
- new net BATT_RAW: C27.2, C42.2, J4.1 (Pin_1), J9.1 (Pin_1)
- no-connect marks 70 -> 69

Commit message: feat: PDU 3.0.0 & laser driving basics
Parts:
- removed C16: 4.7uF, Capacitor_SMD:C_0805_2012Metric, symbol Device:C
- removed C28, C41: 20uF, Capacitor_SMD:C_0805_2012Metric, symbol Device:C
- removed C48, C57: 1uF, Capacitor_SMD:C_0805_2012Metric, symbol Device:C
- removed C49: 4.7uF, Capacitor_SMD:C_0603_1608Metric, symbol Device:C
- removed C52, C53, C55, C56: 10uF, Capacitor_SMD:C_0805_2012Metric, symbol Device:C
- removed C54: 47nF, Capacitor_SMD:C_0805_2012Metric, symbol Device:C
- removed D11, D12: CMSH3-40MA, Diode_SMD:D_SMA, symbol Device:D_Schottky
- removed D18: 1N4148, Diode_SMD:D_SOD-123, symbol Device:D
- removed D19, D20: 150060RS75000, LED_SMD:LED_0603_1608Metric, symbol Device:LED
- removed J10, J14, J9: Conn_01x02, Connector_PinHeader_2.54mm:PinHeader_1x02_P2.54mm_Horizontal, symbol Connector_Generic:Conn_01x02
- removed J7: USB_C_Receptacle_USB2.0_14P, Connector_USB:USB_C_Receptacle_GCT_USB4105-xx-A_16P_TopMnt_Horizontal, symbol Connector:USB_C_Receptacle_USB2.0_14P
- removed L5: AIML-0805-1RO, Inductor_SMD:L_0805_2012Metric, symbol Device:L
- removed L6: TBD, Inductor_SMD:L_0805_2012Metric, symbol Device:L
- removed R15: 0, Resistor_SMD:R_0805_2012Metric, symbol Device:R
- removed R18: 5.1k, Resistor_SMD:R_0805_2012Metric, symbol Device:R
- removed R29: 3.16k, Resistor_SMD:R_0603_1608Metric, symbol Device:R
- removed R42: 5.23k, Resistor_SMD:R_0603_1608Metric, symbol Device:R
- removed R44: 30.1k, Resistor_SMD:R_0603_1608Metric, symbol Device:R
- removed R45: 10k, Resistor_SMD:R_0603_1608Metric, symbol Device:R
- removed R46: 165m, Resistor_SMD:R_0805_2012Metric, symbol Device:R
- removed R49, R50, R61, R62, R64: TBD, Resistor_SMD:R_0805_2012Metric, symbol Device:R
- removed R60, R65: TBD, Resistor_SMD:R_0603_1608Metric, symbol Device:R
- removed TP4, TP5, TP6, TP7: ~, TestPoint:TestPoint_Pad_2.0x2.0mm, symbol Connector:TestPoint
- removed U11: ~, Package_DFN_QFN:VQFN-24-1EP_4x4mm_P0.5mm_EP2.5x2.5mm, symbol pdu:BQ25883RGER
- removed U19: LT3652EDD, Package_DFN_QFN:DFN-12-1EP_3x3mm_P0.45mm_EP1.65x2.38mm, symbol Battery_Management:LT3652EDD
- added C34: 4.7uF, Capacitor_SMD:C_1206_3216Metric, symbol Device:C
- added C35: 4.7uF, Capacitor_Tantalum_SMD:CP_EIA-3528-12_Kemet-T, symbol Device:C
- added D11: 150060VS75000, LED_SMD:LED_0603_1608Metric, symbol Device:LED
- added R34: 549k, Resistor_SMD:R_0603_1608Metric, symbol Device:R
- added R40: 459k, Resistor_SMD:R_0603_1608Metric, symbol Device:R
- added R41: 0, Resistor_SMD:R_0603_1608Metric, symbol Device:R
- added U12: LTM8062AIV-PBF, PDU:LGA-77, symbol pdu:LTM8062AIV-PBF
- R16: value 10k -> 150
- R17: value 5.1k -> 150; footprint Resistor_SMD:R_0805_2012Metric -> Resistor_SMD:R_0603_1608Metric
- R31: value 0 -> 549k; footprint Resistor_SMD:R_0805_2012Metric -> Resistor_SMD:R_0603_1608Metric
Connections:
- net 3V3_BUS is gone; now on net 3V3: J11.2 (Pin_2), J12.2 (Pin_2), J13.2 (Pin_2)
- net 3V3_BUS_STAT is gone; now on net 3V3_STAT: J2.24 (Pin_24)
- net 5V_BUS_STAT is gone; now on net 5V_STAT: J2.23 (Pin_23)
- net GNDA is gone; now on net BATT_THERM_R: R31.1
- net RAW_BATT is gone; now on net VBATT_IN: J1.5 (Pin_5), J1.6 (Pin_6), J1.7 (Pin_7), J1.8 (Pin_8)
- net REGN is gone; now on an unnamed net: R16.2
- net 3V3_S: now also J1.34 (Pin_34), J2.33 (Pin_33)
- net 3V3_S_EN: now also J1.39 (Pin_39)
- net 5V_S: now also J1.45 (Pin_45), J1.46 (Pin_46); no longer J1.21 (Pin_21)
- net CHRG: now also D7.2 (A), U12.K7 (*CHRG)
- net EDFA_5V_EN: now also J1.40 (Pin_40)
- net EDFA_5V_S: now also J1.42 (Pin_42), J1.44 (Pin_44); no longer J2.21 (Pin_21), J2.22 (Pin_22)
- net FAULT: now also D11.2 (A), U12.J7 (*FAULT)
- net GND: now also R16.1, R17.1, U17.2 (A0), U18.2 (A0), C34.1, C35.1, R40.1, U12.A1 (GND), U12.A2 (GND), U12.A3 (GND), U12.A4 (GND), U12.A5 (GND), U12.B1 (GND), U12.B2 (GND), U12.B3 (GND), U12.B4 (GND), U12.B5 (GND), U12.C1 (GND), U12.C2 (GND), U12.C3 (GND), U12.C4 (GND), U12.C5 (GND), U12.D1 (GND), U12.D2 (GND), U12.D3 (GND), U12.D4 (GND), U12.D5 (GND), U12.E1 (GND), U12.E2 (GND), U12.E3 (GND), U12.E4 (GND), U12.E5 (GND), U12.F1 (GND), U12.F2 (GND), U12.F3 (GND), U12.F4 (GND), U12.F5 (GND), U12.G1 (GND), U12.G2 (GND), U12.G3 (GND), U12.G4 (GND), U12.G5 (GND), U12.G6 (GND), U12.H1 (GND), U12.H2 (GND), U12.H3 (GND), U12.H4 (GND), U12.H5 (GND), U12.J1 (GND), U12.J2 (GND), U12.J3 (GND), U12.J4 (GND), U12.J5 (GND), U12.J6 (TMR), U12.L7 (GND); no longer R31.2, U18.1 (A1)
- net GND_REF: no longer R17.2
- net KAPTON_EN: now also J1.37 (Pin_37); no longer J1.13 (Pin_13)
- net SCL: now also U16.2 (A0)
- net SDA: now also U18.1 (A1); no longer U16.2 (A0), U17.2 (A0), U18.2 (A0)
- net SOLAR_PRE_MPPT: now also R41.1, U12.K4 (VINA), U12.K5 (VINA), U12.K6 (RUN), U12.L4 (VINA), U12.L5 (VINA)
- net ADJ: now reaches J1.36 (Pin_36)
- net ADJ: now also R31.2, R34.1, R40.2, U12.H7 (ADJ)
- net BATT_THERM_R: now reaches J1.38 (Pin_38)
- net BATT_RAW renamed VBATT_IN
- net EDFA_EN: no longer names the net of J1.15 (Pin_15)
- net PERIPH_EN: no longer names the net of J1.27 (Pin_27)
- net PERIPH_PWR: no longer names the net of J1.47 (Pin_47)
- net SHDN: no longer names the net of J1.26 (Pin_26)
- net V_BATT renamed VBATT
- net VBATT: now also C35.2, R34.2, U12.A6 (BAT), U12.A7 (BAT), U12.B6 (BAT), U12.B7 (BAT), U12.C6 (BAT), U12.C7 (BAT), U12.D6 (BAT), U12.D7 (BAT), U12.E6 (BAT), U12.E7 (BAT), U12.F6 (BAT), U12.F7 (BAT), U12.G7 (BIAS)
- new net: D11.1 (K), R17.2
- new net CHARGE_VIN: C34.2, U12.K1 (VIN), U12.K2 (VIN), U12.K3 (VIN), U12.L1 (VIN), U12.L2 (VIN), U12.L3 (VIN)
- new net VIN_REG: R41.2, U12.L6 (VINREG)
- no-connect marks 69 -> 68
Other:
- note added: "ALL COMPONENTS ARE 0603 UNLESS OTHERWISE SPECIFIED"
- note added: "I2C Address: 0x40"
- note added: "I2C Address: 0x42"
- note added: "I2C Address: 0x43"
- note added: "I2C Address: 0x48"
- note added: "To Be Integrated into v4 (alongside USB charging)"
- note removed: "ALL COMPONENTS ARE 0805 UNLESS OTHERWISE SPECIFIED"
- note removed: "Analog Ground Jumpers"
- note removed: "Battery Float Voltage Divider"
- note removed: "CHRG"
- note removed: "GND"
- note removed: "I_chrg = 0.6 A"
- note removed: "MPPT Divider"
- note removed: "R = 100mV / I_chrg"
- note removed: "Sense Resistor"
- note removed: "USB"
- note removed: "USB Connector"
- moved on the sheet: C27, C42, J15, J3, J4, J6
