File: Avionics/BatteryBoard/Batt_Boardv1.kicad_sch (KiCad schematic)
At the start: 42 parts, among them J1 Conn_02x26_Odd_Even, J2 Conn_02x26_Odd_Even, Q1 IRF7458, Q2 IRF7458, U2 BQ29200DRBR, U3 TLA2024IRUGR, U4 LM35-LP, U5 LM35-LP, U6 LM35-LP, U7 LM35-LP

Commit message: batt_brd: Update battery footprints
Parts:
- BT_H_1, BT_H_2, BT_H_3, BT_L_1, BT_L_2, BT_L_3: footprint 254:BAT_254_1 -> BattBrdFtPrts:BAT_254_1
- U1: value ~ -> R5460N210AD1
Changed lines of the file:
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@@
 			)
 		)
-		(property "Footprint" "254:BAT_254_1"
+		(property "Footprint" "BattBrdFtPrts:BAT_254_1"
 			(at 202.946 42.926 0)
 			(effects
@@
 			)
 		)
-		(property "Footprint" "254:BAT_254_1"
+		(property "Footprint" "BattBrdFtPrts:BAT_254_1"
 			(at 244.856 30.226 0)
 			(effects
@@
 			)
 		)
-		(property "Footprint" "254:BAT_254_1"
+		(property "Footprint" "BattBrdFtPrts:BAT_254_1"
 			(at 202.946 30.226 0)
 			(effects
@@
 			)
 		)
-		(property "Footprint" "254:BAT_254_1"
+		(property "Footprint" "BattBrdFtPrts:BAT_254_1"
 			(at 202.946 17.526 0)
 			(effects
@@
 			)
 		)
-		(property "Value" "~"
+		(property "Value" "R5460N210AD1"
 			(at 71.12 115.57 0)
 			(effects
@@
 					(size 1.27 1.27)
 				)
+				(hide yes)
 			)
 		)
@@
 			)
 		)
-		(property "Footprint" "254:BAT_254_1"
+		(property "Footprint" "BattBrdFtPrts:BAT_254_1"
 			(at 244.856 42.926 0)
 			(effects
@@
 			)
 		)
-		(property "Footprint" "254:BAT_254_1"
+		(property "Footprint" "BattBrdFtPrts:BAT_254_1"
 			(at 244.856 17.526 0)
 			(effects

Commit message: "Finish" routing
DRC failing; will fix soon
Parts:
- C1, C2, C3, C4: footprint Capacitor_SMD:C_0603_1608Metric -> Capacitor_SMD:C_0805_2012Metric
- C5, C6, C7, C8, C9: footprint (none) -> Capacitor_SMD:C_0805_2012Metric
- R12, R7, R8, R9: footprint (none) -> Resistor_SMD:R_0805_2012Metric
Changed lines of the file:
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@@
 			)
 		)
-		(property "Footprint" ""
+		(property "Footprint" "Capacitor_SMD:C_0805_2012Metric"
 			(at 265.1252 95.25 0)
 			(effects
@@
 			)
 		)
-		(property "Footprint" ""
+		(property "Footprint" "Resistor_SMD:R_0805_2012Metric"
 			(at 192.024 76.454 90)
 			(effects
@@
 			)
 		)
-		(property "Footprint" ""
+		(property "Footprint" "Resistor_SMD:R_0805_2012Metric"
 			(at 265.176 81.534 90)
 			(effects
@@
 			)
 		)
-		(property "Footprint" ""
+		(property "Footprint" "Capacitor_SMD:C_0805_2012Metric"
 			(at 230.8352 154.94 0)
 			(effects
@@
 			)
 		)
-		(property "Footprint" ""
+		(property "Footprint" "Capacitor_SMD:C_0805_2012Metric"
 			(at 200.3552 85.09 0)
 			(effects
@@
 			)
 		)
-		(property "Footprint" "Capacitor_SMD:C_0603_1608Metric"
+		(property "Footprint" "Capacitor_SMD:C_0805_2012Metric"
 			(at 100.0252 124.46 0)
 			(effects
@@
 			)
 		)
-		(property "Footprint" "Capacitor_SMD:C_0603_1608Metric"
+		(property "Footprint" "Capacitor_SMD:C_0805_2012Metric"
 			(at 89.8652 138.43 0)
 			(effects
@@
 			)
 		)
-		(property "Footprint" ""
+		(property "Footprint" "Resistor_SMD:R_0805_2012Metric"
 			(at 192.024 101.854 90)
 			(effects
@@
 			)
 		)
-		(property "Footprint" "Capacitor_SMD:C_0603_1608Metric"
+		(property "Footprint" "Capacitor_SMD:C_0805_2012Metric"
 			(at 113.9952 124.46 0)
 			(effects
@@
 			)
 		)
-		(property "Footprint" "Capacitor_SMD:C_0603_1608Metric"
+		(property "Footprint" "Capacitor_SMD:C_0805_2012Metric"
 			(at 45.72 153.9748 0)
 			(effects
@@
 			)
 		)
-		(property "Footprint" ""
+		(property "Footprint" "Capacitor_SMD:C_0805_2012Metric"
 			(at 200.3552 92.71 0)
 			(effects
@@
 			)
 		)
-		(property "Footprint" ""
+		(property "Footprint" "Resistor_SMD:R_0805_2012Metric"
 			(at 192.024 84.074 90)
 			(effects
@@
 			)
 		)
-		(property "Footprint" ""
+		(property "Footprint" "Capacitor_SMD:C_0805_2012Metric"
 			(at 216.8652 104.14 0)
 			(effects
