File: Avionics/BatteryBoard/heater_ctrl.kicad_sch (KiCad schematic)
At the start: 16 parts, among them U10 LMV331, U11 TPS7A2601DRVR, U13 74AHC1G32, U14 74AHC1G04, U15 74LVC2G08, U8 LM4040DBZ-2.5, U9 TMP36xS

Commit message: "Finish" routing
DRC failing; will fix soon
Parts:
- C10, C11, C12, C13, C14: footprint (none) -> Capacitor_SMD:C_0805_2012Metric
- R13, R14, R15, R5: footprint (none) -> Resistor_SMD:R_0805_2012Metric
- U9: footprint Package_SO:SOIC-8_3.9x4.9mm_P1.27mm -> Package_TO_SOT_THT:TO-92_Inline
Connections:
- net +5VA: now also U9.1 (+Vs); no longer U9.8 (+Vs)
- net GNDREF: now also U9.3 (GND); no longer U9.4 (GND), U9.5 (~{SHUTDOWN})
- net at U10.3 (-): now also U9.2 (V_{OUT}); no longer U9.1 (V_{OUT})
Changed lines of the file:
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@@
 	(wire
 		(pts
-			(xy 25.4 97.79) (xy 25.4 93.98)
-		)
-		(stroke
-			(width 0)
-			(type default)
-		)
-	)
-	(wire
-		(pts
 			(xy 156.21 52.07) (xy 149.86 52.07)
 		)
@@
 	(wire
 		(pts
-			(xy 25.4 93.98) (xy 29.21 93.98)
-		)
-		(stroke
-			(width 0)
-			(type default)
-		)
-	)
-	(wire
-		(pts
 			(xy 68.58 88.9) (xy 71.12 88.9)
 		)
@@
 			)
 		)
-		(property "Footprint" "Package_SO:SOIC-8_3.9x4.9mm_P1.27mm"
+		(property "Footprint" "Package_TO_SOT_THT:TO-92_Inline"
 			(at 41.91 105.41 0)
 			(effects
@@
 			)
 		)
-		(pin "4"
+		(pin "3"
 		)
 		(pin "1"
 		)
-		(pin "5"
-		)
-		(pin "8"
+		(pin "2"
 		)
 		(instances
@@
 			)
 		)
-		(property "Footprint" ""
+		(property "Footprint" "Resistor_SMD:R_0805_2012Metric"
 			(at 58.674 45.974 90)
 			(effects
@@
 			)
 		)
-		(property "Footprint" ""
+		(property "Footprint" "Resistor_SMD:R_0805_2012Metric"
 			(at 48.514 45.974 90)
 			(effects
@@
 			)
 		)
-		(property "Footprint" ""
+		(property "Footprint" "Capacitor_SMD:C_0805_2012Metric"
 			(at 142.24 137.4648 0)
 			(effects
@@
 			)
 		)
-		(property "Footprint" ""
+		(property "Footprint" "Capacitor_SMD:C_0805_2012Metric"
 			(at 45.72 137.4648 0)
 			(effects
@@
 			)
 		)
-		(property "Footprint" ""
+		(property "Footprint" "Capacitor_SMD:C_0805_2012Metric"
 			(at 96.2152 101.6 0)
 			(effects
@@
 			)
 		)
-		(property "Footprint" ""
+		(property "Footprint" "Capacitor_SMD:C_0805_2012Metric"
 			(at 157.1752 48.26 0)
 			(effects
@@
 	)
 	(symbol
-		(lib_id "power:GNDREF")
-		(at 25.4 97.79 0)
-		(unit 1)
-		(exclude_from_sim no)
-		(in_bom yes)
-		(on_board yes)
-		(dnp no)
-		(fields_autoplaced yes)
-		(property "Reference" "#PWR019"
-			(at 25.4 104.14 0)
-			(effects
-				(font
-					(size 1.27 1.27)
-				)
-				(hide yes)
-			)
-		)
-		(property "Value" "GNDREF"
-			(at 25.4 102.87 0)
-			(effects
-				(font
-					(size 1.27 1.27)
-				)
-			)
-		)
-		(property "Footprint" ""
-			(at 25.4 97.79 0)
-			(effects
-				(font
-					(size 1.27 1.27)
-				)
-				(hide yes)
-			)
-		)
-		(property "Datasheet" ""
-			(at 25.4 97.79 0)
-			(effects
-				(font
-					(size 1.27 1.27)
-				)
-				(hide yes)
-			)
-		)
-		(property "Description" "Power symbol creates a global label with name \"GNDREF\" , reference supply ground"
-			(at 25.4 97.79 0)
-			(effects
-				(font
-					(size 1.27 1.27)
-				)
-				(hide yes)
-			)
-		)
-		(pin "1"
-		)
-		(instances
-			(project ""
-				(path "/a5e22de5-0e9e-4e3b-9cf5-d999de47cef4/704e1e38-2a40-4837-82db-8d871c4d1498"
-					(reference "#PWR019")
-					(unit 1)
-				)
-			)
-		)
-	)
-	(symbol
 		(lib_id "power:+5VA")
 		(at 95.25 80.01 0)
@@
 			)
 		)
-		(property "Footprint" ""
+		(property "Footprint" "Resistor_SMD:R_0805_2012Metric"
 			(at 96.266 85.344 90)
 			(effects
@@
 			)
 		)
-		(property "Footprint" ""
+		(property "Footprint" "Capacitor_SMD:C_0805_2012Metric"
 			(at 102.5652 50.8 0)
 			(effects
@@
 			)
 		)
-		(property "Footprint" ""
+		(property "Footprint" "Resistor_SMD:R_0805_2012Metric"
 			(at 44.704 33.274 90)
 			(effects
