File: flight-subsystem-designs/gnc/GPS-RadioPCB/SpaceManiacPCB copy.kicad_sch (KiCad schematic)
At the start: 28 parts, among them U1 LMK1C1104PWR

Commit message: Added Space Maniac final board design 27th Aug, Owen Law
Parts:
- C1, C2, C3, C4: footprint Capacitor_SMD:C_0805_2012Metric -> Capacitor_SMD:C_0402_1005Metric
- D1, D2, D3, D4, D5: value PTVS5V0Z1USK -> TVS5B5CL
- H3, H4: footprint Connector_Molex:Molex_SlimStack_54722-0604_2x30_P0.50mm_Vertical -> Connector_Molex:CON_MolexSlimStack_54363-0689
Connections:
- net 3V3_S: now also C3.1, FB1.2, H1.47 (Pin_47); no longer C1.2, C2.1, C4.2, FB1.1, R1.1, U1.6 (VDD)
- net CLK_2: now also D3.1 (K), U1.7 (Y3); no longer D4.1 (K), U1.5 (Y2)
- net CLK_3: now also D4.1 (K), U1.5 (Y2); no longer D3.1 (K), U1.7 (Y3)
- new net PWR_Fanout: C1.2, C2.1, C4.2, FB1.1, R1.1, U1.6 (VDD)
Changed lines of the file:
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@@
 	)
 	(junction
-		(at 39.37 76.2)
-		(diameter 0)
-		(color 0 0 0 0)
-	)
-	(junction
 		(at 259.08 49.53)
 		(diameter 0)
@@
 	)
 	(junction
-		(at 68.58 154.94)
+		(at 66.04 154.94)
+		(diameter 0)
+		(color 0 0 0 0)
+	)
+	(junction
+		(at 66.04 96.52)
 		(diameter 0)
 		(color 0 0 0 0)
@@
 	(wire
 		(pts
-			(xy 39.37 96.52) (xy 72.39 96.52)
-		)
-		(stroke
-			(width 0)
-			(type default)
-		)
-	)
-	(wire
-		(pts
 			(xy 85.09 38.1) (xy 91.44 38.1)
 		)
@@
 	(wire
 		(pts
+			(xy 66.04 151.13) (xy 66.04 154.94)
+		)
+		(stroke
+			(width 0)
+			(type default)
+		)
+	)
+	(wire
+		(pts
 			(xy 232.41 100.33) (xy 243.84 100.33)
 		)
@@
 	(wire
 		(pts
+			(xy 66.04 154.94) (xy 68.58 154.94)
+		)
+		(stroke
+			(width 0)
+			(type default)
+		)
+	)
+	(wire
+		(pts
 			(xy 226.06 77.47) (xy 243.84 77.47)
 		)
@@
 	(wire
 		(pts
+			(xy 66.04 96.52) (xy 72.39 96.52)
+		)
+		(stroke
+			(width 0)
+			(type default)
+		)
+	)
+	(wire
+		(pts
 			(xy 185.42 49.53) (xy 187.96 49.53)
 		)
@@
 	(wire
 		(pts
-			(xy 29.21 154.94) (xy 68.58 154.94)
+			(xy 29.21 154.94) (xy 66.04 154.94)
 		)
 		(stroke
@@
 		)
 	)
+	(label "PWR_Fanout"
+		(at 66.04 151.13 0)
+		(effects
+			(font
+				(size 1.27 1.27)
+			)
+			(justify left bottom)
+		)
+	)
 	(label "CAN2_H"
 		(at 226.06 74.93 0)
@@
 	)
 	(label "CLK_3"
-		(at 74.93 175.26 0)
+		(at 85.09 172.72 0)
 		(effects
 			(font
@@
 	)
 	(label "CLK_2"
-		(at 85.09 172.72 0)
+		(at 74.93 175.26 0)
 		(effects
 			(font
@@
 		)
 	)
+	(label "PWR_Fanout"
+		(at 39.37 76.2 0)
+		(effects
+			(font
+				(size 1.27 1.27)
+			)
+			(justify left bottom)
+		)
+	)
 	(label "I2C1_SDA"
 		(at 227.33 59.69 0)
@@
 			)
 		)
-		(property "Value" "PTVS5V0Z1USK"
+		(property "Value" "TVS5B5CL"
 			(at 63.754 179.324 90)
 			(effects
@@
 			)
 		)
-		(property "Value" "PTVS5V0Z1USK"
+		(property "Value" "TVS5B5CL"
 			(at 84.582 178.308 90)
 			(effects
@@
 	(symbol
 		(lib_id "power:+3.3V")
-		(at 68.58 154.94 0)
+		(at 39.37 96.52 180)
 		(unit 1)
 		(exclude_from_sim no)
@@
 		(dnp no)
 		(property "Reference" "#PWR013"
-			(at 68.58 158.75 0)
+			(at 39.37 92.71 0)
 			(effects
 				(font
@@
 		)
 		(property "Value" "3V3_S"
-			(at 68.58 151.13 0)
+			(at 39.37 100.33 0)
 			(effects
 				(font
@@
 		)
 		(property "Footprint" ""
-			(at 68.58 154.94 0)
+			(at 39.37 96.52 0)
 			(effects
 				(font
@@
 		)
 		(property "Datasheet" ""
-			(at 68.58 154.94 0)
+			(at 39.37 96.52 0)
 			(effects
 				(font
@@
 		)
 		(property "Description" "Power symbol creates a global label with name \"+3.3V\""
-			(at 68.58 154.94 0)
+			(at 39.37 96.52 0)
 			(effects
 				(font
@@
 			)
 		)
-		(property "Value" "PTVS5V0Z1USK"
+		(property "Value" "TVS5B5CL"
 			(at 93.726 161.29 90)
 			(effects
@@
 	(symbol
 		(lib_id "power:PWR_FLAG")
-		(at 39.37 76.2 90)
+		(at 66.04 96.52 180)
 		(unit 1)
 		(exclude_from_sim no)
@@
 		(dnp no)
 		(property "Reference" "#FLG01"
-			(at 37.465 76.2 0)
+			(at 66.04 98.425 0)
 			(effects
 				(font
@@
 		)
 		(property "Value" "PWR_FLAG"
-			(at 31.242 76.454 90)
+			(at 64.262 100.838 0)
 			(effects
 				(font
@@
 		)
 		(property "Footprint" ""
-			(at 39.37 76.2 0)
+			(at 66.04 96.52 0)
 			(effects
 				(font
@@
 		)
 		(property "Datasheet" "~"
-			(at 39.37 76.2 0)
+			(at 66.04 96.52 0)
 			(effects
 				(font
@@
 		)
 		(property "Description" "Special symbol for telling ERC where power comes from"
-			(at 39.37 76.2 0)
+			(at 66.04 96.52 0)
 			(effects
 				(font
@@
 			)
 		)
-		(property "Footprint" "Capacitor_SMD:C_0805_2012Metric"
+		(property "Footprint" "Capacitor_SMD:C_0402_1005Metric"
 			(at 45.72 83.82 0)
 			(effects
@@
 			)
 		)
-		(property "Footprint" "Capacitor_SMD:C_0805_2012Metric"
+		(property "Footprint" "Capacitor_SMD:C_0402_1005Metric"
 			(at 71.12 158.75 0)
 			(effects
@@
 			)
 		)
-		(property "Footprint" "Capacitor_SMD:C_0805_2012Metric"
+		(property "Footprint" "Capacitor_SMD:C_0402_1005Metric"
 			(at 45.72 78.74 0)
 			(effects
@@
 	(symbol
 		(lib_id "power:+3.3V")
-		(at 39.37 76.2 0)
+		(at 66.04 96.52 90)
 		(unit 1)
 		(exclude_from_sim no)
@@
 		(dnp no)
 		(property "Reference" "#PWR042"
-			(at 39.37 80.01 0)
+			(at 69.85 96.52 0)
 			(effects
 				(font
@@
 		)
 		(property "Value" "3V3_S"
-			(at 39.624 71.628 0)
+			(at 59.944 97.028 90)
 			(effects
 				(font
@@
 		)
 		(property "Footprint" ""
-			(at 39.37 76.2 0)
+			(at 66.04 96.52 0)
 			(effects
 				(font
@@
 		)
 		(property "Datasheet" ""
-			(at 39.37 76.2 0)
+			(at 66.04 96.52 0)
 			(effects
 				(font
@@
 		)
 		(property "Description" "Power symbol creates a global label with name \"+3.3V\""
-			(at 39.37 76.2 0)
+			(at 66.04 96.52 0)
 			(effects
 				(font
@@
 			)
 		)
-		(property "Footprint" "Connector_Molex:Molex_SlimStack_54722-0604_2x30_P0.50mm_Vertical"
+		(property "Footprint" "Connector_Molex:CON_MolexSlimStack_54363-0689"
 			(at 193.04 80.01 0)
 			(effects
@@
 			)
 		)
-		(property "Footprint" "Capacitor_SMD:C_0805_2012Metric"
+		(property "Footprint" "Capacitor_SMD:C_0402_1005Metric"
 			(at 45.72 92.71 0)
 			(effects
@@
 			)
 		)
-		(property "Value" "PTVS5V0Z1USK"
-			(at 14.732 179.07 90)
+		(property "Value" "TVS5B5CL"
+			(at 19.558 173.99 90)
 			(effects
 				(font
@@
 			)
 		)
-		(property "Footprint" "Connector_Molex:Molex_SlimStack_54722-0604_2x30_P0.50mm_Vertical"
+		(property "Footprint" "Connector_Molex:CON_MolexSlimStack_54363-0689"
 			(at 248.92 80.01 0)
 			(effects
@@
 			)
 		)
-		(property "Value" "PTVS5V0Z1USK"
+		(property "Value" "TVS5B5CL"
 			(at 92.202 155.194 90)
 			(effects
