File: flight-subsystem-designs/power/power-distribution/PowerDistribution.kicad_pcb (KiCad board)
At the start: 4 copper layers, 90.2 x 96 mm, 135 parts, among them J1 Conn_02x26_Odd_Even, J11 Conn_01x04, J12 Conn_01x04, J13 Conn_01x04, J15 Conn_01x02, J2 Conn_02x26_Odd_Even, J3 Conn_01x02, J4 Conn_01x02, J5 Conn_01x02, J6 Conn_01x02, J8 Conn_01x02, Q1 BC848ALT1G, Q2 IRLML2803PBFCT, Q3 IRLML2803PBFCT, U1 LT8610, U12 LTM8062AIV-PBF, U16 INA219AxD, U17 INA219AxD, U18 INA219AxD, U2 LT8610, U21 INA219AxD, U6 LT8610

Commit message: feat: PDU 3.0.1, PDU Breakout 1.0
Parts:
- added L4: AIMC-0805-2N2S-T, Inductor_SMD:L_0805_2012Metric, F.Cu at (265.6, 111.2)
- added Q4: NMOS, Package_TO_SOT_SMD:TSOT-23, F.Cu at (260.9, 107.5)
- added Q5: NMOS, Package_TO_SOT_SMD:TSOT-23, F.Cu at (260.9, 112.2)
- added R15: 1M, Resistor_SMD:R_0603_1608Metric, F.Cu at (265.6, 106.4)
- added R18: 1M, Resistor_SMD:R_0603_1608Metric, F.Cu at (265.6, 108.9)
- added U11: ~, Package_DFN_QFN:Texas_RGW0020A_VQFN-20-1EP_5x5mm_P0.65mm_EP3.15x3.15mm_ThermalVias, F.Cu at (260.3, 90.1)
- added U13: ~, Package_DFN_QFN:DFN-8-1EP_6x5mm_P1.27mm_EP2x2mm, F.Cu at (261.4, 98.1)
- C24: value 47uF -> 68uF
- L3: value 4.7uH -> 10uH
- R2, R7: value 18.2k -> 110k
Connections:
- J4 pad 1: /VBATT_IN -> /VBATT_PRE_INH
