File: flight-subsystem-designs/power/power-distribution/PowerDistribution.kicad_sch (KiCad schematic)
At the start: 134 parts, among them J1 Conn_02x26_Odd_Even, J11 Conn_01x04, J12 Conn_01x04, J13 Conn_01x04, J15 Conn_01x02, J2 Conn_02x26_Odd_Even, J3 Conn_01x02, J4 Conn_01x02, J5 Conn_01x02, J6 Conn_01x02, J8 Conn_01x02, Q1 BC848ALT1G, Q2 IRLML2803PBFCT, Q3 IRLML2803PBFCT, U1 LT8610, U12 LTM8062AIV-PBF, U16 INA219AxD, U17 INA219AxD, U18 INA219AxD, U2 LT8610, U21 INA219AxD, U6 LT8610

Commit message: feat: PDU 3.0.1, PDU Breakout 1.0
Parts:
- added J7: Conn_01x02, symbol Connector_Generic:Conn_01x02
- added L4: AIMC-0805-2N2S-T, Inductor_SMD:L_0805_2012Metric, symbol Device:L
- added Q4, Q5: NMOS, Package_TO_SOT_SMD:TSOT-23, symbol Simulation_SPICE:NMOS
- added R15, R18: 1M, Resistor_SMD:R_0603_1608Metric, symbol Device:R
- added R29: 50k, Resistor_SMD:R_0603_1608Metric, symbol Device:R
- added R42: TBD, Resistor_SMD:R_0603_1608Metric, symbol Device:R
- added U11: ~, Package_DFN_QFN:Texas_RGW0020A_VQFN-20-1EP_5x5mm_P0.65mm_EP3.15x3.15mm_ThermalVias, symbol pdu:TPS281C30
- added U13: ~, Package_DFN_QFN:DFN-8-1EP_6x5mm_P1.27mm_EP2x2mm, symbol pdu:MR25H256ACDF
- C12, C3: footprint Capacitor_SMD:C_0805_2012Metric -> Capacitor_SMD:C_1206_3216Metric
- C24: value 47uF -> 68uF
- L3: value 4.7uH -> 10uH
- R11: footprint Resistor_SMD:R_0603_1608Metric -> Capacitor_SMD:C_1206_3216Metric
- R2, R7: value 18.2k -> 110k
- R33: value 2m -> 10m
- R43, R52, R55: value 2m -> 40m
Connections:
- net 3V3: now also U13.8 (VDD); no longer J11.2 (Pin_2), J12.2 (Pin_2), J13.2 (Pin_2)
- net CHRG: no longer D7.2 (A), U12.K7 (*CHRG)
- net FAULT: no longer D11.2 (A), U12.J7 (*FAULT)
- net GND: now also J11.1 (Pin_1), J12.1 (Pin_1), J13.1 (Pin_1), L4.1, R29.2, R42.1, U11.18 (GND), U13.4 (GND)
- net SOLAR_IN_+Y: now also J12.2 (Pin_2), J12.3 (Pin_3); no longer J12.1 (Pin_1)
- net SOLAR_IN_-Y: now also J13.2 (Pin_2), J13.3 (Pin_3); no longer J13.1 (Pin_1)
- net SOLAR_IN_-Z: now also J11.2 (Pin_2), J11.3 (Pin_3); no longer J11.1 (Pin_1)
- net SOLAR_TMP_+Y: no longer J12.3 (Pin_3)
- net SOLAR_TMP_-Y: no longer J13.3 (Pin_3)
- net SOLAR_TMP_-Z: no longer J11.3 (Pin_3)
- net VBATT: now also U11.10 (VS), U11.11 (VS), U11.12 (VS), U11.13 (VS)
- net VBATT_IN: now also J7.1 (Pin_1), Q5.1 (D), R18.2; no longer J4.1 (Pin_1)
- new net: L4.2, Q4.3 (S), R15.1
- new net: Q4.1 (D), Q5.2 (G), R18.1
- new net: R29.1, U11.1 (ILIM)
- new net ADCS_PWR: U11.3 (VOUT), U11.4 (VOUT), U11.5 (VOUT), U11.6 (VOUT)
- new net ADCS_PWR_DIAG: U11.16 (DIAG_EN)
- new net ADCS_PWR_EN: U11.15 (EN)
- new net ADCS_PWR_SNS: R42.2, U11.20 (SNS)
- new net HOLD: U13.7 (HOLD)
- new net MISO: U13.2 (SO)
- new net MOSI: U13.5 (SI)
- new net MRAM_CS: U13.1 (CS)
- new net RBF_SW: J7.2 (Pin_2), Q4.2 (G), R15.2
- new net SCK: U13.6 (SCK)
- new net VBATT_PRE_INH: J4.1 (Pin_1), Q5.3 (S)
- new net WRITE_PROT: U13.3 (WP)
- new net ~{ADCS_PWR_FAULT}: U11.17 (~{FAULT})
- new net ~{CHRG_FAULT}: D11.2 (A), U12.J7 (~{FAULT})
- new net ~{CHRG_STAT}: D7.2 (A), U12.K7 (~{CHRG})
Other:
- note added: "1206"
- note added: "2512 (3W)"
- note added: "50k = 1A Limit"
- note added: "ALL PASSIVES ARE 0603 UNLESS OTHERWISE SPECIFIED"
- note added: "ALL PASSIVES ARE 0805"
- note removed: "ALL COMPONENTS ARE 0603 UNLESS OTHERWISE SPECIFIED"
- note removed: "TO-263 (35W)"
- moved on the sheet: C12, C24, C3, D1, D2, D3, H1, H2, H3, H4, J11, J12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
